File: elec/src/components/lv2842xlvddcr/elec/layout/default/LV2842Kit.kicad_pcb (KiCad board)
At the start: 2 copper layers, 8 parts

Commit message: layout complete
Parts:
- C1: value 10V 10uF X5R ±10% 0603 Multilayer Ceramic Capacitors MLCC - SMD/SMT ROHS -> 2.2µF ±20% 6.3V X5R; footprint lib:C0603 -> atopile:C0402-b3ef17
- C2: value 25V 10uF X5R ±10% 0805 Multilayer Ceramic Capacitors MLCC - SMD/SMT ROHS -> 10µF ±10% 25V X5R; footprint lib:C0805 -> atopile:C0805-3b2e55
- C3: value 16V 100nF X7R ±10% 0402 Multilayer Ceramic Capacitors MLCC - SMD/SMT ROHS -> 470nF ±20% 16V X5R; footprint lib:C0402 -> atopile:C0402-b3ef17
- R1: value 62.5mW Thick Film Resistors 50V ±100ppm/℃ ±1% 14.3kΩ 0402 Chip Resistor - Surface Mount ROHS -> 1kΩ ±1% 62.5mW; footprint lib:R0402 -> atopile:R0402-56259e
- R2: value 62.5mW Thick Film Resistors 50V ±100ppm/℃ ±1% 4.3kΩ 0402 Chip Resistor - Surface Mount ROHS -> 1kΩ ±1% 62.5mW; footprint lib:R0402 -> atopile:R0402-56259e
Connections:
- net cb renamed CB
- net out renamed FB
- net sw renamed cathode
- net vcc renamed VIN
- net vcc-1 renamed hv
