File: elec/layout/cm4-example/cm4-example.kicad_pcb (KiCad board)
At the start: 4 copper layers, 100 x 100 mm, 109 parts, among them U10 10kΩ ±1% 62.5mW, U11 10kΩ ±1% 62.5mW, U13 1kΩ ±1% 62.5mW, U14 1kΩ ±1% 62.5mW, U15 100nF ±10% 16V X7R, U16 10kΩ ±1% 62.5mW, U17 10kΩ ±1% 62.5mW, U19 100nF ±10% 16V X7R, U2 1µF ±10% 25V X5R, U20 10kΩ ±1% 62.5mW, U21 10kΩ ±1% 62.5mW, U22 1kΩ ±1% 62.5mW, U23 1kΩ ±1% 62.5mW, U24 1µF ±10% 25V X5R, U26 1µF ±10% 25V X5R, U27 4.7µF ±10% 10V X5R, U28 10µF ±10% 10V X5R, U3 10kΩ ±1% 62.5mW, U31 1µF ±10% 25V X5R, U33 10pF ±5% 50V C0G, U34 10pF ±5% 50V C0G, U35 4.7µF ±10% 10V X5R, U36 10µF ±10% 10V X5R, U38 4.7nF ±10% 50V X7R, U39 60.4Ω ±1% 100mW, U4 10kΩ ±1% 62.5mW, U40 60.4Ω ±1% 100mW, U41 1µF ±10% 25V X5R, U42 1µF ±10% 25V X5R, U45 100nF ±10% 16V X7R, U46 2.2µF ±10% 25V X5R, U48 10kΩ ±1% 62.5mW, U49 10kΩ ±1% 62.5mW, U50 10kΩ ±1% 62.5mW, U51 10kΩ ±1% 62.5mW, U52 10kΩ ±1% 62.5mW, U53 10kΩ ±1% 62.5mW, U54 10kΩ ±1% 62.5mW, U55 10kΩ ±1% 62.5mW, U56 10kΩ ±1% 62.5mW, U57 10kΩ ±1% 62.5mW, U58 10kΩ ±1% 62.5mW, U59 10kΩ ±1% 62.5mW, U6 1kΩ ±1% 62.5mW, U60 10kΩ ±1% 62.5mW, U61 10kΩ ±1% 62.5mW, U62 10kΩ ±1% 62.5mW, U63 10kΩ ±1% 62.5mW, U64 10kΩ ±1% 62.5mW, U65 1kΩ ±1% 62.5mW, U66 1kΩ ±1% 62.5mW, U67 1µF ±10% 25V X5R, U69 1µF ±10% 25V X5R, U7 1kΩ ±1% 62.5mW, U70 470nF ±20% 16V X5R, U71 1kΩ ±1% 62.5mW, U72 1kΩ ±1% 62.5mW, U75 2.2µF ±20% 6.3V X5R, U76 10µF ±10% 25V X5R, U9 1µF ±10% 25V X5R

Commit message: Cleanup DRCs
Parts:
- moved U74 0.28 mm to (131.1, 76.7)
- moved DS1 0.28 mm to (133.4, 72.4)
- moved U71 0.28 mm to (125.9, 77.1)
- moved U72 0.28 mm to (125.9, 75.2)
- moved U73 0.28 mm to (129.8, 72.2)
- moved U75 0.28 mm to (127.3, 72.6)
- moved U76 0.28 mm to (127.4, 76.3)
- moved U70 0.28 mm to (132.0, 72.9)
Routing:
- net GND: track 0.00 -> 134.9 mm, vias 0 -> 33
- net (no net): track 95.7 -> 0.00 mm, vias 22 -> 0
- net analog_in_1.amplifier.opamp.footprint.pins[6].net-net: track 34.8 -> 0.00 mm, vias 5 -> 0
- net SDA: track 100.0 -> 101.4 mm
- net regulator_5v-out: track 8.33 -> 9.52 mm
- added copper zone on B.Cu, net GND
- added copper zone on F.Cu, net GND
- added copper zone on In2.Cu, net VCC_5V
- removed copper zone on B.Cu, net (none)
- removed copper zone on F.Cu, net (none)
- removed copper zone on In2.Cu, net (none)
- removed copper zone on B.Cu, net VCC_5V

Commit message: layout complete
Parts:
- added USB2: , lib:USB-C-SMD_TYC-324G-a50b79, F.Cu at (198.4, 121.1)
Connections:
- net A10 renamed SSRXN2
- net A11 renamed SSRXP2
- net A2 renamed usb_pd.usb_connector-A2
- net A3 renamed usb_pd.usb_connector-A3
- net A8 renamed usb_pd.usb_connector-A8
- net ADJ_NC renamed analog_in_2.regulator_3v3_isolated-out
- net B10 renamed usb_pd.usb_connector-B10
- net B11 renamed usb_pd.usb_connector-B11
- net B2 renamed SSTXP2
- net B3 renamed SSTXN2
- net B8 renamed SBU2
- net controller.cm4-pins[38] renamed controller.cm4-line-6
- net controller.cm4-pins[46] renamed pins[46]
- net controller.cm4-pins[46]-1 renamed controller.cm4-line-8
- net controller.cm4.hdi_b-pins[26] renamed pins[26]
- net controller.cm4.hdi_b-pins[38] renamed pins[38]
- net pins[55] renamed controller.cm4-line-4
- CN1 pad 20: controller.cm4-line-2 -> controller.cm4-line-5
- CN1 pad 29: controller.cm4-line-3 -> pins[57]
- CN1 pad 75: pins[50] -> controller.cm4-line-2
- CN1 pad 78: controller.cm4-pins[44]-1 -> controller.cm4-pins[44]
- CN1 pad 80: controller.cm4-line-1 -> controller.cm4-line-7
- CN1 pad 85: pins[30] -> controller.cm4-line-1
- CN1 pad 87: controller.cm4-pins[26] -> controller.cm4-line-3
- CN2 pad 78: controller.cm4-pins[44] -> controller.cm4-pins[44]-1
- D1 pad 1: cathode-2 -> cathode
- D2 pad 1: cathode -> cathode-2
- D2 pad 2: gnd -> gnd-2
- D3 pad 3: gnd-2 -> gnd
- D4 pad 1: controller.cm4-cathode -> controller.cm4-cathode-1
- D5 pad 1: controller.cm4-cathode-1 -> controller.cm4-cathode
- J1 pad 4: gnd-2 -> gnd
- R1 pad 1: controller.cm4-cathode -> controller.cm4-cathode-1
- R2 pad 1: controller.cm4-cathode-1 -> controller.cm4-cathode
- R3 pad 2: controller.rj45-anode -> controller.rj45-anode-1
- R4 pad 2: controller.rj45-anode-1 -> controller.rj45-anode
- RF2 pad 2: gnd -> gnd-2
- RF2 pad 3: gnd -> gnd-2
- RF2 pad 4: gnd -> gnd-2
- RJ1 pad 12: controller.rj45-anode -> controller.rj45-anode-1
- RJ1 pad 13: controller.rj45-anode-1 -> controller.rj45-anode
- RJ1 pad P1: controller.rj45.connector-net-1 -> controller.rj45.connector-net
- RJ1 pad P10: controller.rj45.connector-net -> controller.rj45.connector-net-1
- U1 pad 10: line-2 -> line
- U1 pad 4: output-1 -> output
- U1 pad 8: hv-1 -> hv-3
- U1 pad 9: line-3 -> line-2
- U10 pad 2: output -> output-1
- U11 pad 1: gnd -> gnd-2
- U12 pad 1: output -> output-1
- U12 pad 3: cathode -> cathode-2
- U12 pad 4: gnd -> gnd-2
- U12 pad 8: hv-3 -> hv
- U13 pad 1: cathode -> cathode-2
- U13 pad 2: gnd -> gnd-2
- U14 pad 2: cathode -> cathode-2
- U15 pad 1: hv-3 -> hv
- U15 pad 2: gnd -> gnd-2
- U16 pad 2: hv-3 -> hv
- U17 pad 2: hv-3 -> hv
- U18 pad 1: hv-1 -> hv-3
- U18 pad 2: line-1 -> line-3
- U18 pad 3: line -> line-1
- U18 pad 5: gnd -> gnd-2
- U18 pad 8: hv-3 -> hv
- U19 pad 1: hv-1 -> hv-3
- U2 pad 1: hv-1 -> hv-3
- U20 pad 1: line -> line-1
- U20 pad 2: hv-1 -> hv-3
- U21 pad 1: line-1 -> line-3
- U21 pad 2: hv-1 -> hv-3
- U22 pad 2: gnd -> gnd-2
- U23 pad 1: hv-3 -> hv
- U24 pad 1: hv -> hv-1
- U24 pad 2: gnd -> gnd-2
- U25 pad 1: hv -> hv-1
- U25 pad 2: gnd -> gnd-2
- U25 pad 3: hv -> hv-1
- U25 pad 5: hv-3 -> hv
- U26 pad 1: hv-3 -> hv
- U26 pad 2: gnd -> gnd-2
- U28 pad 1: hv -> hv-1
- U28 pad 2: gnd -> gnd-2
- U29 pad 4: gnd -> gnd-2
- U29 pad 6: hv -> hv-1
- U3 pad 2: output-1 -> output
- U30 pad 14: hv-1 -> hv-3
- U31 pad 1: hv-1 -> hv-3
- U36 pad 2: gnd-2 -> gnd
- U37 pad 4: gnd-2 -> gnd
- U38 pad 2: gnd-2 -> gnd
- U41 pad 1: hv-1 -> hv-3
- U42 pad 2: gnd-2 -> gnd
- U43 pad 1: hv-1 -> hv-3
- U43 pad 7: gnd-2 -> gnd
- U45 pad 1: hv-1 -> hv-3
- U46 pad 1: hv-1 -> hv-3
- U47 pad 10: i2c_multiplexer-line-7 -> i2c_multiplexer-line-11
- U47 pad 11: i2c_multiplexer-line-10 -> i2c_multiplexer-line-5
- U47 pad 13: line-1 -> line-3
- U47 pad 14: line -> line-1
- U47 pad 15: i2c_multiplexer-line-5 -> i2c_multiplexer-line-4
- U47 pad 16: i2c_multiplexer-line-9 -> i2c_multiplexer-line-7
- U47 pad 18: i2c_multiplexer-line-2 -> i2c_multiplexer-line
- U47 pad 19: i2c_multiplexer-line-11 -> i2c_multiplexer-line-9
- U47 pad 20: i2c_multiplexer-line -> i2c_multiplexer-line-10
- U47 pad 24: hv-1 -> hv-3
- U47 pad 4: line-3 -> line-2
- U47 pad 5: line-2 -> line
- U47 pad 7: i2c_multiplexer-line-6 -> i2c_multiplexer-line-8
- U47 pad 8: i2c_multiplexer-line-8 -> i2c_multiplexer-line-6
- U47 pad 9: i2c_multiplexer-line-4 -> i2c_multiplexer-line-2
- U48 pad 1: hv-1 -> hv-3
- U48 pad 2: line-2 -> line
- U49 pad 1: hv-1 -> hv-3
- U49 pad 2: line-3 -> line-2
- U5 pad 1: output-1 -> output
- U5 pad 3: cathode-2 -> cathode
- U5 pad 8: hv-1 -> hv-3
- U50 pad 1: hv-1 -> hv-3
- U50 pad 2: i2c_multiplexer-line-6 -> i2c_multiplexer-line-8
- U51 pad 1: hv-1 -> hv-3
- U52 pad 1: hv-1 -> hv-3
- U52 pad 2: i2c_multiplexer-line-4 -> i2c_multiplexer-line-2
- U53 pad 1: hv-1 -> hv-3
- U53 pad 2: i2c_multiplexer-line-8 -> i2c_multiplexer-line-6
- U54 pad 1: hv-1 -> hv-3
- U54 pad 2: i2c_multiplexer-line-10 -> i2c_multiplexer-line-5
- U55 pad 1: hv-1 -> hv-3
- U55 pad 2: i2c_multiplexer-line-7 -> i2c_multiplexer-line-11
- U56 pad 1: hv-1 -> hv-3
- U56 pad 2: line -> line-1
- U57 pad 1: hv-1 -> hv-3
- U57 pad 2: line-1 -> line-3
- U58 pad 1: hv-1 -> hv-3
- U58 pad 2: i2c_multiplexer-line-9 -> i2c_multiplexer-line-7
- U59 pad 1: hv-1 -> hv-3
- U59 pad 2: i2c_multiplexer-line-5 -> i2c_multiplexer-line-4
- U6 pad 1: cathode-2 -> cathode
- U60 pad 1: hv-1 -> hv-3
- U60 pad 2: i2c_multiplexer-line-2 -> i2c_multiplexer-line
- U61 pad 1: hv-1 -> hv-3
- U62 pad 1: hv-1 -> hv-3
- U62 pad 2: i2c_multiplexer-line -> i2c_multiplexer-line-10
- U63 pad 1: hv-1 -> hv-3
- U63 pad 2: i2c_multiplexer-line-11 -> i2c_multiplexer-line-9
- U64 pad 2: hv-1 -> hv-3
- U66 pad 1: hv-1 -> hv-3
- U68 pad 5: hv-1 -> hv-3
- U69 pad 1: hv-1 -> hv-3
- U7 pad 2: cathode-2 -> cathode
- U77 pad 1: usb_pd.pd_controller.pd_controller-line -> usb_pd.pd_controller.pd_controller-line-1
- U77 pad 5: usb_pd.pd_controller.pd_controller-line-1 -> usb_pd.pd_controller.pd_controller-line
- U8 pad 1: gnd -> gnd-2
- U8 pad 3: gnd -> gnd-2
- U8 pad 4: output -> output-1
- U8 pad 8: hv-3 -> hv
- U9 pad 1: hv-3 -> hv
- U9 pad 2: gnd -> gnd-2
Routing:
- net USB2_D_N: track 0.00 -> 86.2 mm, vias 0 -> 3
- net USB2_D_P: track 0.00 -> 85.0 mm, vias 0 -> 3
- net hv-1: track 80.0 -> 14.9 mm, vias 13 -> 0
- net hv-3: track 33.2 -> 80.0 mm, vias 2 -> 13
- net gnd-2: track 52.2 -> 91.7 mm, vias 0 -> 4
- net gnd: track 91.7 -> 52.2 mm, vias 4 -> 0
- net hv: track 14.9 -> 33.2 mm, vias 0 -> 2
- net line-3: track 18.0 -> 32.0 mm
- net line: track 30.9 -> 18.6 mm
- net GND: track 134.9 -> 141.7 mm
- net VCC_5V: track 28.1 -> 33.4 mm, vias 13 -> 17
- net line-1: track 32.0 -> 30.9 mm
- net i2c_multiplexer-line-11: track 3.89 -> 2.94 mm
- net i2c_multiplexer-line-9: track 3.07 -> 3.89 mm
- net i2c_multiplexer-line: track 4.21 -> 3.40 mm
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- added copper zone on In1.Cu, net hv-3
- removed copper zone on In1.Cu, net hv-1
Other:
- board text added: "5V"
- board text added: "AIN1"
- board text added: "AIN2-ISO"
- board text added: "CAN"
- board text added: "CANH"
- board text added: "CANL"
- board text added: "CM4 Example"
- board text added: "GND"
- board text added: "USB2"
- board text added: "USBPD input"

Commit message: rebuild all modules
Connections:
- net A10 renamed usb_connector-A10
- net A11 renamed usb_connector-A11
- net B2 renamed usb_connector-B2
- net B3 renamed usb_connector-B3
- net B8 renamed usb_connector-B8
- net CLKO_SOF renamed can_interface.controller-io-2
- net INT0h_GPIO0_XSTBY renamed can_interface.controller-io-3
- net SBU2 renamed usb_pd.usb_connector-B8
- net SSRXN2 renamed usb_pd.usb_connector-A10
- net SSRXP2 renamed usb_pd.usb_connector-A11
- net SSTXN2 renamed usb_pd.usb_connector-B3
- net SSTXP2 renamed usb_pd.usb_connector-B2
- net usb_connector-A2 renamed SSTXP1
- net usb_connector-A3 renamed SSTXN1
- net usb_connector-A8 renamed usb_connector-SBU1
- net usb_connector-B10 renamed SSRXN1
- net usb_connector-B11 renamed SSRXP1
- net usb_pd.usb_connector-A2 renamed A2
- net usb_pd.usb_connector-A3 renamed A3
- net usb_pd.usb_connector-A8 renamed usb_pd.usb_connector-SBU1
- net usb_pd.usb_connector-B10 renamed B10
- net usb_pd.usb_connector-B11 renamed B11
- CN1 pad 22: controller.cm4-line -> controller.cm4-line-4
- CN1 pad 24: pins[47] -> controller.cm4-line-6
- CN1 pad 28: controller.cm4-line-4 -> controller.cm4-line-2
- CN1 pad 75: controller.cm4-line-2 -> controller.cm4-line
- CN1 pad 77: controller.cm4-line-8 -> controller.cm4-line-3
- CN1 pad 80: controller.cm4-line-7 -> controller.cm4-line-1
- CN1 pad 81: controller.cm4-line-6 -> controller.cm4-line-9
- CN1 pad 85: controller.cm4-line-1 -> controller.cm4-line-7
- CN1 pad 87: controller.cm4-line-3 -> controller.cm4-line-8
- D2 pad 1: cathode-2 -> cathode-1
- DS1 pad 1: cathode-1 -> cathode-2
- R3 pad 2: controller.rj45-anode-1 -> controller.rj45-anode
- R4 pad 2: controller.rj45-anode -> controller.rj45-anode-1
- RF1 pad 1: io -> io-1
- RF2 pad 1: io-1 -> io
- RJ1 pad 12: controller.rj45-anode-1 -> controller.rj45-anode
- RJ1 pad 13: controller.rj45-anode -> controller.rj45-anode-1
- RJ1 pad P1: controller.rj45.connector-net -> controller.rj45.connector-net-1
- RJ1 pad P10: controller.rj45.connector-net-1 -> controller.rj45.connector-net
- U1 pad 10: line -> line-3
- U1 pad 4: output -> output-1
- U1 pad 9: line-2 -> line-1
- U10 pad 1: inverting -> inverting-1
- U10 pad 2: output-1 -> output
- U11 pad 2: inverting -> inverting-1
- U12 pad 1: output-1 -> output
- U12 pad 2: inverting -> inverting-1
- U12 pad 3: cathode-2 -> cathode-1
- U12 pad 8: hv -> hv-1
- U13 pad 1: cathode-2 -> cathode-1
- U14 pad 1: io-1 -> io
- U14 pad 2: cathode-2 -> cathode-1
- U15 pad 1: hv -> hv-1
- U16 pad 2: hv -> hv-1
- U17 pad 2: hv -> hv-1
- U18 pad 2: line-3 -> line-2
- U18 pad 3: line-1 -> line
- U18 pad 8: hv -> hv-1
- U20 pad 1: line-1 -> line
- U21 pad 1: line-3 -> line-2
- U23 pad 1: hv -> hv-1
- U24 pad 1: hv-1 -> hv
- U25 pad 1: hv-1 -> hv
- U25 pad 3: hv-1 -> hv
- U25 pad 5: hv -> hv-1
- U26 pad 1: hv -> hv-1
- U28 pad 1: hv-1 -> hv
- U29 pad 6: hv-1 -> hv
- U3 pad 1: inverting-1 -> inverting
- U3 pad 2: output -> output-1
- U30 pad 4: INTh -> can_interface.controller-io
- U30 pad 8: can_interface.controller-io -> can_interface.controller-io-1
- U4 pad 2: inverting-1 -> inverting
- U47 pad 10: i2c_multiplexer-line-11 -> i2c_multiplexer-line-3
- U47 pad 11: i2c_multiplexer-line-5 -> i2c_multiplexer-line-8
- U47 pad 13: line-3 -> line-2
- U47 pad 14: line-1 -> line
- U47 pad 15: i2c_multiplexer-line-4 -> i2c_multiplexer-line
- U47 pad 16: i2c_multiplexer-line-7 -> i2c_multiplexer-line-6
- U47 pad 17: i2c_multiplexer-line-1 -> i2c_multiplexer-line-10
- U47 pad 18: i2c_multiplexer-line -> i2c_multiplexer-line-11
- U47 pad 19: i2c_multiplexer-line-9 -> i2c_multiplexer-line-4
- U47 pad 20: i2c_multiplexer-line-10 -> i2c_multiplexer-line-9
- U47 pad 4: line-2 -> line-1
- U47 pad 5: line -> line-3
- U47 pad 6: i2c_multiplexer-line-3 -> i2c_multiplexer-line-1
- U47 pad 7: i2c_multiplexer-line-8 -> i2c_multiplexer-line-5
- U47 pad 8: i2c_multiplexer-line-6 -> i2c_multiplexer-line-2
- U47 pad 9: i2c_multiplexer-line-2 -> i2c_multiplexer-line-7
- U48 pad 2: line -> line-3
- U49 pad 2: line-2 -> line-1
- U5 pad 1: output -> output-1
- U5 pad 2: inverting-1 -> inverting
- U50 pad 2: i2c_multiplexer-line-8 -> i2c_multiplexer-line-5
- U51 pad 2: i2c_multiplexer-line-3 -> i2c_multiplexer-line-1
- U52 pad 2: i2c_multiplexer-line-2 -> i2c_multiplexer-line-7
- U53 pad 2: i2c_multiplexer-line-6 -> i2c_multiplexer-line-2
- U54 pad 2: i2c_multiplexer-line-5 -> i2c_multiplexer-line-8
- U55 pad 2: i2c_multiplexer-line-11 -> i2c_multiplexer-line-3
- U56 pad 2: line-1 -> line
- U57 pad 2: line-3 -> line-2
- U58 pad 2: i2c_multiplexer-line-7 -> i2c_multiplexer-line-6
- U59 pad 2: i2c_multiplexer-line-4 -> i2c_multiplexer-line
- U60 pad 2: i2c_multiplexer-line -> i2c_multiplexer-line-11
- U61 pad 2: i2c_multiplexer-line-1 -> i2c_multiplexer-line-10
- U62 pad 2: i2c_multiplexer-line-10 -> i2c_multiplexer-line-9
- U63 pad 2: i2c_multiplexer-line-9 -> i2c_multiplexer-line-4
- U7 pad 1: io -> io-1
- U70 pad 2: cathode-1 -> cathode-2
- U73 pad 6: cathode-1 -> cathode-2
- U74 pad 1: cathode-1 -> cathode-2
- U77 pad 1: usb_pd.pd_controller.pd_controller-line-1 -> usb_pd.pd_controller.pd_controller-line
- U77 pad 5: usb_pd.pd_controller.pd_controller-line -> usb_pd.pd_controller.pd_controller-line-1
- U8 pad 4: output-1 -> output
- U8 pad 8: hv -> hv-1
- U9 pad 1: hv -> hv-1
- USB2 pad B5: (no net) -> B5
Routing:
- net GND: track 141.7 -> 0.00 mm, vias 33 -> 0
- net (no net): track 0.00 -> 141.7 mm, vias 0 -> 33
- net hv-1: track 14.9 -> 33.2 mm, vias 0 -> 2
- net hv: track 33.2 -> 14.9 mm, vias 2 -> 0
- net line-2: track 18.0 -> 32.0 mm
- net line-3: track 32.0 -> 18.6 mm
- net line-1: track 30.9 -> 18.0 mm
- net line: track 18.6 -> 30.9 mm
- net cathode-2: track 8.99 -> 0.00 mm
- net cathode-1: track 0.00 -> 8.99 mm
- net io-1: track 13.9 -> 7.82 mm
- net io: track 7.82 -> 13.9 mm
- net i2c_multiplexer-line-4: track 2.91 -> 3.89 mm
- net i2c_multiplexer-line-10: track 4.21 -> 3.24 mm
- net i2c_multiplexer-line-8: track 2.84 -> 3.42 mm
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- added copper zone on B.Cu, net (none)
- added copper zone on F.Cu, net (none)
- added copper zone on F.Cu, net cathode-2
- removed copper zone on B.Cu, net GND
- removed copper zone on F.Cu, net GND
- removed copper zone on F.Cu, net cathode-1
