File: elec/layout/buck-boost/buck-boost.kicad_pcb (KiCad board)
At the start: 2 copper layers, 0 parts

Commit message: core layout, rebuild modules with compiler updates
Parts:
- added C1: 68µF ±20% infV, atopile:CAP-SMD_BD10.0-L10.3-W10.3-LS11.6-FD-b102ff, F.Cu at (142.9, 64.2)
- added C2: 68µF ±20% infV, atopile:CAP-SMD_BD10.0-L10.3-W10.3-LS11.6-FD-b102ff, F.Cu at (203.2, 74.9)
- added C3: 68µF ±20% infV, atopile:CAP-SMD_BD10.0-L10.3-W10.3-LS11.6-FD-b102ff, F.Cu at (142.9, 74.8)
- added C4: 68µF ±20% infV, atopile:CAP-SMD_BD10.0-L10.3-W10.3-LS11.6-FD-b102ff, F.Cu at (203.2, 64.3)
- added DS1: , atopile:DO-219AB_L2.8-W1.8-LS3.7-RD-212ba1, F.Cu at (80.1, 60.0)
- added DS2: , atopile:DO-219AB_L2.8-W1.8-LS3.7-RD-212ba1, F.Cu at (80.2, 57.3)
- added Q1: , atopile:POWERVDFN-8_L5.8-W4.9-P1.27-LS6.2-BL-167b96, F.Cu at (158.9, 66.9)
- added Q2: , atopile:POWERVDFN-8_L5.8-W4.9-P1.27-LS6.2-BL-167b96, F.Cu at (159.1, 72.3)
- added Q3: , atopile:POWERVDFN-8_L5.8-W4.9-P1.27-LS6.2-BL-167b96, F.Cu at (187.0, 66.9)
- added Q4: , atopile:POWERVDFN-8_L5.8-W4.9-P1.27-LS6.2-BL-167b96, F.Cu at (186.8, 72.3)
- added U1: , atopile:TQFN-36_L6.0-W5.0-P0.50-BL-EP-1-2fce41, F.Cu at (122.9, 68.6)
- added U10: 2.49kΩ ±1% 100mW, atopile:R0603-ebcab9, F.Cu at (133.5, 26.3)
- added U11: 4.7µF ±10% 100V X7R, atopile:C1210-c93926, F.Cu at (157.6, 61.6)
- added U12: 4.7µF ±10% 100V X7R, atopile:C1210-c93926, F.Cu at (160.9, 77.6)
- added U13: 4.7µF ±10% 100V X7R, atopile:C1210-c93926, F.Cu at (160.7, 61.6)
- added U14: 10µF ±10% 100V X7R, atopile:C1210-c93926, F.Cu at (151.2, 61.6)
- added U15: 10µF ±10% 100V X7R, atopile:C1210-c93926, F.Cu at (151.5, 77.6)
- added U16: 10µF ±10% 100V X7R, atopile:C1210-c93926, F.Cu at (154.4, 61.6)
- added U17: 10µF ±10% 100V X7R, atopile:C1210-c93926, F.Cu at (154.6, 77.6)
- added U18: 1µF ±10% 100V X7R, atopile:C1206-f0a137, F.Cu at (150.5, 69.5)
- added U19: 100nF ±10% 100V X7R, atopile:C0805-3b2e55, F.Cu at (152.5, 69.6)
- added U2: 100nF ±10% 50V X7R, atopile:C0603-bd72f6, F.Cu at (165.8, 79.5)
- added U20: 100pF ±5% 100V C0G, atopile:C0805-3b2e55, F.Cu at (154.4, 69.6)
- added U21: 470nF ±20% 16V X5R, atopile:C0402-b3ef17, F.Cu at (185.3, 37.7)
- added U22: 100nF ±10% 16V X7R, atopile:C0402-b3ef17, F.Cu at (150.7, 37.4)
- added U23: 10Ω ±1% 62.5mW, atopile:R0402-56259e, F.Cu at (144.0, 50.6)
- added U24: 100nF ±10% 16V X7R, atopile:C0402-b3ef17, F.Cu at (137.2, 39.2)
- added U25: 10Ω ±1% 62.5mW, atopile:R0402-56259e, F.Cu at (132.6, 43.2)
- added U26: 5mΩ ±1% 1W, atopile:R1206-bdb864, F.Cu at (136.4, 69.5)
- added U27: 4.7µF ±10% 100V X7R, atopile:C1210-c93926, F.Cu at (188.3, 77.6)
- added U28: 4.7µF ±10% 100V X7R, atopile:C1210-c93926, F.Cu at (188.3, 61.6)
- added U29: 4.7µF ±10% 100V X7R, atopile:C1210-c93926, F.Cu at (185.0, 77.6)
- added U3: 100nF ±10% 50V X7R, atopile:C0603-bd72f6, F.Cu at (187.6, 32.0)
- added U30: 10µF ±10% 100V X7R, atopile:C1210-c93926, F.Cu at (191.5, 61.6)
- added U31: 10µF ±10% 100V X7R, atopile:C1210-c93926, F.Cu at (194.7, 77.6)
- added U32: 10µF ±10% 100V X7R, atopile:C1210-c93926, F.Cu at (191.5, 77.6)
- added U33: 10µF ±10% 100V X7R, atopile:C1210-c93926, F.Cu at (194.7, 61.6)
- added U34: 1µF ±10% 100V X7R, atopile:C1206-f0a137, F.Cu at (195.6, 69.5)
- added U35: 100nF ±10% 100V X7R, atopile:C0805-3b2e55, F.Cu at (193.4, 69.6)
- added U36: 100pF ±5% 100V C0G, atopile:C0805-3b2e55, F.Cu at (191.4, 69.6)
- added U37: 470nF ±20% 16V X5R, atopile:C0402-b3ef17, F.Cu at (169.9, 31.0)
- added U38: 100nF ±10% 16V X7R, atopile:C0402-b3ef17, F.Cu at (152.6, 43.2)
- added U39: 10Ω ±1% 62.5mW, atopile:R0402-56259e, F.Cu at (192.6, 43.2)
- added U4: 0Ω 100mW, atopile:R0603-ebcab9, F.Cu at (128.3, 61.4)
- added U40: 100nF ±10% 16V X7R, atopile:C0402-b3ef17, F.Cu at (163.5, 26.3)
- added U41: 10Ω ±1% 62.5mW, atopile:R0402-56259e, F.Cu at (201.0, 54.2)
- added U42: 5mΩ ±1% 1W, atopile:R1206-bdb864, F.Cu at (209.8, 69.4)
- added U43: 13.7kΩ ±1% 62.5mW, atopile:R0402-56259e, F.Cu at (159.9, 31.0)
- added U44: 249kΩ ±1% 62.5mW, atopile:R0402-56259e, F.Cu at (177.6, 32.0)
- added U45: 1MΩ ±1% 250mW, atopile:R1206-bdb864, F.Cu at (110.2, 77.4)
- added U46: 133kΩ ±1% 62.5mW, atopile:R0402-56259e, F.Cu at (175.3, 37.7)
- added U47: 25.5kΩ ±1% 62.5mW, atopile:R0402-56259e, F.Cu at (202.6, 43.2)
- added U48: 4.7µF ±10% 25V X5R, atopile:C0805-3b2e55, F.Cu at (172.3, 86.0)
- added U49: 100nF ±10% 100V X7R, atopile:C0805-3b2e55, F.Cu at (147.6, 32.0)
- added U5: 0Ω 100mW, atopile:R0603-ebcab9, F.Cu at (153.7, 74.0)
- added U50: 1µF ±10% 100V X7R, atopile:C1206-f0a137, F.Cu at (112.6, 77.3)
- added U51: 4.7µF ±10% 100V X7R, atopile:C1210-c93926, F.Cu at (157.8, 77.6)
- added U52: 4.7µF ±10% 100V X7R, atopile:C1210-c93926, F.Cu at (185.1, 61.6)
- added U6: 0Ω 100mW, atopile:R0603-ebcab9, F.Cu at (167.2, 39.2)
- added U7: 0Ω 100mW, atopile:R0603-ebcab9, F.Cu at (182.1, 91.9)
- added U8: , atopile:IND-SMD_L17.2-W17.2-132628, F.Cu at (172.9, 69.4)
- added U9: 4.7µF ±10% 25V X5R, atopile:C0805-3b2e55, F.Cu at (137.6, 32.0)
Routing:
- net input_switching_node: track 0.00 -> 10.3 mm
