File: elec/layout/buck-boost/buck-boost.kicad_pcb (KiCad board)
At the start: 6 copper layers, 69 parts, among them U10 2.49kΩ ±1% 62.5mW, U11 4.7µF ±10% 100V X7R, U12 4.7µF ±10% 100V X7R, U13 4.7µF ±10% 100V X7R, U14 10µF ±10% 100V X7S, U15 10µF ±10% 100V X7S, U16 10µF ±10% 100V X7S, U17 10µF ±10% 100V X7S, U18 1µF ±10% 100V X7R, U19 100nF ±10% 100V X7R, U2 100nF ±10% 50V X7R, U20 100pF ±5% 100V C0G, U21 470nF ±20% 16V X5R, U22 100nF ±10% 16V X7R, U23 10Ω ±1% 62.5mW, U24 100nF ±10% 16V X7R, U25 10Ω ±1% 62.5mW, U26 5mΩ ±1% 1W, U27 4.7µF ±10% 100V X7R, U28 4.7µF ±10% 100V X7R, U29 4.7µF ±10% 100V X7R, U3 100nF ±10% 50V X7R, U30 10µF ±10% 100V X7S, U31 10µF ±10% 100V X7S, U32 10µF ±10% 100V X7S, U33 10µF ±10% 100V X7S, U34 1µF ±10% 100V X7R, U35 100nF ±10% 100V X7R, U36 100pF ±5% 100V C0G, U37 470nF ±20% 16V X5R, U38 100nF ±10% 16V X7R, U39 10Ω ±1% 62.5mW, U4 50kΩ ±1% 62.5mW, U40 100nF ±10% 16V X7R, U41 10Ω ±1% 62.5mW, U42 5mΩ ±1% 1W, U43 13.7kΩ ±1% 62.5mW, U44 249kΩ ±1% 100mW, U45 1MΩ ±1% 100mW, U46 133kΩ ±1% 100mW, U47 25.5kΩ ±0% 100mW, U48 4.7µF ±10% 25V X5R, U49 100nF ±10% 100V X7R, U50 1µF ±10% 250V X7R, U51 4.7µF ±10% 100V X7R, U52 4.7µF ±10% 100V X7R, U54 0Ω 62.5mW, U58 30.1kΩ ±1% 62.5mW, U59 5.23kΩ ±1% 100mW, U9 4.7µF ±10% 25V X5R

Commit message: reduce led brightness on buck-boost indicator leds
Parts:
- R1, R2, R3: value 100Ω ±1% 62.5mW -> 2.7kΩ ±1% 62.5mW
- U14, U15, U16, U17, U30, U31, U32, U33: value 10µF ±10% 100V X7S -> 10µF ±10% 100V X7R
Connections:
- net line-8 renamed gate
- net source renamed drain
- C1 pad 1: hv-3 -> hv
- C1 pad 2: gnd-1 -> gnd
- C2 pad 1: hv-1 -> hv-2
- C2 pad 2: gnd-1 -> gnd
- C3 pad 1: hv -> hv-3
- C3 pad 2: gnd-1 -> gnd
- C4 pad 1: hv-2 -> hv-1
- C4 pad 2: gnd-1 -> gnd
- Q1 pad 4: line-3 -> line-6
- Q1 pad 5: hv-3 -> hv
- Q1 pad 6: hv-3 -> hv
- Q1 pad 7: hv-3 -> hv
- Q1 pad 8: hv-3 -> hv
- Q2 pad 1: gnd-1 -> gnd
- Q2 pad 2: gnd-1 -> gnd
- Q2 pad 3: gnd-1 -> gnd
- Q3 pad 1: line-6 -> line-2
- Q3 pad 2: line-6 -> line-2
- Q3 pad 3: line-6 -> line-2
- Q3 pad 4: line-2 -> line-4
- Q3 pad 5: hv-1 -> hv-2
- Q3 pad 6: hv-1 -> hv-2
- Q3 pad 7: hv-1 -> hv-2
- Q3 pad 8: hv-1 -> hv-2
- Q4 pad 1: gnd-1 -> gnd
- Q4 pad 2: gnd-1 -> gnd
- Q4 pad 3: gnd-1 -> gnd
- Q4 pad 4: line -> gate-1
- Q4 pad 5: line-6 -> line-2
- Q4 pad 6: line-6 -> line-2
- Q4 pad 7: line-6 -> line-2
- Q4 pad 8: line-6 -> line-2
- R1 pad 2: gnd-2 -> gnd-4
- R2 pad 2: gnd-4 -> gnd-1
- R3 pad 2: gnd -> gnd-3
- U1 pad 11: gnd-3 -> gnd-2
- U1 pad 13: line-7 -> line-1
- U1 pad 14: line-5 -> line
- U1 pad 17: gnd-1 -> gnd
- U1 pad 18: line-6 -> line-2
- U1 pad 19: line-2 -> line-4
- U1 pad 21: line -> gate-1
- U1 pad 22: gnd-1 -> gnd
- U1 pad 27: line-3 -> line-6
- U1 pad 29: line-1 -> line-3
- U1 pad 30: line-4 -> line-5
- U1 pad 32: hv -> hv-3
- U1 pad 33: hv-2 -> hv-1
- U1 pad 37: gnd-1 -> gnd
- U1 pad 4: gnd-4 -> gnd-1
- U1 pad 5: gnd -> gnd-3
- U1 pad 6: gnd-2 -> gnd-4
- U1 pad 7: gnd-1 -> gnd
- U10 pad 2: gnd-1 -> gnd
- U11 pad 1: hv-3 -> hv
- U11 pad 2: gnd-1 -> gnd
- U12 pad 1: hv-3 -> hv
- U12 pad 2: gnd-1 -> gnd
- U13 pad 1: hv-3 -> hv
- U13 pad 2: gnd-1 -> gnd
- U14 pad 1: hv-3 -> hv
- U14 pad 2: gnd-1 -> gnd
- U15 pad 1: hv-3 -> hv
- U15 pad 2: gnd-1 -> gnd
- U16 pad 1: hv-3 -> hv
- U16 pad 2: gnd-1 -> gnd
- U17 pad 1: hv-3 -> hv
- U17 pad 2: gnd-1 -> gnd
- U18 pad 1: hv-3 -> hv
- U18 pad 2: gnd-1 -> gnd
- U19 pad 1: hv-3 -> hv
- U19 pad 2: gnd-1 -> gnd
- U20 pad 1: hv-3 -> hv
- U20 pad 2: gnd-1 -> gnd
- U21 pad 1: line-4 -> line-5
- U21 pad 2: line-1 -> line-3
- U22 pad 1: line-1 -> line-3
- U22 pad 2: gnd-1 -> gnd
- U23 pad 1: hv-3 -> hv
- U23 pad 2: line-1 -> line-3
- U24 pad 1: line-4 -> line-5
- U24 pad 2: gnd-1 -> gnd
- U25 pad 1: hv -> hv-3
- U25 pad 2: line-4 -> line-5
- U26 pad 1: hv -> hv-3
- U26 pad 2: hv-3 -> hv
- U27 pad 1: hv-1 -> hv-2
- U27 pad 2: gnd-1 -> gnd
- U28 pad 1: hv-1 -> hv-2
- U28 pad 2: gnd-1 -> gnd
- U29 pad 1: hv-1 -> hv-2
- U29 pad 2: gnd-1 -> gnd
- U3 pad 1: line-6 -> line-2
- U30 pad 1: hv-1 -> hv-2
- U30 pad 2: gnd-1 -> gnd
- U31 pad 1: hv-1 -> hv-2
- U31 pad 2: gnd-1 -> gnd
- U32 pad 1: hv-1 -> hv-2
- U32 pad 2: gnd-1 -> gnd
- U33 pad 1: hv-1 -> hv-2
- U33 pad 2: gnd-1 -> gnd
- U34 pad 1: hv-1 -> hv-2
- U34 pad 2: gnd-1 -> gnd
- U35 pad 1: hv-1 -> hv-2
- U35 pad 2: gnd-1 -> gnd
- U36 pad 1: hv-1 -> hv-2
- U36 pad 2: gnd-1 -> gnd
- U37 pad 1: line-5 -> line
- U37 pad 2: line-7 -> line-1
- U38 pad 1: line-7 -> line-1
- U38 pad 2: gnd-1 -> gnd
- U39 pad 1: hv-2 -> hv-1
- U39 pad 2: line-7 -> line-1
- U4 pad 2: gnd-1 -> gnd
- U40 pad 1: line-5 -> line
- U40 pad 2: gnd-1 -> gnd
- U41 pad 1: hv-1 -> hv-2
- U41 pad 2: line-5 -> line
- U42 pad 1: hv-1 -> hv-2
- U42 pad 2: hv-2 -> hv-1
- U44 pad 1: hv-2 -> hv-1
- U45 pad 1: hv -> hv-3
- U47 pad 2: gnd-1 -> gnd
- U48 pad 2: gnd-1 -> gnd
- U49 pad 1: hv -> hv-3
- U49 pad 2: gnd-1 -> gnd
- U50 pad 1: hv -> hv-3
- U50 pad 2: gnd-1 -> gnd
- U51 pad 1: hv-3 -> hv
- U51 pad 2: gnd-1 -> gnd
- U52 pad 1: hv-1 -> hv-2
- U52 pad 2: gnd-1 -> gnd
- U54 pad 2: gnd-1 -> gnd
- U57 pad 2: gnd-1 -> gnd
- U58 pad 2: gnd-1 -> gnd
- U8 pad 2: line-6 -> line-2
- U9 pad 2: gnd-1 -> gnd
Routing:
- net line-7: track 86.4 -> 0.00 mm, vias 2 -> 0
- net line-5: track 88.9 -> 10.1 mm
- net hv-2: track 78.8 -> 1.69 mm, vias 7 -> 34
- net hv-1: track 1.69 -> 78.8 mm, vias 34 -> 7
- net line-1: track 10.5 -> 86.4 mm
- net gate-1: track 0.00 -> 67.3 mm, vias 0 -> 2
- net gnd-3: track 81.7 -> 15.6 mm
- net gnd-2: track 17.4 -> 81.7 mm
- net line-4: track 10.1 -> 59.3 mm
- net line-6: track 68.3 -> 37.8 mm
- net line-3: track 37.8 -> 10.5 mm
- net hv-3: track 1.67 -> 27.9 mm, vias 33 -> 8
- net hv: track 27.9 -> 1.67 mm, vias 8 -> 33
- net line: track 67.3 -> 88.9 mm
- net gnd-1: track 24.6 -> 12.5 mm, vias 90 -> 2
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- added copper zone on B.Cu, net gnd
- added copper zone on F.Cu, net gnd
- added copper zone on In1.Cu, net gnd
- added copper zone on In2.Cu, net hv
- added copper zone on In2.Cu, net hv-2
- added copper zone on F.Cu, net line-2
- removed copper zone on B.Cu, net gnd-1
- removed copper zone on F.Cu, net gnd-1
- removed copper zone on In1.Cu, net gnd-1
- removed copper zone on In2.Cu, net hv-1
- removed copper zone on In2.Cu, net hv-3
- removed copper zone on F.Cu, net line-6

Commit message: building frozen
Connections:
- net drain renamed source
- net line renamed SRP
- net line-1 renamed SRN
- net line-2 renamed source-1
- net line-3 renamed ACN
- net line-5 renamed ACP
- net line-6 renamed gate-2
- C1 pad 2: gnd -> gnd-1
- C2 pad 1: hv-2 -> hv-3
- C2 pad 2: gnd -> gnd-1
- C3 pad 1: hv-3 -> hv-1
- C3 pad 2: gnd -> gnd-1
- C4 pad 1: hv-1 -> hv-2
- C4 pad 2: gnd -> gnd-1
- DS1 pad 1: cathode-1 -> cathode
- DS2 pad 1: cathode -> cathode-1
- Q2 pad 1: gnd -> gnd-1
- Q2 pad 2: gnd -> gnd-1
- Q2 pad 3: gnd -> gnd-1
- Q2 pad 4: gate -> gate-1
- Q3 pad 4: line-4 -> gate
- Q3 pad 5: hv-2 -> hv-3
- Q3 pad 6: hv-2 -> hv-3
- Q3 pad 7: hv-2 -> hv-3
- Q3 pad 8: hv-2 -> hv-3
- Q4 pad 1: gnd -> gnd-1
- Q4 pad 2: gnd -> gnd-1
- Q4 pad 3: gnd -> gnd-1
- Q4 pad 4: gate-1 -> gate-3
- R1 pad 2: gnd-4 -> gnd-2
- R2 pad 2: gnd-1 -> gnd
- U1 pad 11: gnd-2 -> gnd-4
- U1 pad 17: gnd -> gnd-1
- U1 pad 19: line-4 -> gate
- U1 pad 20: cathode -> cathode-1
- U1 pad 21: gate-1 -> gate-3
- U1 pad 22: gnd -> gnd-1
- U1 pad 25: gate -> gate-1
- U1 pad 26: cathode-1 -> cathode
- U1 pad 32: hv-3 -> hv-1
- U1 pad 33: hv-1 -> hv-2
- U1 pad 37: gnd -> gnd-1
- U1 pad 4: gnd-1 -> gnd
- U1 pad 6: gnd-4 -> gnd-2
- U1 pad 7: gnd -> gnd-1
- U10 pad 2: gnd -> gnd-1
- U11 pad 2: gnd -> gnd-1
- U12 pad 2: gnd -> gnd-1
- U13 pad 2: gnd -> gnd-1
- U14 pad 2: gnd -> gnd-1
- U15 pad 2: gnd -> gnd-1
- U16 pad 2: gnd -> gnd-1
- U17 pad 2: gnd -> gnd-1
- U18 pad 2: gnd -> gnd-1
- U19 pad 2: gnd -> gnd-1
- U2 pad 2: cathode-1 -> cathode
- U20 pad 2: gnd -> gnd-1
- U22 pad 2: gnd -> gnd-1
- U24 pad 2: gnd -> gnd-1
- U25 pad 1: hv-3 -> hv-1
- U26 pad 1: hv-3 -> hv-1
- U27 pad 1: hv-2 -> hv-3
- U27 pad 2: gnd -> gnd-1
- U28 pad 1: hv-2 -> hv-3
- U28 pad 2: gnd -> gnd-1
- U29 pad 1: hv-2 -> hv-3
- U29 pad 2: gnd -> gnd-1
- U3 pad 2: cathode -> cathode-1
- U30 pad 1: hv-2 -> hv-3
- U30 pad 2: gnd -> gnd-1
- U31 pad 1: hv-2 -> hv-3
- U31 pad 2: gnd -> gnd-1
- U32 pad 1: hv-2 -> hv-3
- U32 pad 2: gnd -> gnd-1
- U33 pad 1: hv-2 -> hv-3
- U33 pad 2: gnd -> gnd-1
- U34 pad 1: hv-2 -> hv-3
- U34 pad 2: gnd -> gnd-1
- U35 pad 1: hv-2 -> hv-3
- U35 pad 2: gnd -> gnd-1
- U36 pad 1: hv-2 -> hv-3
- U36 pad 2: gnd -> gnd-1
- U38 pad 2: gnd -> gnd-1
- U39 pad 1: hv-1 -> hv-2
- U4 pad 2: gnd -> gnd-1
- U40 pad 2: gnd -> gnd-1
- U41 pad 1: hv-2 -> hv-3
- U42 pad 1: hv-2 -> hv-3
- U42 pad 2: hv-1 -> hv-2
- U44 pad 1: hv-1 -> hv-2
- U45 pad 1: hv-3 -> hv-1
- U47 pad 2: gnd -> gnd-1
- U48 pad 2: gnd -> gnd-1
- U49 pad 1: hv-3 -> hv-1
- U49 pad 2: gnd -> gnd-1
- U50 pad 1: hv-3 -> hv-1
- U50 pad 2: gnd -> gnd-1
- U51 pad 2: gnd -> gnd-1
- U52 pad 1: hv-2 -> hv-3
- U52 pad 2: gnd -> gnd-1
- U54 pad 2: gnd -> gnd-1
- U57 pad 2: gnd -> gnd-1
- U58 pad 2: gnd -> gnd-1
- U9 pad 2: gnd -> gnd-1
Routing:
- net hv-2: track 1.69 -> 78.8 mm, vias 34 -> 7
- net gate-3: track 0.00 -> 67.3 mm, vias 0 -> 2
- net gnd-4: track 17.4 -> 81.7 mm
- net gnd-2: track 81.7 -> 17.4 mm
- net line-4: track 59.3 -> 0.00 mm, vias 2 -> 0
- net hv-1: track 78.8 -> 27.9 mm, vias 7 -> 8
- net gate-1: track 67.3 -> 38.0 mm
- net hv-3: track 27.9 -> 1.69 mm, vias 8 -> 34
- net gate: track 38.0 -> 59.3 mm
- net gnd-1: track 12.5 -> 24.6 mm, vias 2 -> 90
- net gnd: track 24.6 -> 12.5 mm, vias 90 -> 2
- net cathode-1: track 59.5 -> 62.4 mm
- net cathode: track 62.4 -> 59.5 mm
- added copper zone on B.Cu, net gnd-1
- added copper zone on F.Cu, net gnd-1
- added copper zone on In1.Cu, net gnd-1
- added copper zone on In2.Cu, net hv-3
- removed copper zone on B.Cu, net gnd
- removed copper zone on F.Cu, net gnd
- removed copper zone on In1.Cu, net gnd
- removed copper zone on In2.Cu, net hv-2

Commit message: update buck-boost
Parts:
- U4: value 50kΩ ±1% 62.5mW -> 49.9kΩ ±0% 62.5mW
- U44: value 249kΩ ±1% 100mW -> 249kΩ ±1% 62.5mW; footprint atopile:R0603-ebcab9 -> atopile:R0402-56259e
- U47: value 25.5kΩ ±0% 100mW -> 25.5kΩ ±1% 100mW
- U50: value 1µF ±10% 250V X7R -> 1µF ±10% 100V X7S; footprint atopile:C1812-bfe9b0 -> atopile:C0805-3b2e55
- U59: value 5.23kΩ ±1% 100mW -> 5.23kΩ ±1% 62.5mW; footprint atopile:R0603-ebcab9 -> atopile:R0402-56259e
Connections:
- C1 pad 1: hv -> hv-2
- C1 pad 2: gnd-1 -> gnd-3
- C2 pad 1: hv-3 -> hv-1
- C2 pad 2: gnd-1 -> gnd-3
- C3 pad 1: hv-1 -> hv-3
- C3 pad 2: gnd-1 -> gnd-3
- C4 pad 1: hv-2 -> hv
- C4 pad 2: gnd-1 -> gnd-3
- DS1 pad 1: cathode -> cathode-1
- DS2 pad 1: cathode-1 -> cathode
- Q1 pad 4: gate-2 -> gate-1
- Q1 pad 5: hv -> hv-2
- Q1 pad 6: hv -> hv-2
- Q1 pad 7: hv -> hv-2
- Q1 pad 8: hv -> hv-2
- Q2 pad 1: gnd-1 -> gnd-3
- Q2 pad 2: gnd-1 -> gnd-3
- Q2 pad 3: gnd-1 -> gnd-3
- Q2 pad 4: gate-1 -> gate
- Q3 pad 4: gate -> gate-3
- Q3 pad 5: hv-3 -> hv-1
- Q3 pad 6: hv-3 -> hv-1
- Q3 pad 7: hv-3 -> hv-1
- Q3 pad 8: hv-3 -> hv-1
- Q4 pad 1: gnd-1 -> gnd-3
- Q4 pad 2: gnd-1 -> gnd-3
- Q4 pad 3: gnd-1 -> gnd-3
- Q4 pad 4: gate-3 -> gate-2
- R3 pad 2: gnd-3 -> gnd-1
- U1 pad 17: gnd-1 -> gnd-3
- U1 pad 19: gate -> gate-3
- U1 pad 20: cathode-1 -> cathode
- U1 pad 21: gate-3 -> gate-2
- U1 pad 22: gnd-1 -> gnd-3
- U1 pad 25: gate-1 -> gate
- U1 pad 26: cathode -> cathode-1
- U1 pad 27: gate-2 -> gate-1
- U1 pad 32: hv-1 -> hv-3
- U1 pad 33: hv-2 -> hv
- U1 pad 37: gnd-1 -> gnd-3
- U1 pad 5: gnd-3 -> gnd-1
- U1 pad 7: gnd-1 -> gnd-3
- U10 pad 2: gnd-1 -> gnd-3
- U11 pad 1: hv -> hv-2
- U11 pad 2: gnd-1 -> gnd-3
- U12 pad 1: hv -> hv-2
- U12 pad 2: gnd-1 -> gnd-3
- U13 pad 1: hv -> hv-2
- U13 pad 2: gnd-1 -> gnd-3
- U14 pad 1: hv -> hv-2
- U14 pad 2: gnd-1 -> gnd-3
- U15 pad 1: hv -> hv-2
- U15 pad 2: gnd-1 -> gnd-3
- U16 pad 1: hv -> hv-2
- U16 pad 2: gnd-1 -> gnd-3
- U17 pad 1: hv -> hv-2
- U17 pad 2: gnd-1 -> gnd-3
- U18 pad 1: hv -> hv-2
- U18 pad 2: gnd-1 -> gnd-3
- U19 pad 1: hv -> hv-2
- U19 pad 2: gnd-1 -> gnd-3
- U2 pad 2: cathode -> cathode-1
- U20 pad 1: hv -> hv-2
- U20 pad 2: gnd-1 -> gnd-3
- U22 pad 2: gnd-1 -> gnd-3
- U23 pad 1: hv -> hv-2
- U24 pad 2: gnd-1 -> gnd-3
- U25 pad 1: hv-1 -> hv-3
- U26 pad 1: hv-1 -> hv-3
- U26 pad 2: hv -> hv-2
- U27 pad 1: hv-3 -> hv-1
- U27 pad 2: gnd-1 -> gnd-3
- U28 pad 1: hv-3 -> hv-1
- U28 pad 2: gnd-1 -> gnd-3
- U29 pad 1: hv-3 -> hv-1
- U29 pad 2: gnd-1 -> gnd-3
- U3 pad 2: cathode-1 -> cathode
- U30 pad 1: hv-3 -> hv-1
- U30 pad 2: gnd-1 -> gnd-3
- U31 pad 1: hv-3 -> hv-1
- U31 pad 2: gnd-1 -> gnd-3
- U32 pad 1: hv-3 -> hv-1
- U32 pad 2: gnd-1 -> gnd-3
- U33 pad 1: hv-3 -> hv-1
- U33 pad 2: gnd-1 -> gnd-3
- U34 pad 1: hv-3 -> hv-1
- U34 pad 2: gnd-1 -> gnd-3
- U35 pad 1: hv-3 -> hv-1
- U35 pad 2: gnd-1 -> gnd-3
- U36 pad 1: hv-3 -> hv-1
- U36 pad 2: gnd-1 -> gnd-3
- U38 pad 2: gnd-1 -> gnd-3
- U39 pad 1: hv-2 -> hv
- U4 pad 2: gnd-1 -> gnd-3
- U40 pad 2: gnd-1 -> gnd-3
- U41 pad 1: hv-3 -> hv-1
- U42 pad 1: hv-3 -> hv-1
- U42 pad 2: hv-2 -> hv
- U43 pad 2: output_v_sense-gnd -> gnd-4
- U44 pad 1: hv-2 -> hv
- U45 pad 1: hv-1 -> hv-3
- U47 pad 2: gnd-1 -> gnd-3
- U48 pad 2: gnd-1 -> gnd-3
- U49 pad 1: hv-1 -> hv-3
- U49 pad 2: gnd-1 -> gnd-3
- U50 pad 1: hv-1 -> hv-3
- U50 pad 2: gnd-1 -> gnd-3
- U51 pad 1: hv -> hv-2
- U51 pad 2: gnd-1 -> gnd-3
- U52 pad 1: hv-3 -> hv-1
- U52 pad 2: gnd-1 -> gnd-3
- U54 pad 2: gnd-1 -> gnd-3
- U57 pad 2: gnd-1 -> gnd-3
- U58 pad 2: gnd-1 -> gnd-3
- U9 pad 2: gnd-1 -> gnd-3
Routing:
- net hv: track 1.67 -> 83.3 mm, vias 33 -> 7
- net hv-2: track 78.8 -> 1.67 mm, vias 7 -> 33
- net gate-2: track 37.8 -> 67.3 mm
- net hv-3: track 1.69 -> 27.9 mm, vias 34 -> 8
- net hv-1: track 27.9 -> 1.69 mm, vias 8 -> 34
- net gate: track 59.3 -> 38.0 mm
- net gnd-3: track 15.6 -> 24.6 mm, vias 2 -> 90
- net gnd-1: track 24.6 -> 15.6 mm, vias 90 -> 2
- net gate-3: track 67.3 -> 59.3 mm
- net cathode-1: track 62.4 -> 59.5 mm
- net cathode: track 59.5 -> 62.4 mm
- net gnd-4: track 81.7 -> 82.3 mm
- added copper zone on B.Cu, net gnd-3
- added copper zone on F.Cu, net gnd-3
- added copper zone on In1.Cu, net gnd-3
- added copper zone on In2.Cu, net hv-1
- added copper zone on In2.Cu, net hv-2
- removed copper zone on B.Cu, net gnd-1
- removed copper zone on F.Cu, net gnd-1
- removed copper zone on In1.Cu, net gnd-1
- removed copper zone on In2.Cu, net hv
- removed copper zone on In2.Cu, net hv-3

Commit message: Build everything with ordered params to fix frozen builds
Connections:
- C1 pad 1: hv-2 -> hv
- C1 pad 2: gnd-3 -> gnd
- C2 pad 2: gnd-3 -> gnd
- C3 pad 2: gnd-3 -> gnd
- C4 pad 1: hv -> hv-2
- C4 pad 2: gnd-3 -> gnd
- Q1 pad 1: source -> drain
- Q1 pad 2: source -> drain
- Q1 pad 3: source -> drain
- Q1 pad 4: gate-1 -> gate-3
- Q1 pad 5: hv-2 -> hv
- Q1 pad 6: hv-2 -> hv
- Q1 pad 7: hv-2 -> hv
- Q1 pad 8: hv-2 -> hv
- Q2 pad 1: gnd-3 -> gnd
- Q2 pad 2: gnd-3 -> gnd
- Q2 pad 3: gnd-3 -> gnd
- Q2 pad 4: gate -> gate-2
- Q2 pad 5: source -> drain
- Q2 pad 6: source -> drain
- Q2 pad 7: source -> drain
- Q2 pad 8: source -> drain
- Q3 pad 1: source-1 -> source
- Q3 pad 2: source-1 -> source
- Q3 pad 3: source-1 -> source
- Q3 pad 4: gate-3 -> gate
- Q4 pad 1: gnd-3 -> gnd
- Q4 pad 2: gnd-3 -> gnd
- Q4 pad 3: gnd-3 -> gnd
- Q4 pad 4: gate-2 -> gate-1
- Q4 pad 5: source-1 -> source
- Q4 pad 6: source-1 -> source
- Q4 pad 7: source-1 -> source
- Q4 pad 8: source-1 -> source
- R1 pad 2: gnd-2 -> gnd-4
- R2 pad 2: gnd -> gnd-3
- U1 pad 11: gnd-4 -> gnd-2
- U1 pad 17: gnd-3 -> gnd
- U1 pad 18: source-1 -> source
- U1 pad 19: gate-3 -> gate
- U1 pad 21: gate-2 -> gate-1
- U1 pad 22: gnd-3 -> gnd
- U1 pad 25: gate -> gate-2
- U1 pad 27: gate-1 -> gate-3
- U1 pad 28: source -> drain
- U1 pad 33: hv -> hv-2
- U1 pad 37: gnd-3 -> gnd
- U1 pad 4: gnd -> gnd-3
- U1 pad 6: gnd-2 -> gnd-4
- U1 pad 7: gnd-3 -> gnd
- U10 pad 2: gnd-3 -> gnd
- U11 pad 1: hv-2 -> hv
- U11 pad 2: gnd-3 -> gnd
- U12 pad 1: hv-2 -> hv
- U12 pad 2: gnd-3 -> gnd
- U13 pad 1: hv-2 -> hv
- U13 pad 2: gnd-3 -> gnd
- U14 pad 1: hv-2 -> hv
- U14 pad 2: gnd-3 -> gnd
- U15 pad 1: hv-2 -> hv
- U15 pad 2: gnd-3 -> gnd
- U16 pad 1: hv-2 -> hv
- U16 pad 2: gnd-3 -> gnd
- U17 pad 1: hv-2 -> hv
- U17 pad 2: gnd-3 -> gnd
- U18 pad 1: hv-2 -> hv
- U18 pad 2: gnd-3 -> gnd
- U19 pad 1: hv-2 -> hv
- U19 pad 2: gnd-3 -> gnd
- U2 pad 1: source -> drain
- U20 pad 1: hv-2 -> hv
- U20 pad 2: gnd-3 -> gnd
- U22 pad 2: gnd-3 -> gnd
- U23 pad 1: hv-2 -> hv
- U24 pad 2: gnd-3 -> gnd
- U26 pad 2: hv-2 -> hv
- U27 pad 2: gnd-3 -> gnd
- U28 pad 2: gnd-3 -> gnd
- U29 pad 2: gnd-3 -> gnd
- U3 pad 1: source-1 -> source
- U30 pad 2: gnd-3 -> gnd
- U31 pad 2: gnd-3 -> gnd
- U32 pad 2: gnd-3 -> gnd
- U33 pad 2: gnd-3 -> gnd
- U34 pad 2: gnd-3 -> gnd
- U35 pad 2: gnd-3 -> gnd
- U36 pad 2: gnd-3 -> gnd
- U38 pad 2: gnd-3 -> gnd
- U39 pad 1: hv -> hv-2
- U4 pad 2: gnd-3 -> gnd
- U40 pad 2: gnd-3 -> gnd
- U42 pad 2: hv -> hv-2
- U43 pad 2: gnd-4 -> gnd-2
- U44 pad 1: hv -> hv-2
- U47 pad 2: gnd-3 -> gnd
- U48 pad 2: gnd-3 -> gnd
- U49 pad 2: gnd-3 -> gnd
- U50 pad 2: gnd-3 -> gnd
- U51 pad 1: hv-2 -> hv
- U51 pad 2: gnd-3 -> gnd
- U52 pad 2: gnd-3 -> gnd
- U54 pad 2: gnd-3 -> gnd
- U57 pad 2: gnd-3 -> gnd
- U58 pad 2: gnd-3 -> gnd
- U8 pad 1: source -> drain
- U8 pad 2: source-1 -> source
- U9 pad 2: gnd-3 -> gnd
Routing:
- net hv-2: track 1.67 -> 83.3 mm, vias 33 -> 7
- net hv: track 83.3 -> 1.67 mm, vias 7 -> 33
- net source-1: track 68.3 -> 0.00 mm, vias 2 -> 0
- net gnd-4: track 82.3 -> 17.4 mm
- net gnd-2: track 17.4 -> 82.3 mm
- net drain: track 0.00 -> 55.2 mm, vias 0 -> 3
- net gate-1: track 37.8 -> 67.3 mm
- net gate-2: track 67.3 -> 38.0 mm
- net gate-3: track 59.3 -> 37.8 mm
- net gate: track 38.0 -> 59.3 mm
- net source: track 55.2 -> 68.3 mm, vias 3 -> 2
- net gnd-3: track 24.6 -> 12.5 mm, vias 90 -> 2
- net gnd: track 12.5 -> 24.6 mm, vias 2 -> 90
- added copper zone on F.Cu, net drain
- added copper zone on B.Cu, net gnd
- added copper zone on F.Cu, net gnd
- added copper zone on In1.Cu, net gnd
- added copper zone on In2.Cu, net hv
- removed copper zone on B.Cu, net gnd-3
- removed copper zone on F.Cu, net gnd-3
- removed copper zone on In1.Cu, net gnd-3
- removed copper zone on In2.Cu, net hv-2
- removed copper zone on F.Cu, net source-1

Commit message: Cleanup layout for usb hub and usb-uart, add CM5 controller heatsink outline
Connections:
- C1 pad 1: hv -> hv-2
- C2 pad 1: hv-1 -> hv
- C3 pad 1: hv-3 -> hv-1
- C4 pad 1: hv-2 -> hv-3
- Q1 pad 5: hv -> hv-2
- Q1 pad 6: hv -> hv-2
- Q1 pad 7: hv -> hv-2
- Q1 pad 8: hv -> hv-2
- Q2 pad 4: gate-2 -> gate-1
- Q3 pad 5: hv-1 -> hv
- Q3 pad 6: hv-1 -> hv
- Q3 pad 7: hv-1 -> hv
- Q3 pad 8: hv-1 -> hv
- Q4 pad 4: gate-1 -> gate-2
- R1 pad 2: gnd-4 -> gnd-1
- R2 pad 2: gnd-3 -> gnd-4
- R3 pad 2: gnd-1 -> gnd-2
- U1 pad 11: gnd-2 -> gnd-3
- U1 pad 21: gate-1 -> gate-2
- U1 pad 25: gate-2 -> gate-1
- U1 pad 32: hv-3 -> hv-1
- U1 pad 33: hv-2 -> hv-3
- U1 pad 4: gnd-3 -> gnd-4
- U1 pad 5: gnd-1 -> gnd-2
- U1 pad 6: gnd-4 -> gnd-1
- U11 pad 1: hv -> hv-2
- U12 pad 1: hv -> hv-2
- U13 pad 1: hv -> hv-2
- U14 pad 1: hv -> hv-2
- U15 pad 1: hv -> hv-2
- U16 pad 1: hv -> hv-2
- U17 pad 1: hv -> hv-2
- U18 pad 1: hv -> hv-2
- U19 pad 1: hv -> hv-2
- U20 pad 1: hv -> hv-2
- U23 pad 1: hv -> hv-2
- U25 pad 1: hv-3 -> hv-1
- U26 pad 1: hv-3 -> hv-1
- U26 pad 2: hv -> hv-2
- U27 pad 1: hv-1 -> hv
- U28 pad 1: hv-1 -> hv
- U29 pad 1: hv-1 -> hv
- U30 pad 1: hv-1 -> hv
- U31 pad 1: hv-1 -> hv
- U32 pad 1: hv-1 -> hv
- U33 pad 1: hv-1 -> hv
- U34 pad 1: hv-1 -> hv
- U35 pad 1: hv-1 -> hv
- U36 pad 1: hv-1 -> hv
- U39 pad 1: hv-2 -> hv-3
- U41 pad 1: hv-1 -> hv
- U42 pad 1: hv-1 -> hv
- U42 pad 2: hv-2 -> hv-3
- U43 pad 2: gnd-2 -> gnd-3
- U44 pad 1: hv-2 -> hv-3
- U45 pad 1: hv-3 -> hv-1
- U49 pad 1: hv-3 -> hv-1
- U50 pad 1: hv-3 -> hv-1
- U51 pad 1: hv -> hv-2
- U52 pad 1: hv-1 -> hv
Routing:
- net hv-2: track 83.3 -> 1.67 mm, vias 7 -> 33
- net gnd-3: track 12.5 -> 82.3 mm
- net gnd-2: track 82.3 -> 15.6 mm
- net hv-3: track 27.9 -> 83.3 mm, vias 8 -> 7
- net gate-2: track 38.0 -> 67.3 mm
- net gate-1: track 67.3 -> 38.0 mm
- net hv-1: track 1.69 -> 27.9 mm, vias 34 -> 8
- net gnd-4: track 17.4 -> 12.5 mm
- net gnd-1: track 15.6 -> 17.4 mm
- net hv: track 1.67 -> 1.69 mm, vias 33 -> 34
- added copper zone on In2.Cu, net hv-2
- removed copper zone on In2.Cu, net hv-1

Commit message: checkin
Connections:
- net drain renamed source-1
- C1 pad 2: gnd -> gnd-3
- C2 pad 1: hv -> hv-3
- C2 pad 2: gnd -> gnd-3
- C3 pad 2: gnd -> gnd-3
- C4 pad 1: hv-3 -> hv
- C4 pad 2: gnd -> gnd-3
- Q2 pad 1: gnd -> gnd-3
- Q2 pad 2: gnd -> gnd-3
- Q2 pad 3: gnd -> gnd-3
- Q2 pad 4: gate-1 -> gate-2
- Q3 pad 5: hv -> hv-3
- Q3 pad 6: hv -> hv-3
- Q3 pad 7: hv -> hv-3
- Q3 pad 8: hv -> hv-3
- Q4 pad 1: gnd -> gnd-3
- Q4 pad 2: gnd -> gnd-3
- Q4 pad 3: gnd -> gnd-3
- Q4 pad 4: gate-2 -> gate-1
- R1 pad 2: gnd-1 -> gnd-2
- R2 pad 2: gnd-4 -> gnd
- R3 pad 2: gnd-2 -> gnd-4
- U1 pad 11: gnd-3 -> gnd-1
- U1 pad 17: gnd -> gnd-3
- U1 pad 21: gate-2 -> gate-1
- U1 pad 22: gnd -> gnd-3
- U1 pad 25: gate-1 -> gate-2
- U1 pad 33: hv-3 -> hv
- U1 pad 37: gnd -> gnd-3
- U1 pad 4: gnd-4 -> gnd
- U1 pad 5: gnd-2 -> gnd-4
- U1 pad 6: gnd-1 -> gnd-2
- U1 pad 7: gnd -> gnd-3
- U10 pad 2: gnd -> gnd-3
- U11 pad 2: gnd -> gnd-3
- U12 pad 2: gnd -> gnd-3
- U13 pad 2: gnd -> gnd-3
- U14 pad 2: gnd -> gnd-3
- U15 pad 2: gnd -> gnd-3
- U16 pad 2: gnd -> gnd-3
- U17 pad 2: gnd -> gnd-3
- U18 pad 2: gnd -> gnd-3
- U19 pad 2: gnd -> gnd-3
- U20 pad 2: gnd -> gnd-3
- U22 pad 2: gnd -> gnd-3
- U24 pad 2: gnd -> gnd-3
- U27 pad 1: hv -> hv-3
- U27 pad 2: gnd -> gnd-3
- U28 pad 1: hv -> hv-3
- U28 pad 2: gnd -> gnd-3
- U29 pad 1: hv -> hv-3
- U29 pad 2: gnd -> gnd-3
- U30 pad 1: hv -> hv-3
- U30 pad 2: gnd -> gnd-3
- U31 pad 1: hv -> hv-3
- U31 pad 2: gnd -> gnd-3
- U32 pad 1: hv -> hv-3
- U32 pad 2: gnd -> gnd-3
- U33 pad 1: hv -> hv-3
- U33 pad 2: gnd -> gnd-3
- U34 pad 1: hv -> hv-3
- U34 pad 2: gnd -> gnd-3
- U35 pad 1: hv -> hv-3
- U35 pad 2: gnd -> gnd-3
- U36 pad 1: hv -> hv-3
- U36 pad 2: gnd -> gnd-3
- U38 pad 2: gnd -> gnd-3
- U39 pad 1: hv-3 -> hv
- U4 pad 2: gnd -> gnd-3
- U40 pad 2: gnd -> gnd-3
- U41 pad 1: hv -> hv-3
- U42 pad 1: hv -> hv-3
- U42 pad 2: hv-3 -> hv
- U43 pad 2: gnd-3 -> gnd-1
- U44 pad 1: hv-3 -> hv
- U47 pad 2: gnd -> gnd-3
- U48 pad 2: gnd -> gnd-3
- U49 pad 2: gnd -> gnd-3
- U50 pad 2: gnd -> gnd-3
- U51 pad 2: gnd -> gnd-3
- U52 pad 1: hv -> hv-3
- U52 pad 2: gnd -> gnd-3
- U54 pad 2: gnd -> gnd-3
- U57 pad 2: gnd -> gnd-3
- U58 pad 2: gnd -> gnd-3
- U9 pad 2: gnd -> gnd-3
Routing:
- net hv-3: track 83.3 -> 1.69 mm, vias 7 -> 34
- net hv: track 1.69 -> 83.3 mm, vias 34 -> 7
- net gnd-1: track 17.4 -> 82.3 mm
- net gnd-3: track 82.3 -> 24.6 mm, vias 2 -> 90
- net gate-2: track 67.3 -> 38.0 mm
- net gate-1: track 38.0 -> 67.3 mm
- net gnd: track 24.6 -> 12.5 mm, vias 90 -> 2
- net gnd-4: track 12.5 -> 15.6 mm
- net gnd-2: track 15.6 -> 17.4 mm
- added copper zone on B.Cu, net gnd-3
- added copper zone on F.Cu, net gnd-3
- added copper zone on In1.Cu, net gnd-3
- added copper zone on In2.Cu, net hv-3
- removed copper zone on B.Cu, net gnd
- removed copper zone on F.Cu, net gnd
- removed copper zone on In1.Cu, net gnd
- removed copper zone on In2.Cu, net hv
