File: elec/layout/buck-boost/buck-boost.kicad_pcb (KiCad board)
At the start: 6 copper layers, 69 parts, among them U10 2.49kΩ ±1% 62.5mW, U11 4.7µF ±10% 100V X7R, U12 4.7µF ±10% 100V X7R, U13 4.7µF ±10% 100V X7R, U14 10µF ±10% 100V X7R, U15 10µF ±10% 100V X7R, U16 10µF ±10% 100V X7R, U17 10µF ±10% 100V X7R, U18 1µF ±10% 100V X7R, U19 100nF ±10% 100V X7R, U2 100nF ±10% 50V X7R, U20 100pF ±5% 100V C0G, U21 470nF ±20% 16V X5R, U22 100nF ±10% 16V X7R, U23 10Ω ±1% 62.5mW, U24 100nF ±10% 16V X7R, U25 10Ω ±1% 62.5mW, U26 5mΩ ±1% 1W, U27 4.7µF ±10% 100V X7R, U28 4.7µF ±10% 100V X7R, U29 4.7µF ±10% 100V X7R, U3 100nF ±10% 50V X7R, U30 10µF ±10% 100V X7R, U31 10µF ±10% 100V X7R, U32 10µF ±10% 100V X7R, U33 10µF ±10% 100V X7R, U34 1µF ±10% 100V X7R, U35 100nF ±10% 100V X7R, U36 100pF ±5% 100V C0G, U37 470nF ±20% 16V X5R, U38 100nF ±10% 16V X7R, U39 10Ω ±1% 62.5mW, U4 49.9kΩ ±0% 62.5mW, U40 100nF ±10% 16V X7R, U41 10Ω ±1% 62.5mW, U42 5mΩ ±1% 1W, U43 13.7kΩ ±1% 62.5mW, U44 249kΩ ±1% 62.5mW, U45 1MΩ ±1% 100mW, U46 133kΩ ±1% 100mW, U47 25.5kΩ ±1% 100mW, U48 4.7µF ±10% 25V X5R, U49 100nF ±10% 100V X7R, U50 1µF ±10% 100V X7S, U51 4.7µF ±10% 100V X7R, U52 4.7µF ±10% 100V X7R, U54 0Ω 62.5mW, U58 30.1kΩ ±1% 62.5mW, U59 5.23kΩ ±1% 62.5mW, U9 4.7µF ±10% 25V X5R

Commit message: build with excluded checks
Connections:
- C1 pad 2: gnd-3 -> gnd-4
- C2 pad 2: gnd-3 -> gnd-4
- C3 pad 2: gnd-3 -> gnd-4
- C4 pad 2: gnd-3 -> gnd-4
- DS1 pad 2: anode-1 -> anode
- DS2 pad 2: anode-1 -> anode
- Q1 pad 1: source-1 -> source
- Q1 pad 2: source-1 -> source
- Q1 pad 3: source-1 -> source
- Q1 pad 4: gate-3 -> gate-2
- Q2 pad 1: gnd-3 -> gnd-4
- Q2 pad 2: gnd-3 -> gnd-4
- Q2 pad 3: gnd-3 -> gnd-4
- Q2 pad 4: gate-2 -> gate-1
- Q2 pad 5: source-1 -> source
- Q2 pad 6: source-1 -> source
- Q2 pad 7: source-1 -> source
- Q2 pad 8: source-1 -> source
- Q3 pad 1: source -> source-1
- Q3 pad 2: source -> source-1
- Q3 pad 3: source -> source-1
- Q4 pad 1: gnd-3 -> gnd-4
- Q4 pad 2: gnd-3 -> gnd-4
- Q4 pad 3: gnd-3 -> gnd-4
- Q4 pad 4: gate-1 -> gate-3
- Q4 pad 5: source -> source-1
- Q4 pad 6: source -> source-1
- Q4 pad 7: source -> source-1
- Q4 pad 8: source -> source-1
- R1 pad 2: gnd-2 -> gnd-3
- R3 pad 2: gnd-4 -> gnd-2
- U1 pad 17: gnd-3 -> gnd-4
- U1 pad 18: source -> source-1
- U1 pad 21: gate-1 -> gate-3
- U1 pad 22: gnd-3 -> gnd-4
- U1 pad 23: anode-1 -> anode
- U1 pad 24: anode -> anode-1
- U1 pad 25: gate-2 -> gate-1
- U1 pad 27: gate-3 -> gate-2
- U1 pad 28: source-1 -> source
- U1 pad 37: gnd-3 -> gnd-4
- U1 pad 5: gnd-4 -> gnd-2
- U1 pad 6: gnd-2 -> gnd-3
- U1 pad 7: gnd-3 -> gnd-4
- U10 pad 2: gnd-3 -> gnd-4
- U11 pad 2: gnd-3 -> gnd-4
- U12 pad 2: gnd-3 -> gnd-4
- U13 pad 2: gnd-3 -> gnd-4
- U14 pad 2: gnd-3 -> gnd-4
- U15 pad 2: gnd-3 -> gnd-4
- U16 pad 2: gnd-3 -> gnd-4
- U17 pad 2: gnd-3 -> gnd-4
- U18 pad 2: gnd-3 -> gnd-4
- U19 pad 2: gnd-3 -> gnd-4
- U2 pad 1: source-1 -> source
- U20 pad 2: gnd-3 -> gnd-4
- U22 pad 2: gnd-3 -> gnd-4
- U24 pad 2: gnd-3 -> gnd-4
- U27 pad 2: gnd-3 -> gnd-4
- U28 pad 2: gnd-3 -> gnd-4
- U29 pad 2: gnd-3 -> gnd-4
- U3 pad 1: source -> source-1
- U30 pad 2: gnd-3 -> gnd-4
- U31 pad 2: gnd-3 -> gnd-4
- U32 pad 2: gnd-3 -> gnd-4
- U33 pad 2: gnd-3 -> gnd-4
- U34 pad 2: gnd-3 -> gnd-4
- U35 pad 2: gnd-3 -> gnd-4
- U36 pad 2: gnd-3 -> gnd-4
- U38 pad 2: gnd-3 -> gnd-4
- U4 pad 2: gnd-3 -> gnd-4
- U40 pad 2: gnd-3 -> gnd-4
- U47 pad 2: gnd-3 -> gnd-4
- U48 pad 1: anode -> anode-1
- U48 pad 2: gnd-3 -> gnd-4
- U49 pad 2: gnd-3 -> gnd-4
- U5 pad 2: anode -> anode-1
- U50 pad 2: gnd-3 -> gnd-4
- U51 pad 2: gnd-3 -> gnd-4
- U52 pad 2: gnd-3 -> gnd-4
- U54 pad 2: gnd-3 -> gnd-4
- U55 pad 2: anode -> anode-1
- U57 pad 2: gnd-3 -> gnd-4
- U58 pad 2: gnd-3 -> gnd-4
- U59 pad 1: anode -> anode-1
- U7 pad 2: anode -> anode-1
- U8 pad 1: source-1 -> source
- U8 pad 2: source -> source-1
- U9 pad 1: anode-1 -> anode
- U9 pad 2: gnd-3 -> gnd-4
Routing:
- net anode-1: track 70.3 -> 35.4 mm, vias 2 -> 3
- net anode: track 35.4 -> 70.3 mm, vias 3 -> 2
- net gate-3: track 37.8 -> 67.3 mm
- net gate-1: track 67.3 -> 38.0 mm
- net source-1: track 55.2 -> 68.3 mm, vias 3 -> 2
- net source: track 68.3 -> 55.2 mm, vias 2 -> 3
- net gnd-4: track 15.6 -> 24.6 mm, vias 2 -> 90
- net gnd-3: track 24.6 -> 17.4 mm, vias 90 -> 2
- net gnd-2: track 17.4 -> 15.6 mm
- added copper zone on B.Cu, net gnd-4
- added copper zone on F.Cu, net gnd-4
- added copper zone on In1.Cu, net gnd-4
- removed copper zone on B.Cu, net gnd-3
- removed copper zone on F.Cu, net gnd-3
- removed copper zone on In1.Cu, net gnd-3
