File: elec/layout/space-bms-hil/space-bms-hil.kicad_pcb (KiCad board)
At the start: 4 copper layers, 90 x 70 mm, 135 parts, among them U1 10nF ±10% 50V X7R, U10 12.4kΩ ±1% 62.5mW, U100 1kΩ ±1% 62.5mW, U102 1kΩ ±1% 62.5mW, U105 10kΩ ±1% 62.5mW, U106 1kΩ ±1% 62.5mW, U108 1kΩ ±1% 62.5mW, U11 1nF ±10% 50V X7R, U12 220Ω ±1% 62.5mW, U13 1MΩ ±1% 62.5mW, U15 10pF ±5% 50V C0G, U16 10pF ±5% 50V C0G, U19 10nF ±10% 50V X7R, U2 220Ω ±1% 62.5mW, U20 6.8nF ±10% 50V X7R, U21 33Ω ±1% 62.5mW, U22 49.9Ω ±1% 62.5mW, U23 6.8nF ±10% 50V X7R, U24 33Ω ±1% 62.5mW, U25 49.9Ω ±1% 62.5mW, U26 4.7µF ±10% 10V X5R, U27 22nF ±10% 50V X7R, U28 10Ω ±1% 62.5mW, U29 33Ω ±1% 62.5mW, U3 10µF ±10% 25V X5R, U30 49.9Ω ±1% 62.5mW, U31 33Ω ±1% 62.5mW, U32 49.9Ω ±1% 62.5mW, U34 10µF ±10% 25V X5R, U35 10µF ±10% 25V X5R, U37 10kΩ ±1% 62.5mW, U39 10kΩ ±1% 62.5mW, U4 100nF ±10% 16V X7R, U41 100nF ±10% 16V X7R, U42 100nF ±10% 16V X7R, U43 2.2µF ±10% 25V X5R, U45 10kΩ ±1% 62.5mW, U46 10kΩ ±1% 62.5mW, U47 10kΩ ±1% 62.5mW, U48 10kΩ ±1% 62.5mW, U49 10kΩ ±1% 62.5mW, U5 100nF ±10% 16V X7R, U50 10kΩ ±1% 62.5mW, U51 10kΩ ±1% 62.5mW, U52 10kΩ ±1% 62.5mW, U53 10kΩ ±1% 62.5mW, U54 10kΩ ±1% 62.5mW, U55 10kΩ ±1% 62.5mW, U56 10kΩ ±1% 62.5mW, U57 10kΩ ±1% 62.5mW, U58 10kΩ ±1% 62.5mW, U59 10kΩ ±1% 62.5mW, U6 100nF ±10% 16V X7R, U60 10kΩ ±1% 62.5mW, U61 10kΩ ±1% 62.5mW, U62 10kΩ ±1% 62.5mW, U63 10kΩ ±1% 62.5mW, U66 100nF ±10% 16V X7R, U67 10kΩ ±1% 62.5mW, U68 10kΩ ±1% 62.5mW, U69 10kΩ ±1% 62.5mW, U7 100nF ±10% 16V X7R, U72 100nF ±10% 16V X7R, U73 10kΩ ±1% 62.5mW, U74 10kΩ ±1% 62.5mW, U75 10kΩ ±1% 62.5mW, U78 100nF ±10% 16V X7R, U79 10kΩ ±1% 62.5mW, U8 100nF ±10% 16V X7R, U80 10kΩ ±1% 62.5mW, U81 10kΩ ±1% 62.5mW, U84 100nF ±10% 16V X7R, U85 10kΩ ±1% 62.5mW, U86 10kΩ ±1% 62.5mW, U87 18kΩ ±0% 62.5mW, U88 1µF ±10% 25V X5R, U9 100nF ±10% 16V X7R, U90 1µF ±10% 25V X5R, U91 470nF ±20% 16V X5R, U92 10kΩ ±1% 62.5mW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

Commit message: add CAN communication block and RPI CM4 block
Connections:
- net i2c_multiplexer-io renamed RESET_
- net regulator_3v3-out renamed out
- net regulator_5v-out renamed FB
- D1 pad 1: io-3 -> io
- D2 pad 1: io-2 -> io-1
- D3 pad 1: io-1 -> io-3
- D4 pad 1: io -> io-2
- DS1 pad 1: cathode-1 -> cathode-2
- R2 pad 1: line-13 -> line-8
- R3 pad 1: line-3 -> line-10
- U101 pad 1: cathode-2 -> cathode-1
- U102 pad 1: cathode-2 -> cathode-1
- U103 pad 5: hv-3 -> hv
- U103 pad 6: hv-4 -> hv-3
- U104 pad 10: sep_relay.gpio_expander-net-3 -> sep_relay.gpio_expander-net-5
- U104 pad 12: line-2 -> line-4
- U104 pad 13: line-5 -> line-1
- U104 pad 3: sep_relay.gpio_expander-net -> sep_relay.gpio_expander-net-1
- U104 pad 4: sep_relay.gpio_expander-net-1 -> sep_relay.gpio_expander-net-3
- U104 pad 5: sep_relay.gpio_expander-net-2 -> sep_relay.gpio_expander-net-4
- U104 pad 7: sep_relay.gpio_expander-net-4 -> sep_relay.gpio_expander-net
- U104 pad 8: sep_relay.gpio_expander-net-6 -> sep_relay.gpio_expander-net-2
- U104 pad 9: sep_relay.gpio_expander-net-5 -> sep_relay.gpio_expander-net-6
- U109 pad 3: sep_relay-gnd-1 -> sep_relay-gnd
- U109 pad 4: sep_relay-gnd -> sep_relay-gnd-1
- U109 pad 5: hv-1 -> hv-4
- U109 pad 6: hv -> hv-1
- U110 pad 1: hv-4 -> hv-3
- U110 pad 2: hv-3 -> hv
- U111 pad 1: hv -> hv-1
- U111 pad 2: hv-1 -> hv-4
- U112 pad 1: vsh_connector-net-10 -> vsh_connector-net-3
- U112 pad 10: vsh_connector-net-3 -> vsh_connector-net-2
- U112 pad 11: vsh_connector-net-12 -> vsh_connector-net-9
- U112 pad 12: vsh_connector-net-9 -> vsh_connector-net-6
- U112 pad 13: vsh_connector-net-6 -> vsh_connector-net-1
- U112 pad 14: vsh_connector-net-5 -> vsh_connector-net-11
- U112 pad 15: io-3 -> io
- U112 pad 17: io-2 -> io-1
- U112 pad 19: io-1 -> io-3
- U112 pad 2: vsh_connector-net-1 -> vsh_connector-net-8
- U112 pad 21: io -> io-2
- U112 pad 3: vsh_connector-net -> vsh_connector-net-5
- U112 pad 4: vsh_connector-net-4 -> vsh_connector-net
- U112 pad 5: vsh_connector-net-7 -> vsh_connector-net-10
- U112 pad 6: vsh_connector-net-11 -> vsh_connector-net-13
- U112 pad 7: vsh_connector-net-8 -> vsh_connector-net-12
- U112 pad 8: vsh_connector-net-2 -> vsh_connector-net-7
- U112 pad 9: vsh_connector-net-13 -> vsh_connector-net-4
- U17 pad 10: dep_relay.gpio_expander-net-2 -> dep_relay.gpio_expander-net-3
- U17 pad 12: line-8 -> line-3
- U17 pad 13: line-9 -> line-12
- U17 pad 3: dep_relay.gpio_expander-net-1 -> dep_relay.gpio_expander-net-4
- U17 pad 4: dep_relay.gpio_expander-net -> dep_relay.gpio_expander-net-1
- U17 pad 5: dep_relay.gpio_expander-net-4 -> dep_relay.gpio_expander-net-6
- U17 pad 7: dep_relay.gpio_expander-net-3 -> dep_relay.gpio_expander-net-2
- U17 pad 8: dep_relay.gpio_expander-net-6 -> dep_relay.gpio_expander-net
- U20 pad 1: controller.ethernet-net-1 -> controller.ethernet-net
- U21 pad 2: controller.ethernet-net-1 -> controller.ethernet-net
- U23 pad 1: controller.ethernet-net -> controller.ethernet-net-1
- U24 pad 2: controller.ethernet-net -> controller.ethernet-net-1
- U36 pad 1: in-1 -> in
- U36 pad 2: in-1 -> in
- U37 pad 2: in-1 -> in
- U38 pad 1: in -> in-1
- U38 pad 2: in -> in-1
- U39 pad 2: in -> in-1
- U40 pad 27: in-1 -> in
- U40 pad 3: in -> in-1
- U40 pad 6: line-13 -> line-8
- U40 pad 7: line-3 -> line-10
- U44 pad 11: line-12 -> line-13
- U44 pad 13: line -> line-9
- U44 pad 15: line-1 -> line-5
- U44 pad 16: line-10 -> line-6
- U44 pad 17: line-5 -> line-1
- U44 pad 18: line-2 -> line-4
- U44 pad 19: line-9 -> line-12
- U44 pad 20: line-8 -> line-3
- U44 pad 22: line-13 -> line-8
- U44 pad 23: line-3 -> line-10
- U44 pad 4: i2c_multiplexer-line-1 -> i2c_multiplexer-line
- U44 pad 5: i2c_multiplexer-line -> i2c_multiplexer-line-2
- U44 pad 6: i2c_multiplexer-line-2 -> i2c_multiplexer-line-1
- U44 pad 8: line-6 -> line
- U44 pad 9: line-4 -> line-2
- U45 pad 2: i2c_multiplexer-line -> i2c_multiplexer-line-2
- U46 pad 2: i2c_multiplexer-line-1 -> i2c_multiplexer-line
- U48 pad 2: i2c_multiplexer-line-2 -> i2c_multiplexer-line-1
- U49 pad 2: line-4 -> line-2
- U50 pad 2: line-6 -> line
- U51 pad 2: line-12 -> line-13
- U54 pad 2: line -> line-9
- U55 pad 2: line-10 -> line-6
- U56 pad 2: line-1 -> line-5
- U57 pad 2: line-2 -> line-4
- U58 pad 2: line-5 -> line-1
- U59 pad 2: line-8 -> line-3
- U60 pad 2: line-9 -> line-12
- U62 pad 2: io-3 -> io
- U64 pad 1: io-3 -> io
- U65 pad 4: line-6 -> line
- U65 pad 5: line-4 -> line-2
- U68 pad 2: io-2 -> io-1
- U70 pad 1: io-2 -> io-1
- U71 pad 5: line-12 -> line-13
- U74 pad 2: io-1 -> io-3
- U76 pad 1: io-1 -> io-3
- U76 pad 3: non_inverting-1 -> non_inverting-3
- U77 pad 4: line -> line-9
- U78 pad 1: non_inverting-1 -> non_inverting-3
- U79 pad 2: non_inverting-1 -> non_inverting-3
- U80 pad 2: io -> io-2
- U82 pad 1: io -> io-2
- U82 pad 3: non_inverting-3 -> non_inverting-1
- U83 pad 4: line-1 -> line-5
- U83 pad 5: line-10 -> line-6
- U84 pad 1: non_inverting-3 -> non_inverting-1
- U85 pad 2: non_inverting-3 -> non_inverting-1
- U91 pad 2: cathode-1 -> cathode-2
- U94 pad 6: cathode-1 -> cathode-2
- U95 pad 1: cathode-1 -> cathode-2
- U98 pad 7: line-13 -> line-8
- U98 pad 8: line-3 -> line-10
Routing:
- net line-13: track 60.8 -> 15.6 mm, vias 3 -> 0
- net line-3: track 61.0 -> 24.2 mm, vias 4 -> 2
- net line-8: track 24.2 -> 60.8 mm, vias 2 -> 3
- net line-10: track 29.1 -> 61.0 mm, vias 2 -> 4
- net in-1: track 9.92 -> 32.2 mm, vias 0 -> 2
- net in: track 32.2 -> 9.92 mm, vias 2 -> 0
- net line-4: track 12.0 -> 34.0 mm
- net line-2: track 34.0 -> 12.0 mm
- net line-6: track 12.7 -> 29.1 mm
- net io: track 22.7 -> 31.8 mm
- net io-3: track 31.8 -> 23.3 mm
- net line-12: track 15.6 -> 24.0 mm, vias 0 -> 2
- net line-9: track 24.0 -> 17.0 mm
- net line-5: track 35.1 -> 30.3 mm
- net line-1: track 30.3 -> 35.1 mm
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- added copper zone on F.Cu, net cathode-2
- removed copper zone on F.Cu, net cathode-1

Commit message: rebuild all modules
Parts:
- added U113: 1µF ±10% 25V X5R, atopile:C0402-b3ef17, F.Cu at (910.0, -5.00)
- added U114: 1µF ±10% 25V X5R, atopile:C0402-b3ef17, F.Cu at (1370.0, -5.00)
- added U115: 1µF ±10% 25V X5R, atopile:C0402-b3ef17, F.Cu at (860.0, -5.00)
- added U116: 1µF ±10% 25V X5R, atopile:C0402-b3ef17, F.Cu at (240.0, -5.00)
Connections:
- net FB renamed regulator_5v-out
- net RESET_ renamed i2c_multiplexer-io
- net SBU1 renamed A8
- net SSRXN1 renamed B10
- net out renamed regulator_3v3-out
- D1 pad 1: io -> io-1
- D2 pad 1: io-1 -> io-2
- D4 pad 1: io-2 -> io
- R2 pad 1: line-8 -> line-5
- R3 pad 1: line-10 -> line-9
- U101 pad 1: cathode-1 -> cathode
- U102 pad 1: cathode-1 -> cathode
- U103 pad 3: dep_relay-gnd -> dep_relay-gnd-1
- U103 pad 4: dep_relay-gnd-1 -> dep_relay-gnd
- U103 pad 5: hv -> hv-4
- U104 pad 12: line-4 -> line-2
- U104 pad 13: line-1 -> line
- U104 pad 3: sep_relay.gpio_expander-net-1 -> sep_relay.gpio_expander-net-3
- U104 pad 4: sep_relay.gpio_expander-net-3 -> sep_relay.gpio_expander-net-1
- U104 pad 5: sep_relay.gpio_expander-net-4 -> sep_relay.gpio_expander-net-2
- U104 pad 8: sep_relay.gpio_expander-net-2 -> sep_relay.gpio_expander-net-6
- U104 pad 9: sep_relay.gpio_expander-net-6 -> sep_relay.gpio_expander-net-4
- U107 pad 1: cathode -> cathode-1
- U108 pad 1: cathode -> cathode-1
- U109 pad 5: hv-4 -> hv
- U110 pad 2: hv -> hv-4
- U111 pad 2: hv-4 -> hv
- U112 pad 1: vsh_connector-net-3 -> vsh_connector-net-5
- U112 pad 10: vsh_connector-net-2 -> vsh_connector-net-1
- U112 pad 11: vsh_connector-net-9 -> vsh_connector-net-8
- U112 pad 12: vsh_connector-net-6 -> vsh_connector-net
- U112 pad 13: vsh_connector-net-1 -> vsh_connector-net-13
- U112 pad 14: vsh_connector-net-11 -> vsh_connector-net-12
- U112 pad 15: io -> io-1
- U112 pad 17: io-1 -> io-2
- U112 pad 2: vsh_connector-net-8 -> vsh_connector-net-9
- U112 pad 21: io-2 -> io
- U112 pad 3: vsh_connector-net-5 -> vsh_connector-net-4
- U112 pad 4: vsh_connector-net -> vsh_connector-net-11
- U112 pad 5: vsh_connector-net-10 -> vsh_connector-net-2
- U112 pad 6: vsh_connector-net-13 -> vsh_connector-net-10
- U112 pad 7: vsh_connector-net-12 -> vsh_connector-net-7
- U112 pad 8: vsh_connector-net-7 -> vsh_connector-net-3
- U112 pad 9: vsh_connector-net-4 -> vsh_connector-net-6
- U17 pad 10: dep_relay.gpio_expander-net-3 -> dep_relay.gpio_expander-net-1
- U17 pad 12: line-3 -> line-13
- U17 pad 13: line-12 -> line-11
- U17 pad 3: dep_relay.gpio_expander-net-4 -> dep_relay.gpio_expander-net
- U17 pad 4: dep_relay.gpio_expander-net-1 -> dep_relay.gpio_expander-net-4
- U17 pad 7: dep_relay.gpio_expander-net-2 -> dep_relay.gpio_expander-net-5
- U17 pad 8: dep_relay.gpio_expander-net -> dep_relay.gpio_expander-net-3
- U17 pad 9: dep_relay.gpio_expander-net-5 -> dep_relay.gpio_expander-net-2
- U36 pad 1: in -> in-1
- U36 pad 2: in -> in-1
- U37 pad 2: in -> in-1
- U38 pad 1: in-1 -> in
- U38 pad 2: in-1 -> in
- U39 pad 2: in-1 -> in
- U40 pad 27: in -> in-1
- U40 pad 3: in-1 -> in
- U40 pad 6: line-8 -> line-5
- U40 pad 7: line-10 -> line-9
- U44 pad 10: line-11 -> line-10
- U44 pad 11: line-13 -> line-1
- U44 pad 13: line-9 -> line-8
- U44 pad 14: line-7 -> line-3
- U44 pad 15: line-5 -> line-6
- U44 pad 16: line-6 -> line-7
- U44 pad 17: line-1 -> line
- U44 pad 18: line-4 -> line-2
- U44 pad 19: line-12 -> line-11
- U44 pad 20: line-3 -> line-13
- U44 pad 22: line-8 -> line-5
- U44 pad 23: line-10 -> line-9
- U44 pad 4: i2c_multiplexer-line -> i2c_multiplexer-line-1
- U44 pad 5: i2c_multiplexer-line-2 -> i2c_multiplexer-line
- U44 pad 6: i2c_multiplexer-line-1 -> i2c_multiplexer-line-3
- U44 pad 7: i2c_multiplexer-line-3 -> i2c_multiplexer-line-2
- U44 pad 8: line -> line-4
- U44 pad 9: line-2 -> line-12
- U45 pad 2: i2c_multiplexer-line-2 -> i2c_multiplexer-line
- U46 pad 2: i2c_multiplexer-line -> i2c_multiplexer-line-1
- U47 pad 2: i2c_multiplexer-line-3 -> i2c_multiplexer-line-2
- U48 pad 2: i2c_multiplexer-line-1 -> i2c_multiplexer-line-3
- U49 pad 2: line-2 -> line-12
- U50 pad 2: line -> line-4
- U51 pad 2: line-13 -> line-1
- U52 pad 2: line-11 -> line-10
- U53 pad 2: line-7 -> line-3
- U54 pad 2: line-9 -> line-8
- U55 pad 2: line-6 -> line-7
- U56 pad 2: line-5 -> line-6
- U57 pad 2: line-4 -> line-2
- U58 pad 2: line-1 -> line
- U59 pad 2: line-3 -> line-13
- U60 pad 2: line-12 -> line-11
- U62 pad 1: inverting-3 -> inverting
- U62 pad 2: io -> io-1
- U63 pad 2: inverting-3 -> inverting
- U64 pad 1: io -> io-1
- U64 pad 2: inverting-3 -> inverting
- U64 pad 3: non_inverting -> non_inverting-2
- U65 pad 4: line -> line-4
- U65 pad 5: line-2 -> line-12
- U66 pad 1: non_inverting -> non_inverting-2
- U67 pad 2: non_inverting -> non_inverting-2
- U68 pad 1: inverting-1 -> inverting-2
- U68 pad 2: io-1 -> io-2
- U69 pad 2: inverting-1 -> inverting-2
- U70 pad 1: io-1 -> io-2
- U70 pad 2: inverting-1 -> inverting-2
- U70 pad 3: non_inverting-2 -> non_inverting-3
- U71 pad 4: line-11 -> line-10
- U71 pad 5: line-13 -> line-1
- U72 pad 1: non_inverting-2 -> non_inverting-3
- U73 pad 2: non_inverting-2 -> non_inverting-3
- U74 pad 1: inverting -> inverting-1
- U75 pad 2: inverting -> inverting-1
- U76 pad 2: inverting -> inverting-1
- U76 pad 3: non_inverting-3 -> non_inverting-1
- U77 pad 4: line-9 -> line-8
- U77 pad 5: line-7 -> line-3
- U78 pad 1: non_inverting-3 -> non_inverting-1
- U79 pad 2: non_inverting-3 -> non_inverting-1
- U80 pad 1: inverting-2 -> inverting-3
- U80 pad 2: io-2 -> io
- U81 pad 2: inverting-2 -> inverting-3
- U82 pad 1: io-2 -> io
- U82 pad 2: inverting-2 -> inverting-3
- U82 pad 3: non_inverting-1 -> non_inverting
- U83 pad 4: line-5 -> line-6
- U83 pad 5: line-6 -> line-7
- U84 pad 1: non_inverting-1 -> non_inverting
- U85 pad 2: non_inverting-1 -> non_inverting
- U98 pad 7: line-8 -> line-5
- U98 pad 8: line-10 -> line-9
Routing:
- net line-10: track 61.0 -> 16.3 mm, vias 4 -> 0
- net line-9: track 17.0 -> 61.0 mm, vias 2 -> 4
- net line-8: track 60.8 -> 17.0 mm, vias 3 -> 2
- net line-5: track 30.3 -> 60.8 mm, vias 2 -> 3
- net line: track 12.7 -> 35.1 mm
- net in-1: track 32.2 -> 9.92 mm, vias 2 -> 0
- net in: track 9.92 -> 32.2 mm, vias 0 -> 2
- net line-2: track 12.0 -> 34.0 mm
- net line-4: track 34.0 -> 12.7 mm
- net line-1: track 35.1 -> 15.6 mm, vias 2 -> 0
- net line-7: track 15.0 -> 29.1 mm
- net line-12: track 24.0 -> 12.0 mm
- net line-3: track 24.2 -> 15.0 mm
- net io: track 31.8 -> 22.7 mm
- net line-13: track 15.6 -> 24.2 mm, vias 0 -> 2
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
Commit message: Fix layout for CM4, update ato, delete CM4 example, replacing with SpaceBMSHIL
Parts:
- removed D6, D7: , atopile:DFN1610-2_L1.6-W1.0-P1.05-RD-57a24e
- removed DS1: , lib:SOD-323_L1.8-W1.3-LS2.5-RD
- removed Q2, Q3: , lib:SOT-23-3_L2.9-W1.3-P1.90-LS2.4-BR
- removed U10: 12.4kΩ ±1% 62.5mW, atopile:R0402-56259e
- removed U100, U102, U106, U108: 1kΩ ±1% 62.5mW, atopile:R0402-56259e
- removed U101, U107: , lib:LED0603-RD
- removed U103, U109: , lib:RELAY-SMD_HFD4-5-SR
- removed U104, U17: , lib:QFN-16_L3.0-W3.0-P0.50-BL-EP1.7
- removed U105, U37, U39, U45, U46, U47, U48, U49, U50, U51, U52, U53, U54, U55, U56, U57, U58, U59, U60, U61, U62, U63, U67, U68, U69, U73, U74, U75, U79, U80, U81, U85, U86, U92, U99: 10kΩ ±1% 62.5mW, atopile:R0402-56259e
- removed U11: 1nF ±10% 50V X7R, atopile:C0805-3b2e55
- removed U110, U111: , lib:CON2_1X2_U_DF13
- removed U112: , lib:CON_5030912221_MOL
- removed U113, U114, U115, U116, U88, U90: 1µF ±10% 25V X5R, atopile:C0402-b3ef17
- removed U12: 220Ω ±1% 62.5mW, atopile:R0402-56259e
- removed U13: 1MΩ ±1% 62.5mW, atopile:R0402-56259e
- removed U14: , lib:CRYSTAL-SMD_4P-L3.2-W2.5-BL
- removed U15, U16: 10pF ±5% 50V C0G, atopile:C0402-b3ef17
- removed U18: , lib:RJ45-TH_J1B1211CCD
- removed U19: 10nF ±10% 50V X7R, atopile:C0402-b3ef17
- removed U20, U23: 6.8nF ±10% 50V X7R, atopile:C0402-b3ef17
- removed U21, U24, U29, U31: 33Ω ±1% 62.5mW, atopile:R0402-56259e
- removed U22, U25, U30, U32: 49.9Ω ±1% 62.5mW, atopile:R0402-56259e
- removed U26: 4.7µF ±10% 10V X5R, atopile:C0402-b3ef17
- removed U27: 22nF ±10% 50V X7R, atopile:C0402-b3ef17
- removed U28: 10Ω ±1% 62.5mW, atopile:R0402-56259e
- removed U3, U34, U35, U97: 10µF ±10% 25V X5R, atopile:C0805-3b2e55
- removed U33: , lib:LQFP-48_L7.0-W7.0-P0.50-LS9.0-BL
- removed U36, U38: , lib:KEY-SMD_4P-L4.2-W3.2-P2.20-LS4.6
- removed U4, U41, U42, U5, U6, U66, U7, U72, U78, U8, U84, U9: 100nF ±10% 16V X7R, atopile:C0402-b3ef17
- removed U40: , lib:WIRELM-SMD_ESP32-S3-WROOM-1
- removed U43: 2.2µF ±10% 25V X5R, atopile:C0603-bd72f6
- removed U44: , lib:TSSOP-24_L7.8-W4.4-P0.65-LS6.4-BL
- removed U64, U70, U76, U82: , atopile:SOIC-8_L5.0-W4.0-P1.27-LS6.0-BL-294f77
- removed U65, U71, U77, U83: , lib:SOT-23-6_L2.9-W1.6-P0.95-LS2.8-BL
- removed U87: 18kΩ ±0% 62.5mW, atopile:R0402-56259e
- removed U89: , lib:SOT-23-5_L3.0-W1.7-P0.95-LS2.8-BL
- removed U91: 470nF ±20% 16V X5R, atopile:C0402-b3ef17
- removed U93: 56kΩ ±0% 62.5mW, atopile:R0402-56259e
- removed U94: , lib:SOT-23-6_L2.9-W1.6-P0.95-LS2.8-BR
- removed U95: , lib:IND-SMD_L4.0-W4.0
- removed U96: 2.2µF ±20% 6.3V X5R, atopile:C0402-b3ef17
- removed U98: , atopile:QFN-24_L4.0-W4.0-P0.50-BL-EP2.8-2a85a7
- added CN1: , atopile:CONN-SMD_DF40C-100DS-0.4V-51-ceffa9, F.Cu at (164.1, 84.2)
- added CN2: , atopile:CONN-SMD_DF40C-100DS-0.4V-51-ceffa9, F.Cu at (164.1, 118.2)
- added R10: 22kΩ ±1% 62.5mW, atopile:R0402-56259e, F.Cu at (159.5, 40.8)
- added R11: 100Ω ±1% 62.5mW, atopile:R0402-56259e, F.Cu at (158.3, 42.2)
- added R8: 1kΩ ±1% 62.5mW, atopile:R0402-56259e, F.Cu at (156.1, 44.3)
- added R9: 100kΩ ±1% 62.5mW, atopile:R0402-56259e, F.Cu at (158.3, 40.2)
- added RJ1: , atopile:RJ45-TH_HR911130A-5845d4, F.Cu at (185.2, 70.9)
- D1: footprint atopile:SMB_L4.6-W3.6-LS5.3-RD-330cb3 -> atopile:LED0603-RD-YELLOW-5af84a
- D2: footprint atopile:SMB_L4.6-W3.6-LS5.3-RD-330cb3 -> atopile:LED0603-RD-c81ffb
- D3: footprint atopile:SMB_L4.6-W3.6-LS5.3-RD-330cb3 -> atopile:SOT-323-3_L2.1-W1.3-P1.32-LS2.1-BR-ee9edb
- D4: footprint atopile:SMB_L4.6-W3.6-LS5.3-RD-330cb3 -> atopile:DFN1610-2_L1.6-W1.0-P1.05-RD-57a24e
- D5: footprint atopile:SOT-323-3_L2.1-W1.3-P1.32-LS2.1-BR-ee9edb -> atopile:DFN1610-2_L1.6-W1.0-P1.05-RD-57a24e
- R2: value 4.7kΩ ±1% 62.5mW -> 1kΩ ±1% 62.5mW
- R3: value 4.7kΩ ±1% 62.5mW -> 470Ω ±1% 100mW; footprint atopile:R0402-56259e -> atopile:R0603-ebcab9
- R4: value 1kΩ ±1% 62.5mW -> 470Ω ±1% 100mW; footprint atopile:R0402-56259e -> atopile:R0603-ebcab9
- R5: value 100kΩ ±1% 62.5mW -> 1kΩ ±1% 62.5mW
- R6: value 22kΩ ±1% 62.5mW -> 4.7kΩ ±1% 62.5mW
- R7: value 100Ω ±1% 62.5mW -> 4.7kΩ ±1% 62.5mW
- U1: value 10nF ±10% 50V X7R -> (none); footprint atopile:C0402-b3ef17 -> atopile:SOT-23-5_L3.0-W1.7-P0.95-LS2.8-BR-9d80aa
- U2: value 220Ω ±1% 62.5mW -> (none); footprint atopile:R0402-56259e -> atopile:QFN-24_L4.0-W4.0-P0.50-BL-EP2.8-2a85a7
- moved R4 92.8 mm to (189.2, 61.8), turned to 0 degrees
- moved D5 91.2 mm to (153.6, 40.6)
- moved R3 85.9 mm to (189.2, 80.0), turned to 0 degrees
- moved C1 84.3 mm to (153.6, 45.5)
- moved C2 84.3 mm to (160.5, 43.1)
- moved C3 84.3 mm to (159.5, 43.1)
- moved C4 84.3 mm to (157.7, 43.7)
- moved Q1 84.3 mm to (156.2, 41.2)
- moved USB1 84.3 mm to (148.5, 44.1)
- moved R5 79.1 mm to (155.0, 44.3), turned to -90 degrees
- moved R7 77.2 mm to (155.0, 48.4), turned to 90 degrees
- moved R6 75.9 mm to (156.0, 48.4)
- moved R1 67.6 mm to (169.8, 79.4)
- moved R2 56.0 mm to (151.4, 79.4), turned to -90 degrees
- moved D3 40.5 mm to (153.1, 48.1)
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Connections:
- net SSRXP1 renamed B11
- net SSTXN1 renamed A3
- net SSTXP1 renamed A2
- net dm renamed power-line-2
- net dp renamed power-line-1
- C1 pad 1: gnd -> power-gnd
- C2 pad 1: gnd -> power-gnd
- C3 pad 1: gnd -> power-gnd
- C4 pad 1: usb_pd.pd_controller-net -> power.pd_controller-net
- D1 pad 1: io-1 -> controller.cm4-cathode
- D1 pad 2: gnd -> VCC_3V3
- D2 pad 1: io-2 -> controller.cm4-cathode-1
- D2 pad 2: gnd -> VCC_3V3
- D3 pad 1: io-3 -> CC1
- D3 pad 2: gnd -> CC2
- D4 pad 1: io -> VBUS
- D4 pad 2: gnd -> power-gnd
- D5 pad 1: CC1 -> VSINK_VCC
- D5 pad 2: CC2 -> power-gnd
- Q1 pad 4: usb_pd.pd_controller-gate -> gate
- R1 pad 1: VBUS -> controller.cm4-cathode
- R1 pad 2: DISCH -> pins[19]
- R2 pad 1: line-5 -> controller.cm4-cathode-1
- R2 pad 2: usb_pd-hv -> controller.cm4-line
- R3 pad 1: line-9 -> VCC_3V3
- R3 pad 2: usb_pd-hv -> controller.rj45-anode-1
- R4 pad 1: VBUS -> VCC_3V3
- R4 pad 2: VBUS_VS_DISCH -> controller.rj45-anode
- R5 pad 1: usb_pd.pd_controller-gate -> VBUS
- R5 pad 2: VSINK_VCC -> DISCH
- R6 pad 1: usb_pd.pd_controller-gate -> power-line
- R6 pad 2: VBUS_EN_SNK -> hv
- R7 pad 1: usb_pd.pd_controller-gate -> power-line-3
- R7 pad 2: usb_pd.pd_controller-net -> hv
- U1 pad 1: _1V2O -> N_C_
- U1 pad 2: gnd -> PWR_LED
- U2 pad 1: ACTLED -> power.pd_controller.pd_controller-line-1
- U2 pad 2: RLED_minus -> CC1
- USB1 pad 1: gnd -> power-gnd
- USB1 pad 2: gnd -> power-gnd
- USB1 pad 3: gnd -> power-gnd
- USB1 pad 4: gnd -> power-gnd
- USB1 pad A1: gnd -> power-gnd
- USB1 pad A12: gnd -> power-gnd
- USB1 pad B1: gnd -> power-gnd
- USB1 pad B12: gnd -> power-gnd
Routing:
- net gnd: track 232.6 -> 0.00 mm, vias 53 -> 0
- net hv-2: track 98.6 -> 0.00 mm, vias 26 -> 0
- net anode: track 68.3 -> 0.00 mm, vias 2 -> 0
- net line-9: track 61.0 -> 0.00 mm, vias 4 -> 0
- net line-5: track 60.8 -> 0.00 mm, vias 3 -> 0
- net RLED_minus: track 44.2 -> 0.00 mm
- net LLED_minus: track 42.9 -> 0.00 mm
- net mosi: track 35.6 -> 0.00 mm, vias 2 -> 0
- net line: track 35.1 -> 0.00 mm, vias 2 -> 0
- net line-2: track 34.0 -> 0.00 mm, vias 2 -> 0
- net cs: track 32.4 -> 0.00 mm, vias 2 -> 0
- net in: track 32.2 -> 0.00 mm, vias 2 -> 0
- net ETH_LED_ACTIVITY: track 0.00 -> 32.0 mm, vias 0 -> 1
- net io-1: track 31.8 -> 0.00 mm
- net sck: track 31.0 -> 0.00 mm, vias 2 -> 0
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- added copper zone on B.Cu, net power-gnd
- added copper zone on F.Cu, net power-gnd
- removed copper zone on F.Cu, net VSINK_VCC
- removed copper zone on F.Cu, net anode
- removed copper zone on F.Cu, net cathode-2
- removed copper zone on B.Cu, net gnd
- removed copper zone on F.Cu, net gnd
- removed copper zone on In1.Cu, net gnd
- removed copper zone on F.Cu, net hv-2
- removed copper zone on In2.Cu, net hv-2
Other:
- board outline removed
- board text removed: "BMS HIL"
- board text removed: "BOOT"
- board text removed: "DEP"
- board text removed: "Made with atopile"
- board text removed: "NTC1"
- board text removed: "NTC2"
- board text removed: "NTC3"
- board text removed: "NTC4"
- board text removed: "RESET"
- board text removed: "SEP"
- board text removed: "{{GITHASH}}"

Commit message: analog out, relay, cleanup
Connections:
- CN1 pad 15: controller-line -> controller-line-2
- CN1 pad 17: controller-line-3 -> controller-line
- CN1 pad 22: controller.cm4-line-7 -> controller.cm4-line-3
- CN1 pad 24: controller.cm4-line-1 -> controller.cm4-line-7
- CN1 pad 75: controller.cm4-line-3 -> controller.cm4-line-4
- CN1 pad 78: controller.cm4-line-4 -> controller.cm4-line-6
- CN1 pad 81: controller.cm4-line-6 -> controller.cm4-line-2
- CN1 pad 82: controller-line-2 -> controller-line-3
- CN1 pad 85: controller.cm4-line-2 -> controller.cm4-line-1
- R6 pad 1: power-line -> power-line-2
- R7 pad 1: power-line-3 -> power-line
- RJ1 pad P1: controller.rj45.connector-net-1 -> controller.rj45.connector-net
- RJ1 pad P10: controller.rj45.connector-net -> controller.rj45.connector-net-1
- U2 pad 7: power-line -> power-line-2
- U2 pad 8: power-line-3 -> power-line
- USB1 pad A6: power-line-1 -> power-line-3
- USB1 pad A7: power-line-2 -> power-line-1
- USB1 pad B6: power-line-1 -> power-line-3
- USB1 pad B7: power-line-2 -> power-line-1
Routing:
- net power-line-1: track 0.82 -> 5.17 mm, vias 0 -> 2
- net power-line-3: track 4.26 -> 0.82 mm
- net power-line-2: track 5.17 -> 2.17 mm, vias 2 -> 1
- net power-line: track 2.17 -> 4.26 mm, vias 1 -> 0

Commit message: Everything builds
Connections:
- net controller.cm4-pins[49] renamed controller.cm4-line-9
- net controller.cm4.hdi_b-pins[23] renamed pins[23]
- net controller.cm4.hdi_b-pins[28] renamed pins[28]
- net controller.cm4.hdi_b-pins[49] renamed pins[49]
- net pins[44] renamed controller.cm4-pins[44]-1
- net pins[45] renamed controller.cm4-line-8
- net pins[46] renamed controller.cm4-pins[46]
- CN1 pad 12: controller.cm4-pins[23] -> controller.cm4-line-7
- CN1 pad 15: controller-line-2 -> controller-line
- CN1 pad 17: controller-line -> controller-line-3
- CN1 pad 19: pins[37] -> controller.cm4-line-6
- CN1 pad 22: controller.cm4-line-3 -> pins[43]
- CN1 pad 24: controller.cm4-line-7 -> controller.cm4-line-4
- CN1 pad 29: pins[57] -> controller.cm4-line-2
- CN1 pad 75: controller.cm4-line-4 -> controller.cm4-line
- CN1 pad 77: controller.cm4-line-5 -> controller.cm4-pins[46]-1
- CN1 pad 78: controller.cm4-line-6 -> controller.cm4-pins[44]
- CN1 pad 81: controller.cm4-line-2 -> controller.cm4-line-5
- CN1 pad 82: controller-line-3 -> controller-line-2
- CN1 pad 85: controller.cm4-line-1 -> pins[30]
- CN1 pad 86: controller.cm4-pins[28] -> controller.cm4-line-1
- D1 pad 1: controller.cm4-cathode -> controller.cm4-cathode-1
- D2 pad 1: controller.cm4-cathode-1 -> controller.cm4-cathode
- R1 pad 1: controller.cm4-cathode -> controller.cm4-cathode-1
- R2 pad 1: controller.cm4-cathode-1 -> controller.cm4-cathode
- R2 pad 2: controller.cm4-line -> controller.cm4-line-3
- R3 pad 2: controller.rj45-anode-1 -> controller.rj45-anode
- R4 pad 2: controller.rj45-anode -> controller.rj45-anode-1
- R6 pad 1: power-line-2 -> power-line-1
- R7 pad 1: power-line -> power-line-3
- RJ1 pad 12: controller.rj45-anode-1 -> controller.rj45-anode
- RJ1 pad 13: controller.rj45-anode -> controller.rj45-anode-1
- U1 pad 4: controller.cm4-line -> controller.cm4-line-3
- U2 pad 7: power-line-2 -> power-line-1
- U2 pad 8: power-line -> power-line-3
- USB1 pad A6: power-line-3 -> power-line-2
- USB1 pad A7: power-line-1 -> power-line
- USB1 pad B6: power-line-3 -> power-line-2
- USB1 pad B7: power-line-1 -> power-line
Routing:
- net power-line-3: track 0.82 -> 4.26 mm
- net power-line-1: track 5.17 -> 2.17 mm, vias 2 -> 1
- net controller.cm4-line-3: track 0.00 -> 1.86 mm
- net controller.cm4-line: track 1.86 -> 0.00 mm
- net power-line-2: track 2.17 -> 0.82 mm, vias 1 -> 0
- net power-line: track 4.26 -> 5.17 mm, vias 0 -> 2
