File: elec/layout/i2c-relay/i2c-relay.kicad_pcb (KiCad board)
At the start: 2 copper layers, 7 parts, among them U2 10kΩ ±1% 62.5mW, U3 1kΩ ±1% 62.5mW, U5 1kΩ ±1% 62.5mW

Commit message: remove default build, build everything locally
Connections:
- Q1 pad 2: gnd-1 -> gnd-2
- U1 pad 10: gpio_expander-net-2 -> gpio_expander-net-3
- U1 pad 3: gpio_expander-net-5 -> gpio_expander-net
- U1 pad 4: gpio_expander-net-4 -> gpio_expander-net-6
- U1 pad 5: gpio_expander-net -> gpio_expander-net-2
- U1 pad 7: gpio_expander-net-6 -> gpio_expander-net-1
- U1 pad 8: gpio_expander-net-1 -> gpio_expander-net-4
- U1 pad 9: gpio_expander-net-3 -> gpio_expander-net-5
- U3 pad 2: gnd-1 -> gnd-2
- U6 pad 3: gnd-2 -> gnd-1
Routing:
- net gnd-2: track 0.00 -> 1.46 mm
- net gnd-1: track 1.46 -> 0.00 mm

Commit message: fix resistor values while solver isnt ready
Connections:
- net VCCP renamed VCCI
- Q1 pad 2: gnd-2 -> gnd-1
- U1 pad 10: gpio_expander-net-3 -> gpio_expander-net-4
- U1 pad 12: line-1 -> line
- U1 pad 13: line -> line-1
- U1 pad 16: gnd -> gnd-2
- U1 pad 17: gnd -> gnd-2
- U1 pad 3: gpio_expander-net -> gpio_expander-net-6
- U1 pad 4: gpio_expander-net-6 -> gpio_expander-net-2
- U1 pad 5: gpio_expander-net-2 -> gpio_expander-net-3
- U1 pad 6: gnd -> gnd-2
- U1 pad 7: gpio_expander-net-1 -> gpio_expander-net
- U1 pad 8: gpio_expander-net-4 -> gpio_expander-net-1
- U3 pad 2: gnd-2 -> gnd-1
- U6 pad 3: gnd-1 -> gnd
Routing:
- net gnd: track 2.55 -> 0.00 mm, vias 1 -> 0
- net gnd-1: track 0.00 -> 1.46 mm
- net gnd-2: track 1.46 -> 2.55 mm, vias 0 -> 1
Changed lines of the file:
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@@
             (outputdirectory "")))
     (net 0 "")
-    (net 1 "gpio_expander-net-6")
-    (net 2 "line-1")
-    (net 3 "gpio_expander-net-3")
+    (net 1 "gpio_expander-net-2")
+    (net 2 "line")
+    (net 3 "gpio_expander-net-4")
     (net 4 "hv")
-    (net 5 "gpio_expander-net-1")
+    (net 5 "gpio_expander-net")
     (net 6 "gpio_expander-net-5")
     (net 7 "anode")
     (net 8 "input")
-    (net 9 "gnd-1")
+    (net 9 "gnd")
     (net 10 "INT")
-    (net 11 "gpio_expander-net-4")
-    (net 12 "VCCP")
+    (net 11 "gpio_expander-net-1")
+    (net 12 "VCCI")
     (net 13 "hv-1")
-    (net 14 "line")
-    (net 15 "gpio_expander-net-2")
+    (net 14 "line-1")
+    (net 15 "gpio_expander-net-3")
     (net 16 "gnd-3")
-    (net 17 "gnd-2")
+    (net 17 "gnd-1")
     (net 18 "cathode")
     (net 19 "relay-gnd")
     (net 20 "gate")
-    (net 21 "gpio_expander-net")
-    (net 22 "gnd")
+    (net 21 "gpio_expander-net-6")
+    (net 22 "gnd-2")
     (footprint "atopile:R0402-56259e"
         (layer "F.Cu")
@@
             (layers "F.Cu" "F.Paste" "F.Mask")
             (remove_unused_layers no)
-            (net 17 "gnd-2")))
+            (net 17 "gnd-1")))
     (footprint "lib:LED0603-RD"
         (layer "F.Cu")
@@
             (layers "F.Cu" "F.Paste" "F.Mask")
             (remove_unused_layers no)
-            (net 9 "gnd-1"))
+            (net 9 "gnd"))
         (pad "4" smd rect
             (at 3.84 3.17 0)
@@
             (layers "F.Cu" "F.Paste" "F.Mask")
             (remove_unused_layers no)
-            (net 17 "gnd-2"))
+            (net 17 "gnd-1"))
         (pad "3" smd rect
             (at -1 0 180)
@@
             (layers "F.Cu" "F.Paste" "F.Mask")
             (remove_unused_layers no)
-            (net 12 "VCCP"))
+            (net 12 "VCCI"))
         (pad "2" smd rect
             (at -0.25 1.41 90)
@@
             (layers "F.Cu" "F.Paste" "F.Mask")
             (remove_unused_layers no)
-            (net 21 "gpio_expander-net"))
+            (net 21 "gpio_expander-net-6"))
         (pad "4" smd rect
             (at 0.75 1.41 90)
@@
             (layers "F.Cu" "F.Paste" "F.Mask")
             (remove_unused_layers no)
-            (net 1 "gpio_expander-net-6"))
+            (net 1 "gpio_expander-net-2"))
         (pad "5" smd rect
             (at 1.41 0.75 90)
@@
             (layers "F.Cu" "F.Paste" "F.Mask")
             (remove_unused_layers no)
-            (net 15 "gpio_expander-net-2"))
+            (net 15 "gpio_expander-net-3"))
         (pad "6" smd rect
             (at 1.41 0.25 90)
@@
             (layers "F.Cu" "F.Paste" "F.Mask")
             (remove_unused_layers no)
-            (net 22 "gnd"))
+            (net 22 "gnd-2"))
         (pad "7" smd rect
             (at 1.41 -0.25 90)
@@
             (layers "F.Cu" "F.Paste" "F.Mask")
             (remove_unused_layers no)
-            (net 5 "gpio_expander-net-1"))
+            (net 5 "gpio_expander-net"))
         (pad "8" smd rect
             (at 1.41 -0.75 90)
@@
             (layers "F.Cu" "F.Paste" "F.Mask")
             (remove_unused_layers no)
-            (net 11 "gpio_expander-net-4"))
+            (net 11 "gpio_expander-net-1"))
         (pad "9" smd rect
             (at 0.75 -1.41 90)
@@
             (layers "F.Cu" "F.Paste" "F.Mask")
             (remove_unused_layers no)
-            (net 3 "gpio_expander-net-3"))
+            (net 3 "gpio_expander-net-4"))
         (pad "11" smd rect
             (at -0.25 -1.41 90)
@@
             (layers "F.Cu" "F.Paste" "F.Mask")
             (remove_unused_layers no)
-            (net 2 "line-1"))
+            (net 2 "line"))
         (pad "13" smd rect
             (at -1.41 -0.75 90)
@@
             (layers "F.Cu" "F.Paste" "F.Mask")
             (remove_unused_layers no)
-            (net 14 "line"))
+            (net 14 "line-1"))
         (pad "14" smd rect
             (at -1.41 -0.25 90)
@@
             (layers "F.Cu" "F.Paste" "F.Mask")
             (remove_unused_layers no)
-            (net 12 "VCCP"))
+            (net 12 "VCCI"))
         (pad "15" smd rect
             (at -1.41 0.25 90)
@@
             (layers "F.Cu" "F.Paste" "F.Mask")
             (remove_unused_layers no)
-            (net 12 "VCCP"))
+            (net 12 "VCCI"))
         (pad "16" smd rect
             (at -1.41 0.75 90)
@@
             (layers "F.Cu" "F.Paste" "F.Mask")
             (remove_unused_layers no)
-            (net 22 "gnd"))
+            (net 22 "gnd-2"))
         (pad "17" smd rect
             (at 0 0 90)
@@
             (layers "F.Cu" "F.Paste" "F.Mask")
             (remove_unused_layers no)
-            (net 22 "gnd"))
+            (net 22 "gnd-2"))
         (model "/Users/narayanpowderly/projects/hil-blocks/build/footprints/footprints.3dshapes/QFN-16_L3.0-W3.0-H0.9-P0.50.step"
             (offset

Commit message: add module builds back in to ato.yaml with mfg-data excluded in config
Connections:
- net VCCI renamed VCCP
- Q1 pad 2: gnd-1 -> gnd-2
- U1 pad 12: line -> line-1
- U1 pad 13: line-1 -> line
- U1 pad 16: gnd-2 -> gnd-1
- U1 pad 17: gnd-2 -> gnd-1
- U1 pad 3: gpio_expander-net-6 -> gpio_expander-net-2
- U1 pad 4: gpio_expander-net-2 -> gpio_expander-net-5
- U1 pad 5: gpio_expander-net-3 -> gpio_expander-net
- U1 pad 6: gnd-2 -> gnd-1
- U1 pad 7: gpio_expander-net -> gpio_expander-net-6
- U1 pad 8: gpio_expander-net-1 -> gpio_expander-net-3
- U1 pad 9: gpio_expander-net-5 -> gpio_expander-net-1
- U3 pad 2: gnd-1 -> gnd-2
- U6 pad 5: hv-1 -> hv
- U6 pad 6: hv -> hv-1
Routing:
- net gnd-2: track 2.55 -> 1.46 mm, vias 1 -> 0
- net gnd-1: track 1.46 -> 2.55 mm, vias 0 -> 1
Changed lines of the file:
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@@
             (outputdirectory "")))
     (net 0 "")
-    (net 1 "gpio_expander-net-2")
-    (net 2 "line")
+    (net 1 "gpio_expander-net-5")
+    (net 2 "line-1")
     (net 3 "gpio_expander-net-4")
-    (net 4 "hv")
-    (net 5 "gpio_expander-net")
-    (net 6 "gpio_expander-net-5")
+    (net 4 "hv-1")
+    (net 5 "gpio_expander-net-6")
+    (net 6 "gpio_expander-net-1")
     (net 7 "anode")
     (net 8 "input")
     (net 9 "gnd")
     (net 10 "INT")
-    (net 11 "gpio_expander-net-1")
-    (net 12 "VCCI")
-    (net 13 "hv-1")
-    (net 14 "line-1")
-    (net 15 "gpio_expander-net-3")
+    (net 11 "gpio_expander-net-3")
+    (net 12 "VCCP")
+    (net 13 "hv")
+    (net 14 "line")
+    (net 15 "gpio_expander-net")
     (net 16 "gnd-3")
-    (net 17 "gnd-1")
+    (net 17 "gnd-2")
     (net 18 "cathode")
     (net 19 "relay-gnd")
     (net 20 "gate")
-    (net 21 "gpio_expander-net-6")
-    (net 22 "gnd-2")
+    (net 21 "gpio_expander-net-2")
+    (net 22 "gnd-1")
     (footprint "atopile:R0402-56259e"
         (layer "F.Cu")
@@
             (layers "F.Cu" "F.Paste" "F.Mask")
             (remove_unused_layers no)
-            (net 17 "gnd-1")))
+            (net 17 "gnd-2")))
     (footprint "lib:LED0603-RD"
         (layer "F.Cu")
@@
             (layers "F.Cu" "F.Paste" "F.Mask")
             (remove_unused_layers no)
-            (net 13 "hv-1"))
+            (net 13 "hv"))
         (pad "6" smd rect
             (at 1.64 -3.18 0)
@@
             (layers "F.Cu" "F.Paste" "F.Mask")
             (remove_unused_layers no)
-            (net 4 "hv"))
+            (net 4 "hv-1"))
         (pad "7" smd rect
             (at -0.56 -3.18 0)
@@
             (layers "F.Cu" "F.Paste" "F.Mask")
             (remove_unused_layers no)
-            (net 17 "gnd-1"))
+            (net 17 "gnd-2"))
         (pad "3" smd rect
             (at -1 0 180)
@@
             (layers "F.Cu" "F.Paste" "F.Mask")
             (remove_unused_layers no)
-            (net 12 "VCCI"))
+            (net 12 "VCCP"))
         (pad "2" smd rect
             (at -0.25 1.41 90)
@@
             (layers "F.Cu" "F.Paste" "F.Mask")
             (remove_unused_layers no)
-            (net 21 "gpio_expander-net-6"))
+            (net 21 "gpio_expander-net-2"))
         (pad "4" smd rect
             (at 0.75 1.41 90)
@@
             (layers "F.Cu" "F.Paste" "F.Mask")
             (remove_unused_layers no)
-            (net 1 "gpio_expander-net-2"))
+            (net 1 "gpio_expander-net-5"))
         (pad "5" smd rect
             (at 1.41 0.75 90)
@@
             (layers "F.Cu" "F.Paste" "F.Mask")
             (remove_unused_layers no)
-            (net 15 "gpio_expander-net-3"))
+            (net 15 "gpio_expander-net"))
         (pad "6" smd rect
             (at 1.41 0.25 90)
@@
             (layers "F.Cu" "F.Paste" "F.Mask")
             (remove_unused_layers no)
-            (net 22 "gnd-2"))
+            (net 22 "gnd-1"))
         (pad "7" smd rect
             (at 1.41 -0.25 90)
@@
             (layers "F.Cu" "F.Paste" "F.Mask")
             (remove_unused_layers no)
-            (net 5 "gpio_expander-net"))
+            (net 5 "gpio_expander-net-6"))
         (pad "8" smd rect
             (at 1.41 -0.75 90)
@@
             (layers "F.Cu" "F.Paste" "F.Mask")
             (remove_unused_layers no)
-            (net 11 "gpio_expander-net-1"))
+            (net 11 "gpio_expander-net-3"))
         (pad "9" smd rect
             (at 0.75 -1.41 90)
@@
             (layers "F.Cu" "F.Paste" "F.Mask")
             (remove_unused_layers no)
-            (net 6 "gpio_expander-net-5"))
+            (net 6 "gpio_expander-net-1"))
         (pad "10" smd rect
             (at 0.25 -1.41 90)
@@
             (layers "F.Cu" "F.Paste" "F.Mask")
             (remove_unused_layers no)
-            (net 2 "line"))
+            (net 2 "line-1"))
         (pad "13" smd rect
             (at -1.41 -0.75 90)
@@
             (layers "F.Cu" "F.Paste" "F.Mask")
             (remove_unused_layers no)
-            (net 14 "line-1"))
+            (net 14 "line"))
         (pad "14" smd rect
             (at -1.41 -0.25 90)
@@
             (layers "F.Cu" "F.Paste" "F.Mask")
             (remove_unused_layers no)
-            (net 12 "VCCI"))
+            (net 12 "VCCP"))
         (pad "15" smd rect
             (at -1.41 0.25 90)
@@
             (layers "F.Cu" "F.Paste" "F.Mask")
             (remove_unused_layers no)
-            (net 12 "VCCI"))
+            (net 12 "VCCP"))
         (pad "16" smd rect
             (at -1.41 0.75 90)
@@
             (layers "F.Cu" "F.Paste" "F.Mask")
             (remove_unused_layers no)
-            (net 22 "gnd-2"))
+            (net 22 "gnd-1"))
         (pad "17" smd rect
             (at 0 0 90)
@@
             (layers "F.Cu" "F.Paste" "F.Mask")
             (remove_unused_layers no)
-            (net 22 "gnd-2"))
+            (net 22 "gnd-1"))
         (model "/Users/narayanpowderly/projects/hil-blocks/build/footprints/footprints.3dshapes/QFN-16_L3.0-W3.0-H0.9-P0.50.step"
             (offset

Commit message: rebuild all modules
Connections:
- net VCCP renamed VCCI
- Q1 pad 2: gnd-2 -> gnd-1
- U1 pad 16: gnd-1 -> gnd-2
- U1 pad 17: gnd-1 -> gnd-2
- U1 pad 3: gpio_expander-net-2 -> gpio_expander-net-3
- U1 pad 4: gpio_expander-net-5 -> gpio_expander-net-2
- U1 pad 6: gnd-1 -> gnd-2
- U1 pad 7: gpio_expander-net-6 -> gpio_expander-net-1
- U1 pad 8: gpio_expander-net-3 -> gpio_expander-net-6
- U1 pad 9: gpio_expander-net-1 -> gpio_expander-net-5
- U3 pad 2: gnd-2 -> gnd-1
- U6 pad 5: hv -> hv-1
- U6 pad 6: hv-1 -> hv
Routing:
- net gnd-2: track 1.46 -> 2.55 mm, vias 0 -> 1
- net gnd-1: track 2.55 -> 1.46 mm, vias 1 -> 0
Changed lines of the file:
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@@
             (outputdirectory "")))
     (net 0 "")
-    (net 1 "gpio_expander-net-5")
+    (net 1 "gpio_expander-net-2")
     (net 2 "line-1")
     (net 3 "gpio_expander-net-4")
-    (net 4 "hv-1")
-    (net 5 "gpio_expander-net-6")
-    (net 6 "gpio_expander-net-1")
+    (net 4 "hv")
+    (net 5 "gpio_expander-net-1")
+    (net 6 "gpio_expander-net-5")
     (net 7 "anode")
     (net 8 "input")
     (net 9 "gnd")
     (net 10 "INT")
-    (net 11 "gpio_expander-net-3")
-    (net 12 "VCCP")
-    (net 13 "hv")
+    (net 11 "gpio_expander-net-6")
+    (net 12 "VCCI")
+    (net 13 "hv-1")
     (net 14 "line")
     (net 15 "gpio_expander-net")
     (net 16 "gnd-3")
-    (net 17 "gnd-2")
+    (net 17 "gnd-1")
     (net 18 "cathode")
     (net 19 "relay-gnd")
     (net 20 "gate")
-    (net 21 "gpio_expander-net-2")
-    (net 22 "gnd-1")
+    (net 21 "gpio_expander-net-3")
+    (net 22 "gnd-2")
     (footprint "atopile:R0402-56259e"
         (layer "F.Cu")
@@
             (layers "F.Cu" "F.Paste" "F.Mask")
             (remove_unused_layers no)
-            (net 17 "gnd-2")))
+            (net 17 "gnd-1")))
     (footprint "lib:LED0603-RD"
         (layer "F.Cu")
@@
             (layers "F.Cu" "F.Paste" "F.Mask")
             (remove_unused_layers no)
-            (net 13 "hv"))
+            (net 13 "hv-1"))
         (pad "6" smd rect
             (at 1.64 -3.18 0)
@@
             (layers "F.Cu" "F.Paste" "F.Mask")
             (remove_unused_layers no)
-            (net 4 "hv-1"))
+            (net 4 "hv"))
         (pad "7" smd rect
             (at -0.56 -3.18 0)
@@
             (layers "F.Cu" "F.Paste" "F.Mask")
             (remove_unused_layers no)
-            (net 17 "gnd-2"))
+            (net 17 "gnd-1"))
         (pad "3" smd rect
             (at -1 0 180)
@@
             (layers "F.Cu" "F.Paste" "F.Mask")
             (remove_unused_layers no)
-            (net 12 "VCCP"))
+            (net 12 "VCCI"))
         (pad "2" smd rect
             (at -0.25 1.41 90)
@@
             (layers "F.Cu" "F.Paste" "F.Mask")
             (remove_unused_layers no)
-            (net 21 "gpio_expander-net-2"))
+            (net 21 "gpio_expander-net-3"))
         (pad "4" smd rect
             (at 0.75 1.41 90)
@@
             (layers "F.Cu" "F.Paste" "F.Mask")
             (remove_unused_layers no)
-            (net 1 "gpio_expander-net-5"))
+            (net 1 "gpio_expander-net-2"))
         (pad "5" smd rect
             (at 1.41 0.75 90)
@@
             (layers "F.Cu" "F.Paste" "F.Mask")
             (remove_unused_layers no)
-            (net 22 "gnd-1"))
+            (net 22 "gnd-2"))
         (pad "7" smd rect
             (at 1.41 -0.25 90)
@@
             (layers "F.Cu" "F.Paste" "F.Mask")
             (remove_unused_layers no)
-            (net 5 "gpio_expander-net-6"))
+            (net 5 "gpio_expander-net-1"))
         (pad "8" smd rect
             (at 1.41 -0.75 90)
@@
             (layers "F.Cu" "F.Paste" "F.Mask")
             (remove_unused_layers no)
-            (net 11 "gpio_expander-net-3"))
+            (net 11 "gpio_expander-net-6"))
         (pad "9" smd rect
             (at 0.75 -1.41 90)
@@
             (layers "F.Cu" "F.Paste" "F.Mask")
             (remove_unused_layers no)
-            (net 6 "gpio_expander-net-1"))
+            (net 6 "gpio_expander-net-5"))
         (pad "10" smd rect
             (at 0.25 -1.41 90)
@@
             (layers "F.Cu" "F.Paste" "F.Mask")
             (remove_unused_layers no)
-            (net 12 "VCCP"))
+            (net 12 "VCCI"))
         (pad "15" smd rect
             (at -1.41 0.25 90)
@@
             (layers "F.Cu" "F.Paste" "F.Mask")
             (remove_unused_layers no)
-            (net 12 "VCCP"))
+            (net 12 "VCCI"))
         (pad "16" smd rect
             (at -1.41 0.75 90)
@@
             (layers "F.Cu" "F.Paste" "F.Mask")
             (remove_unused_layers no)
-            (net 22 "gnd-1"))
+            (net 22 "gnd-2"))
         (pad "17" smd rect
             (at 0 0 90)
@@
             (layers "F.Cu" "F.Paste" "F.Mask")
             (remove_unused_layers no)
-            (net 22 "gnd-1"))
+            (net 22 "gnd-2"))
         (model "/Users/narayanpowderly/projects/hil-blocks/build/footprints/footprints.3dshapes/QFN-16_L3.0-W3.0-H0.9-P0.50.step"
             (offset
