File: elec/layout/isolator-i2c/isolator-i2c.kicad_pcb (KiCad board)
At the start: 2 copper layers, 7 parts, among them U1 1kΩ ±1% 62.5mW, U2 1kΩ ±1% 62.5mW, U4 1kΩ ±1% 62.5mW, U5 1kΩ ±1% 62.5mW, U6 100nF ±10% 16V X7R, U7 100nF ±10% 16V X7R

Commit message: update syntax, delete vendored packages
Parts:
- U1, U2, U4, U5: value 1kΩ ±1% 62.5mW -> 10kΩ ±1% 62.5mW
Connections:
- U1 pad 1: line-1 -> line-2
- U1 pad 2: hv -> hv-1
- U2 pad 1: line-3 -> line-1
- U2 pad 2: hv -> hv-1
- U3 pad 1: hv-1 -> hv
- U3 pad 2: line-2 -> line
- U3 pad 3: line -> line-3
- U3 pad 6: line-1 -> line-2
- U3 pad 7: line-3 -> line-1
- U3 pad 8: hv -> hv-1
- U4 pad 1: line -> line-3
- U4 pad 2: hv-1 -> hv
- U5 pad 1: line-2 -> line
- U5 pad 2: hv-1 -> hv
- U6 pad 1: hv -> hv-1
- U7 pad 1: hv-1 -> hv
Changed lines of the file:
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@@
             (outputdirectory "")))
     (net 0 "")
-    (net 1 "line-3")
-    (net 2 "line")
-    (net 3 "hv")
-    (net 4 "line-2")
-    (net 5 "line-1")
+    (net 1 "line-1")
+    (net 2 "line-3")
+    (net 3 "hv-1")
+    (net 4 "line")
+    (net 5 "line-2")
     (net 6 "gnd")
-    (net 7 "hv-1")
+    (net 7 "hv")
     (net 8 "gnd-1")
     (footprint "atopile:R0402-56259e"
@@
                     (size 0.7 0.7)
                     (thickness 0.2))))
-        (property "Value" "1kΩ ±1% 62.5mW"
+        (property "Value" "10kΩ ±1% 62.5mW"
             (at 0 4 90)
             (layer "F.Fab")
@@
                     (size 0.125 0.125)
                     (thickness 0.01875))))
-        (property "LCSC" "C11702"
-            (at 0 0 90)
-            (layer "User.9")
-            (hide yes)
-            (effects
-                (font
-                    (size 0.125 0.125)
-                    (thickness 0.01875))))
-        (property "Partnumber" "0402WGF1001TCE"
+        (property "LCSC" "C25744"
+            (at 0 0 90)
+            (layer "User.9")
+            (hide yes)
+            (effects
+                (font
+                    (size 0.125 0.125)
+                    (thickness 0.01875))))
+        (property "Partnumber" "0402WGF1002TCE"
             (at 0 0 90)
             (layer "User.9")
@@
                     (size 0.125 0.125)
                     (thickness 0.01875))))
-        (property "JLCPCB description" "62.5mW Thick Film Resistors 50V ±100ppm/℃ ±1% 1kΩ 0402 Chip Resistor - Surface Mount ROHS"
+        (property "JLCPCB description" "62.5mW Thick Film Resistors 50V ±100ppm/℃ ±1% 10kΩ 0402 Chip Resistor - Surface Mount ROHS"
             (at 0 0 90)
             (layer "User.9")
@@
             (layers "F.Cu" "F.Paste" "F.Mask")
             (remove_unused_layers no)
-            (net 1 "line-3"))
+            (net 1 "line-1"))
         (pad "2" smd rect
             (at 0.43 0 90)
@@
             (layers "F.Cu" "F.Paste" "F.Mask")
             (remove_unused_layers no)
-            (net 3 "hv")))
+            (net 3 "hv-1")))
     (footprint "atopile:SOIC-8_L4.9-W3.9-P1.27-LS6.0-TL-e13595"
         (layer "F.Cu")
@@
             (layers "F.Cu" "F.Paste" "F.Mask")
             (remove_unused_layers no)
-            (net 5 "line-1"))
+            (net 5 "line-2"))
         (pad "7" smd oval
             (at 2.74 -0.63 90)
@@
             (layers "F.Cu" "F.Paste" "F.Mask")
             (remove_unused_layers no)
-            (net 1 "line-3"))
+            (net 1 "line-1"))
         (pad "8" smd oval
             (at 2.74 -1.9 90)
@@
             (layers "F.Cu" "F.Paste" "F.Mask")
             (remove_unused_layers no)
-            (net 3 "hv"))
+            (net 3 "hv-1"))
         (pad "4" smd oval
             (at -2.74 1.91 90)
@@
             (layers "F.Cu" "F.Paste" "F.Mask")
             (remove_unused_layers no)
-            (net 2 "line"))
+            (net 2 "line-3"))
         (pad "2" smd oval
             (at -2.74 -0.63 90)
@@
             (layers "F.Cu" "F.Paste" "F.Mask")
             (remove_unused_layers no)
-            (net 4 "line-2"))
+            (net 4 "line"))
         (pad "1" smd oval
             (at -2.74 -1.9 90)
@@
             (layers "F.Cu" "F.Paste" "F.Mask")
             (remove_unused_layers no)
-            (net 7 "hv-1")))
+            (net 7 "hv")))
     (footprint "atopile:C0402-b3ef17"
         (layer "F.Cu")
@@
             (layers "F.Cu" "F.Paste" "F.Mask")
             (remove_unused_layers no)
-            (net 3 "hv"))
+            (net 3 "hv-1"))
         (pad "2" smd rect
             (at 0.55 0 180)
@@
             (layers "F.Cu" "F.Paste" "F.Mask")
             (remove_unused_layers no)
-            (net 7 "hv-1"))
+            (net 7 "hv"))
         (pad "2" smd rect
             (at 0.55 0 0)
@@
                     (size 0.7 0.7)
                     (thickness 0.2))))
-        (property "Value" "1kΩ ±1% 62.5mW"
+        (property "Value" "10kΩ ±1% 62.5mW"
             (at 0 4 90)
             (layer "F.Fab")
@@
                     (size 0.125 0.125)
                     (thickness 0.01875))))
-        (property "LCSC" "C11702"
-            (at 0 0 90)
-            (layer "User.9")
-            (hide yes)
-            (effects
-                (font
-                    (size 0.125 0.125)
-                    (thickness 0.01875))))
-        (property "Partnumber" "0402WGF1001TCE"
+        (property "LCSC" "C25744"
+            (at 0 0 90)
+            (layer "User.9")
+            (hide yes)
+            (effects
+                (font
+                    (size 0.125 0.125)
+                    (thickness 0.01875))))
+        (property "Partnumber" "0402WGF1002TCE"
             (at 0 0 90)
             (layer "User.9")
@@
                     (size 0.125 0.125)
                     (thickness 0.01875))))
-        (property "JLCPCB description" "62.5mW Thick Film Resistors 50V ±100ppm/℃ ±1% 1kΩ 0402 Chip Resistor - Surface Mount ROHS"
+        (property "JLCPCB description" "62.5mW Thick Film Resistors 50V ±100ppm/℃ ±1% 10kΩ 0402 Chip Resistor - Surface Mount ROHS"
             (at 0 0 90)
             (layer "User.9")
@@
             (layers "F.Cu" "F.Paste" "F.Mask")
             (remove_unused_layers no)
-            (net 5 "line-1"))
+            (net 5 "line-2"))
         (pad "2" smd rect
             (at 0.43 0 270)
@@
             (layers "F.Cu" "F.Paste" "F.Mask")
             (remove_unused_layers no)
-            (net 3 "hv")))
+            (net 3 "hv-1")))
     (footprint "atopile:R0402-56259e"
         (layer "F.Cu")
@@
                     (size 0.7 0.7)
                     (thickness 0.2))))
-        (property "Value" "1kΩ ±1% 62.5mW"
+        (property "Value" "10kΩ ±1% 62.5mW"
             (at 0 4 90)
             (layer "F.Fab")
@@
                     (size 0.125 0.125)
                     (thickness 0.01875))))
-        (property "LCSC" "C11702"
-            (at 0 0 90)
-            (layer "User.9")
-            (hide yes)
-            (effects
-                (font
-                    (size 0.125 0.125)
-                    (thickness 0.01875))))
-        (property "Partnumber" "0402WGF1001TCE"
+        (property "LCSC" "C25744"
+            (at 0 0 90)
+            (layer "User.9")
+            (hide yes)
+            (effects
+                (font
+                    (size 0.125 0.125)
+                    (thickness 0.01875))))
+        (property "Partnumber" "0402WGF1002TCE"
             (at 0 0 90)
             (layer "User.9")
@@
                     (size 0.125 0.125)
                     (thickness 0.01875))))
-        (property "JLCPCB description" "62.5mW Thick Film Resistors 50V ±100ppm/℃ ±1% 1kΩ 0402 Chip Resistor - Surface Mount ROHS"
+        (property "JLCPCB description" "62.5mW Thick Film Resistors 50V ±100ppm/℃ ±1% 10kΩ 0402 Chip Resistor - Surface Mount ROHS"
             (at 0 0 90)
             (layer "User.9")
@@
             (layers "F.Cu" "F.Paste" "F.Mask")
             (remove_unused_layers no)
-            (net 4 "line-2"))
+            (net 4 "line"))
         (pad "2" smd rect
             (at 0.43 0 90)
@@
             (layers "F.Cu" "F.Paste" "F.Mask")
             (remove_unused_layers no)
-            (net 7 "hv-1")))
+            (net 7 "hv")))
     (footprint "atopile:R0402-56259e"
         (layer "F.Cu")
@@
                     (size 0.7 0.7)
                     (thickness 0.2))))
-        (property "Value" "1kΩ ±1% 62.5mW"
+        (property "Value" "10kΩ ±1% 62.5mW"
             (at 0 4 90)
             (layer "F.Fab")
@@
                     (size 0.125 0.125)
                     (thickness 0.01875))))
-        (property "LCSC" "C11702"
-            (at 0 0 90)
-            (layer "User.9")
-            (hide yes)
-            (effects
-                (font
-                    (size 0.125 0.125)
-                    (thickness 0.01875))))
-        (property "Partnumber" "0402WGF1001TCE"
+        (property "LCSC" "C25744"
+            (at 0 0 90)
+            (layer "User.9")
+            (hide yes)
+            (effects
+                (font
+                    (size 0.125 0.125)
+                    (thickness 0.01875))))
+        (property "Partnumber" "0402WGF1002TCE"
             (at 0 0 90)
             (layer "User.9")
@@
                     (size 0.125 0.125)
                     (thickness 0.01875))))
-        (property "JLCPCB description" "62.5mW Thick Film Resistors 50V ±100ppm/℃ ±1% 1kΩ 0402 Chip Resistor - Surface Mount ROHS"
+        (property "JLCPCB description" "62.5mW Thick Film Resistors 50V ±100ppm/℃ ±1% 10kΩ 0402 Chip Resistor - Surface Mount ROHS"
             (at 0 0 90)
             (layer "User.9")
@@
             (layers "F.Cu" "F.Paste" "F.Mask")
             (remove_unused_layers no)
-            (net 2 "line"))
+            (net 2 "line-3"))
         (pad "2" smd rect
             (at 0.43 0 270)
@@
             (layers "F.Cu" "F.Paste" "F.Mask")
             (remove_unused_layers no)
-            (net 7 "hv-1")))
+            (net 7 "hv")))
     (segment
         (start 152.24 99.87)

Commit message: build and re-link layouts
Connections:
- U1 pad 1: line-2 -> line-3
- U1 pad 2: hv-1 -> hv
- U2 pad 1: line-1 -> line-2
- U2 pad 2: hv-1 -> hv
- U3 pad 1: hv -> hv-1
- U3 pad 2: line -> line-1
- U3 pad 3: line-3 -> line
- U3 pad 6: line-2 -> line-3
- U3 pad 7: line-1 -> line-2
- U3 pad 8: hv-1 -> hv
- U4 pad 1: line-3 -> line
- U4 pad 2: hv -> hv-1
- U5 pad 1: line -> line-1
- U5 pad 2: hv -> hv-1
- U6 pad 1: hv-1 -> hv
- U7 pad 1: hv -> hv-1
Changed lines of the file:
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@@
             (outputdirectory "")))
     (net 0 "")
-    (net 1 "line-1")
-    (net 2 "line-3")
-    (net 3 "hv-1")
-    (net 4 "line")
-    (net 5 "line-2")
+    (net 1 "line-2")
+    (net 2 "line")
+    (net 3 "hv")
+    (net 4 "line-1")
+    (net 5 "line-3")
     (net 6 "gnd")
-    (net 7 "hv")
+    (net 7 "hv-1")
     (net 8 "gnd-1")
     (footprint "atopile:R0402-56259e"
@@
             (layers "F.Cu" "F.Paste" "F.Mask")
             (remove_unused_layers no)
-            (net 1 "line-1"))
+            (net 1 "line-2"))
         (pad "2" smd rect
             (at 0.43 0 90)
@@
             (layers "F.Cu" "F.Paste" "F.Mask")
             (remove_unused_layers no)
-            (net 3 "hv-1")))
+            (net 3 "hv")))
     (footprint "atopile:SOIC-8_L4.9-W3.9-P1.27-LS6.0-TL-e13595"
         (layer "F.Cu")
@@
             (layers "F.Cu" "F.Paste" "F.Mask")
             (remove_unused_layers no)
-            (net 5 "line-2"))
+            (net 5 "line-3"))
         (pad "7" smd oval
             (at 2.74 -0.63 90)
@@
             (layers "F.Cu" "F.Paste" "F.Mask")
             (remove_unused_layers no)
-            (net 1 "line-1"))
+            (net 1 "line-2"))
         (pad "8" smd oval
             (at 2.74 -1.9 90)
@@
             (layers "F.Cu" "F.Paste" "F.Mask")
             (remove_unused_layers no)
-            (net 3 "hv-1"))
+            (net 3 "hv"))
         (pad "4" smd oval
             (at -2.74 1.91 90)
@@
             (layers "F.Cu" "F.Paste" "F.Mask")
             (remove_unused_layers no)
-            (net 2 "line-3"))
+            (net 2 "line"))
         (pad "2" smd oval
             (at -2.74 -0.63 90)
@@
             (layers "F.Cu" "F.Paste" "F.Mask")
             (remove_unused_layers no)
-            (net 4 "line"))
+            (net 4 "line-1"))
         (pad "1" smd oval
             (at -2.74 -1.9 90)
@@
             (layers "F.Cu" "F.Paste" "F.Mask")
             (remove_unused_layers no)
-            (net 7 "hv")))
+            (net 7 "hv-1")))
     (footprint "atopile:C0402-b3ef17"
         (layer "F.Cu")
@@
             (layers "F.Cu" "F.Paste" "F.Mask")
             (remove_unused_layers no)
-            (net 3 "hv-1"))
+            (net 3 "hv"))
         (pad "2" smd rect
             (at 0.55 0 180)
@@
             (layers "F.Cu" "F.Paste" "F.Mask")
             (remove_unused_layers no)
-            (net 7 "hv"))
+            (net 7 "hv-1"))
         (pad "2" smd rect
             (at 0.55 0 0)
@@
             (layers "F.Cu" "F.Paste" "F.Mask")
             (remove_unused_layers no)
-            (net 5 "line-2"))
+            (net 5 "line-3"))
         (pad "2" smd rect
             (at 0.43 0 270)
@@
             (layers "F.Cu" "F.Paste" "F.Mask")
             (remove_unused_layers no)
-            (net 3 "hv-1")))
+            (net 3 "hv")))
     (footprint "atopile:R0402-56259e"
         (layer "F.Cu")
@@
             (layers "F.Cu" "F.Paste" "F.Mask")
             (remove_unused_layers no)
-            (net 4 "line"))
+            (net 4 "line-1"))
         (pad "2" smd rect
             (at 0.43 0 90)
@@
             (layers "F.Cu" "F.Paste" "F.Mask")
             (remove_unused_layers no)
-            (net 7 "hv")))
+            (net 7 "hv-1")))
     (footprint "atopile:R0402-56259e"
         (layer "F.Cu")
@@
             (layers "F.Cu" "F.Paste" "F.Mask")
             (remove_unused_layers no)
-            (net 2 "line-3"))
+            (net 2 "line"))
         (pad "2" smd rect
             (at 0.43 0 270)
@@
             (layers "F.Cu" "F.Paste" "F.Mask")
             (remove_unused_layers no)
-            (net 7 "hv")))
+            (net 7 "hv-1")))
     (segment
         (start 152.24 99.87)
