File: elec/layout/isolator-24v-3v3/isolator-24v-3v3.kicad_pcb (KiCad board)
At the start: 2 copper layers, 13 parts, among them U1 470nF ±20% 16V X5R, U11 1kΩ ±1% 62.5mW, U12 2.2µF ±10% 25V X7R, U2 1kΩ ±1% 62.5mW, U3 1kΩ ±1% 62.5mW, U6 2.2µF ±20% 6.3V X5R, U7 10µF ±10% 25V X5R, U9 2.2µF ±10% 25V X7R

Commit message: remove default build, build everything locally
Connections:
- net out renamed FB

Commit message: add module builds back in to ato.yaml with mfg-data excluded in config
Connections:
- net FB renamed out
- DS1 pad 1: cathode -> cathode-1
- U1 pad 2: cathode -> cathode-1
- U10 pad 1: cathode-1 -> cathode
- U11 pad 1: cathode-1 -> cathode
- U3 pad 1: hv -> hv-1
- U4 pad 4: hv-1 -> hv
- U4 pad 5: hv-1 -> hv
- U4 pad 6: cathode -> cathode-1
- U5 pad 1: cathode -> cathode-1
- U5 pad 2: hv -> hv-1
- U6 pad 1: hv-1 -> hv
- U7 pad 1: hv -> hv-1
- U8 pad 1: hv-1 -> hv
- U9 pad 1: hv-1 -> hv
Changed lines of the file:
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@@
     (net 0 "")
     (net 1 "gnd-1")
-    (net 2 "cathode")
-    (net 3 "hv-1")
-    (net 4 "cathode-1")
+    (net 2 "cathode-1")
+    (net 3 "hv")
+    (net 4 "cathode")
     (net 5 "gnd")
     (net 6 "anode")
     (net 7 "CB")
-    (net 8 "hv")
-    (net 9 "FB")
+    (net 8 "hv-1")
+    (net 9 "out")
     (footprint "atopile:PWRM-TH_BXXXXS-2WR3-d8b2fb"
         (layer "F.Cu")
@@
             (layers "*.Cu" "*.Mask")
             (remove_unused_layers no)
-            (net 3 "hv-1"))
+            (net 3 "hv"))
         (pad "2" thru_hole circle
             (at -3.81 0 0)
@@
             (layers "F.Cu" "F.Paste" "F.Mask")
             (remove_unused_layers no)
-            (net 2 "cathode"))
+            (net 2 "cathode-1"))
         (pad "2" smd rect
             (at 1.17 0 0)
@@
             (layers "F.Cu" "F.Paste" "F.Mask")
             (remove_unused_layers no)
-            (net 4 "cathode-1"))
+            (net 4 "cathode"))
         (pad "2" smd rect
             (at 0.8 0 90)
@@
             (layers "F.Cu" "F.Paste" "F.Mask")
             (remove_unused_layers no)
-            (net 2 "cathode")))
+            (net 2 "cathode-1")))
     (footprint "lib:SOT-23-6_L2.9-W1.6-P0.95-LS2.8-BR"
         (layer "F.Cu")
@@
             (layers "F.Cu" "F.Paste" "F.Mask")
             (remove_unused_layers no)
-            (net 9 "FB"))
+            (net 9 "out"))
         (pad "4" smd rect
             (at -1.35 -0.95 0)
@@
             (layers "F.Cu" "F.Paste" "F.Mask")
             (remove_unused_layers no)
-            (net 3 "hv-1"))
+            (net 3 "hv"))
         (pad "5" smd rect
             (at -1.35 0 0)
@@
             (layers "F.Cu" "F.Paste" "F.Mask")
             (remove_unused_layers no)
-            (net 3 "hv-1"))
+            (net 3 "hv"))
         (pad "6" smd rect
             (at -1.35 0.95 0)
@@
             (layers "F.Cu" "F.Paste" "F.Mask")
             (remove_unused_layers no)
-            (net 2 "cathode"))
+            (net 2 "cathode-1"))
         (model "${KIPRJMOD}/../../../build/footprints/footprints.3dshapes/SOT-23-6_L2.9-W1.6-H1.5-LS2.8-P0.95.step"
             (offset
@@
             (layers "F.Cu" "F.Paste" "F.Mask")
             (remove_unused_layers no)
-            (net 8 "hv"))
+            (net 8 "hv-1"))
         (pad "2" smd rect
             (at 1 0 0)
@@
             (layers "F.Cu" "F.Paste" "F.Mask")
             (remove_unused_layers no)
-            (net 4 "cathode-1"))
+            (net 4 "cathode"))
         (pad "2" smd rect
             (at 0.43 0 0)
@@
             (layers "F.Cu" "F.Paste" "F.Mask")
             (remove_unused_layers no)
-            (net 3 "hv-1"))
+            (net 3 "hv"))
         (pad "2" smd rect
             (at 0.55 0 0)
@@
             (layers "F.Cu" "F.Paste" "F.Mask")
             (remove_unused_layers no)
-            (net 3 "hv-1"))
+            (net 3 "hv"))
         (pad "2" smd rect
             (at 1 0 0)
@@
             (layers "F.Cu" "F.Paste" "F.Mask")
             (remove_unused_layers no)
-            (net 8 "hv"))
+            (net 8 "hv-1"))
         (pad "2" smd rect
             (at 0.43 0 0)
@@
             (layers "F.Cu" "F.Paste" "F.Mask")
             (remove_unused_layers no)
-            (net 9 "FB")))
+            (net 9 "out")))
     (footprint "atopile:R0402-56259e"
         (layer "F.Cu")
@@
             (layers "F.Cu" "F.Paste" "F.Mask")
             (remove_unused_layers no)
-            (net 9 "FB"))
+            (net 9 "out"))
         (pad "2" smd rect
             (at 0.43 0 0)
@@
             (layers "F.Cu" "F.Paste" "F.Mask")
             (remove_unused_layers no)
-            (net 2 "cathode"))
+            (net 2 "cathode-1"))
         (pad "2" smd rect
             (at 1.6 0 0)
@@
             (layers "F.Cu" "F.Paste" "F.Mask")
             (remove_unused_layers no)
-            (net 8 "hv"))
+            (net 8 "hv-1"))
         (model "/Users/narayanpowderly/projects/hil-blocks/build/footprints/footprints.3dshapes/IND-SMD_L4.0-W4.0-H1.9.step"
             (offset

Commit message: add CAN isolator, cellsim cell
Connections:
- DS1 pad 1: cathode-1 -> cathode
- DS1 pad 2: gnd -> gnd-1
- U1 pad 2: cathode-1 -> cathode
- U10 pad 1: cathode -> cathode-1
- U11 pad 1: cathode -> cathode-1
- U11 pad 2: gnd-1 -> gnd
- U12 pad 2: gnd-1 -> gnd
- U2 pad 2: gnd -> gnd-1
- U3 pad 1: hv-1 -> hv
- U4 pad 2: gnd -> gnd-1
- U4 pad 4: hv -> hv-1
- U4 pad 5: hv -> hv-1
- U4 pad 6: cathode-1 -> cathode
- U5 pad 1: cathode-1 -> cathode
- U5 pad 2: hv-1 -> hv
- U6 pad 1: hv -> hv-1
- U6 pad 2: gnd -> gnd-1
- U7 pad 1: hv-1 -> hv
- U7 pad 2: gnd -> gnd-1
- U8 pad 1: hv -> hv-1
- U8 pad 2: gnd -> gnd-1
- U8 pad 4: gnd-1 -> gnd
- U9 pad 1: hv -> hv-1
- U9 pad 2: gnd -> gnd-1
Changed lines of the file:
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@@
             (outputdirectory "")))
     (net 0 "")
-    (net 1 "gnd-1")
-    (net 2 "cathode-1")
-    (net 3 "hv")
-    (net 4 "cathode")
-    (net 5 "gnd")
+    (net 1 "gnd")
+    (net 2 "cathode")
+    (net 3 "hv-1")
+    (net 4 "cathode-1")
+    (net 5 "gnd-1")
     (net 6 "anode")
     (net 7 "CB")
-    (net 8 "hv-1")
+    (net 8 "hv")
     (net 9 "out")
     (footprint "atopile:PWRM-TH_BXXXXS-2WR3-d8b2fb"
@@
             (layers "*.Cu" "*.Mask")
             (remove_unused_layers no)
-            (net 3 "hv"))
+            (net 3 "hv-1"))
         (pad "2" thru_hole circle
             (at -3.81 0 0)
@@
             (layers "*.Cu" "*.Mask")
             (remove_unused_layers no)
-            (net 5 "gnd"))
+            (net 5 "gnd-1"))
         (pad "4" thru_hole circle
             (at 1.27 0 0)
@@
             (layers "*.Cu" "*.Mask")
             (remove_unused_layers no)
-            (net 1 "gnd-1"))
+            (net 1 "gnd"))
         (pad "6" thru_hole circle
             (at 6.35 0 0)
@@
             (layers "F.Cu" "F.Paste" "F.Mask")
             (remove_unused_layers no)
-            (net 2 "cathode-1"))
+            (net 2 "cathode"))
         (pad "2" smd rect
             (at 1.17 0 0)
@@
             (layers "F.Cu" "F.Paste" "F.Mask")
             (remove_unused_layers no)
-            (net 5 "gnd"))
+            (net 5 "gnd-1"))
         (model "/Users/narayanpowderly/projects/hil-blocks/build/footprints/footprints.3dshapes/SOD-323_L1.7-W1.3-H1.1-LS2.5.step"
             (offset
@@
             (layers "F.Cu" "F.Paste" "F.Mask")
             (remove_unused_layers no)
-            (net 4 "cathode"))
+            (net 4 "cathode-1"))
         (pad "2" smd rect
             (at 0.8 0 90)
@@
             (layers "F.Cu" "F.Paste" "F.Mask")
             (remove_unused_layers no)
-            (net 2 "cathode-1")))
+            (net 2 "cathode")))
     (footprint "lib:SOT-23-6_L2.9-W1.6-P0.95-LS2.8-BR"
         (layer "F.Cu")
@@
             (layers "F.Cu" "F.Paste" "F.Mask")
             (remove_unused_layers no)
-            (net 5 "gnd"))
+            (net 5 "gnd-1"))
         (pad "3" smd rect
             (at 1.35 -0.95 0)
@@
             (layers "F.Cu" "F.Paste" "F.Mask")
             (remove_unused_layers no)
-            (net 3 "hv"))
+            (net 3 "hv-1"))
         (pad "5" smd rect
             (at -1.35 0 0)
@@
             (layers "F.Cu" "F.Paste" "F.Mask")
             (remove_unused_layers no)
-            (net 3 "hv"))
+            (net 3 "hv-1"))
         (pad "6" smd rect
             (at -1.35 0.95 0)
@@
             (layers "F.Cu" "F.Paste" "F.Mask")
             (remove_unused_layers no)
-            (net 2 "cathode-1"))
+            (net 2 "cathode"))
         (model "${KIPRJMOD}/../../../build/footprints/footprints.3dshapes/SOT-23-6_L2.9-W1.6-H1.5-LS2.8-P0.95.step"
             (offset
@@
             (layers "F.Cu" "F.Paste" "F.Mask")
             (remove_unused_layers no)
-            (net 8 "hv-1"))
+            (net 8 "hv"))
         (pad "2" smd rect
             (at 1 0 0)
@@
             (layers "F.Cu" "F.Paste" "F.Mask")
             (remove_unused_layers no)
-            (net 5 "gnd")))
+            (net 5 "gnd-1")))
     (footprint "atopile:R0402-56259e"
         (layer "F.Cu")
@@
             (layers "F.Cu" "F.Paste" "F.Mask")
             (remove_unused_layers no)
-            (net 4 "cathode"))
+            (net 4 "cathode-1"))
         (pad "2" smd rect
             (at 0.43 0 0)
@@
             (layers "F.Cu" "F.Paste" "F.Mask")
             (remove_unused_layers no)
-            (net 1 "gnd-1")))
+            (net 1 "gnd")))
     (footprint "atopile:C0402-b3ef17"
         (layer "F.Cu")
@@
             (layers "F.Cu" "F.Paste" "F.Mask")
             (remove_unused_layers no)
-            (net 3 "hv"))
+            (net 3 "hv-1"))
         (pad "2" smd rect
             (at 0.55 0 0)
@@
             (layers "F.Cu" "F.Paste" "F.Mask")
             (remove_unused_layers no)
-            (net 5 "gnd")))
+            (net 5 "gnd-1")))
     (footprint "atopile:C0805-3b2e55"
         (layer "F.Cu")
@@
             (layers "F.Cu" "F.Paste" "F.Mask")
             (remove_unused_layers no)
-            (net 3 "hv"))
+            (net 3 "hv-1"))
         (pad "2" smd rect
             (at 1 0 0)
@@
             (layers "F.Cu" "F.Paste" "F.Mask")
             (remove_unused_layers no)
-            (net 5 "gnd")))
+            (net 5 "gnd-1")))
     (footprint "atopile:R0402-56259e"
         (layer "F.Cu")
@@
             (layers "F.Cu" "F.Paste" "F.Mask")
             (remove_unused_layers no)
-            (net 8 "hv-1"))
+            (net 8 "hv"))
         (pad "2" smd rect
             (at 0.43 0 0)
@@
             (layers "F.Cu" "F.Paste" "F.Mask")
             (remove_unused_layers no)
-            (net 5 "gnd")))
+            (net 5 "gnd-1")))
     (footprint "lib:IND-SMD_L4.0-W4.0"
         (layer "F.Cu")
@@
             (layers "F.Cu" "F.Paste" "F.Mask")
             (remove_unused_layers no)
-            (net 2 "cathode-1"))
+            (net 2 "cathode"))
         (pad "2" smd rect
             (at 1.6 0 0)
@@
             (layers "F.Cu" "F.Paste" "F.Mask")
             (remove_unused_layers no)
-            (net 8 "hv-1"))
+            (net 8 "hv"))
         (model "/Users/narayanpowderly/projects/hil-blocks/build/footprints/footprints.3dshapes/IND-SMD_L4.0-W4.0-H1.9.step"
             (offset
@@
             (layers "F.Cu" "F.Paste" "F.Mask")
             (remove_unused_layers no)
-            (net 1 "gnd-1"))))
+            (net 1 "gnd"))))

Commit message: rebuild all modules
Connections:
- DS1 pad 2: gnd-1 -> gnd
- U11 pad 2: gnd -> gnd-1
- U12 pad 2: gnd -> gnd-1
- U2 pad 2: gnd-1 -> gnd
- U3 pad 1: hv -> hv-1
- U4 pad 2: gnd-1 -> gnd
- U4 pad 4: hv-1 -> hv
- U4 pad 5: hv-1 -> hv
- U5 pad 2: hv -> hv-1
- U6 pad 1: hv-1 -> hv
- U6 pad 2: gnd-1 -> gnd
- U7 pad 1: hv -> hv-1
- U7 pad 2: gnd-1 -> gnd
- U8 pad 1: hv-1 -> hv
- U8 pad 2: gnd-1 -> gnd
- U8 pad 4: gnd -> gnd-1
- U9 pad 1: hv-1 -> hv
- U9 pad 2: gnd-1 -> gnd
Changed lines of the file:
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@@
             (outputdirectory "")))
     (net 0 "")
-    (net 1 "gnd")
+    (net 1 "gnd-1")
     (net 2 "cathode")
-    (net 3 "hv-1")
+    (net 3 "hv")
     (net 4 "cathode-1")
-    (net 5 "gnd-1")
+    (net 5 "gnd")
     (net 6 "anode")
     (net 7 "CB")
-    (net 8 "hv")
+    (net 8 "hv-1")
     (net 9 "out")
     (footprint "atopile:PWRM-TH_BXXXXS-2WR3-d8b2fb"
@@
             (layers "*.Cu" "*.Mask")
             (remove_unused_layers no)
-            (net 3 "hv-1"))
+            (net 3 "hv"))
         (pad "2" thru_hole circle
             (at -3.81 0 0)
@@
             (layers "*.Cu" "*.Mask")
             (remove_unused_layers no)
-            (net 5 "gnd-1"))
+            (net 5 "gnd"))
         (pad "4" thru_hole circle
             (at 1.27 0 0)
@@
             (layers "*.Cu" "*.Mask")
             (remove_unused_layers no)
-            (net 1 "gnd"))
+            (net 1 "gnd-1"))
         (pad "6" thru_hole circle
             (at 6.35 0 0)
@@
             (layers "F.Cu" "F.Paste" "F.Mask")
             (remove_unused_layers no)
-            (net 5 "gnd-1"))
+            (net 5 "gnd"))
         (model "/Users/narayanpowderly/projects/hil-blocks/build/footprints/footprints.3dshapes/SOD-323_L1.7-W1.3-H1.1-LS2.5.step"
             (offset
@@
             (layers "F.Cu" "F.Paste" "F.Mask")
             (remove_unused_layers no)
-            (net 5 "gnd-1"))
+            (net 5 "gnd"))
         (pad "3" smd rect
             (at 1.35 -0.95 0)
@@
             (layers "F.Cu" "F.Paste" "F.Mask")
             (remove_unused_layers no)
-            (net 3 "hv-1"))
+            (net 3 "hv"))
         (pad "5" smd rect
             (at -1.35 0 0)
@@
             (layers "F.Cu" "F.Paste" "F.Mask")
             (remove_unused_layers no)
-            (net 3 "hv-1"))
+            (net 3 "hv"))
         (pad "6" smd rect
             (at -1.35 0.95 0)
@@
             (layers "F.Cu" "F.Paste" "F.Mask")
             (remove_unused_layers no)
-            (net 8 "hv"))
+            (net 8 "hv-1"))
         (pad "2" smd rect
             (at 1 0 0)
@@
             (layers "F.Cu" "F.Paste" "F.Mask")
             (remove_unused_layers no)
-            (net 5 "gnd-1")))
+            (net 5 "gnd")))
     (footprint "atopile:R0402-56259e"
         (layer "F.Cu")
@@
             (layers "F.Cu" "F.Paste" "F.Mask")
             (remove_unused_layers no)
-            (net 1 "gnd")))
+            (net 1 "gnd-1")))
     (footprint "atopile:C0402-b3ef17"
         (layer "F.Cu")
@@
             (layers "F.Cu" "F.Paste" "F.Mask")
             (remove_unused_layers no)
-            (net 3 "hv-1"))
+            (net 3 "hv"))
         (pad "2" smd rect
             (at 0.55 0 0)
@@
             (layers "F.Cu" "F.Paste" "F.Mask")
             (remove_unused_layers no)
-            (net 5 "gnd-1")))
+            (net 5 "gnd")))
     (footprint "atopile:C0805-3b2e55"
         (layer "F.Cu")
@@
             (layers "F.Cu" "F.Paste" "F.Mask")
             (remove_unused_layers no)
-            (net 3 "hv-1"))
+            (net 3 "hv"))
         (pad "2" smd rect
             (at 1 0 0)
@@
             (layers "F.Cu" "F.Paste" "F.Mask")
             (remove_unused_layers no)
-            (net 5 "gnd-1")))
+            (net 5 "gnd")))
     (footprint "atopile:R0402-56259e"
         (layer "F.Cu")
@@
             (layers "F.Cu" "F.Paste" "F.Mask")
             (remove_unused_layers no)
-            (net 8 "hv"))
+            (net 8 "hv-1"))
         (pad "2" smd rect
             (at 0.43 0 0)
@@
             (layers "F.Cu" "F.Paste" "F.Mask")
             (remove_unused_layers no)
-            (net 5 "gnd-1")))
+            (net 5 "gnd")))
     (footprint "lib:IND-SMD_L4.0-W4.0"
         (layer "F.Cu")
@@
             (layers "F.Cu" "F.Paste" "F.Mask")
             (remove_unused_layers no)
-            (net 8 "hv"))
+            (net 8 "hv-1"))
         (model "/Users/narayanpowderly/projects/hil-blocks/build/footprints/footprints.3dshapes/IND-SMD_L4.0-W4.0-H1.9.step"
             (offset
@@
             (layers "F.Cu" "F.Paste" "F.Mask")
             (remove_unused_layers no)
-            (net 1 "gnd"))))
+            (net 1 "gnd-1"))))

Commit message: Everything builds
Parts:
- U10: value (none) -> 2.75V
- U3: value 1kΩ ±1% 62.5mW -> infΩ infW
- U5: value (none) -> 10µH ±20%
Connections:
- DS1 pad 2: gnd -> gnd-1
- U11 pad 2: gnd-1 -> gnd
- U12 pad 2: gnd-1 -> gnd
- U2 pad 2: gnd -> gnd-1
- U4 pad 2: gnd -> gnd-1
- U6 pad 2: gnd -> gnd-1
- U7 pad 2: gnd -> gnd-1
- U8 pad 2: gnd -> gnd-1
- U8 pad 4: gnd-1 -> gnd
- U9 pad 2: gnd -> gnd-1
Changed lines of the file:
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@@
             (outputdirectory "")))
     (net 0 "")
-    (net 1 "gnd-1")
+    (net 1 "gnd")
     (net 2 "cathode")
     (net 3 "hv")
     (net 4 "cathode-1")
-    (net 5 "gnd")
+    (net 5 "gnd-1")
     (net 6 "anode")
     (net 7 "CB")
@@
             (layers "*.Cu" "*.Mask")
             (remove_unused_layers no)
-            (net 5 "gnd"))
+            (net 5 "gnd-1"))
         (pad "4" thru_hole circle
             (at 1.27 0 0)
@@
             (layers "*.Cu" "*.Mask")
             (remove_unused_layers no)
-            (net 1 "gnd-1"))
+            (net 1 "gnd"))
         (pad "6" thru_hole circle
             (at 6.35 0 0)
@@
             (layers "F.Cu" "F.Paste" "F.Mask")
             (remove_unused_layers no)
-            (net 5 "gnd"))
+            (net 5 "gnd-1"))
         (model "/Users/narayanpowderly/projects/hil-blocks/build/footprints/footprints.3dshapes/SOD-323_L1.7-W1.3-H1.1-LS2.5.step"
             (offset
@@
                     (size 1 1)
                     (thickness 0.15))))
-        (property "Value" ""
+        (property "Value" "2.75V"
             (at 0 4 0)
             (layer "F.Fab")
@@
             (layers "F.Cu" "F.Paste" "F.Mask")
             (remove_unused_layers no)
-            (net 5 "gnd"))
+            (net 5 "gnd-1"))
         (pad "3" smd rect
             (at 1.35 -0.95 0)
@@
             (layers "F.Cu" "F.Paste" "F.Mask")
             (remove_unused_layers no)
-            (net 5 "gnd")))
+            (net 5 "gnd-1")))
     (footprint "atopile:R0402-56259e"
         (layer "F.Cu")
@@
             (layers "F.Cu" "F.Paste" "F.Mask")
             (remove_unused_layers no)
-            (net 1 "gnd-1")))
+            (net 1 "gnd")))
     (footprint "atopile:C0402-b3ef17"
         (layer "F.Cu")
@@
             (layers "F.Cu" "F.Paste" "F.Mask")
             (remove_unused_layers no)
-            (net 5 "gnd")))
+            (net 5 "gnd-1")))
     (footprint "atopile:C0805-3b2e55"
         (layer "F.Cu")
@@
             (layers "F.Cu" "F.Paste" "F.Mask")
             (remove_unused_layers no)
-            (net 5 "gnd")))
+            (net 5 "gnd-1")))
     (footprint "atopile:R0402-56259e"
         (layer "F.Cu")
@@
                     (size 1 1)
                     (thickness 0.15))))
-        (property "Value" "1kΩ ±1% 62.5mW"
+        (property "Value" "infΩ infW"
             (at 0 4 0)
             (layer "F.Fab")
@@
                     (size 0.125 0.125)
                     (thickness 0.01875))))
-        (property "LCSC" "C11702"
-            (at 0 0 0)
-            (layer "User.9")
-            (hide yes)
-            (effects
-                (font
-                    (size 0.125 0.125)
-                    (thickness 0.01875))))
-        (property "Partnumber" "0402WGF1001TCE"
-            (at 0 0 0)
-            (layer "User.9")
-            (hide yes)
-            (effects
-                (font
-                    (size 0.125 0.125)
-                    (thickness 0.01875))))
-        (property "Manufacturer" "UNI-ROYAL(Uniroyal Elec)"
-            (at 0 0 0)
-            (layer "User.9")
-            (hide yes)
-            (effects
-                (font
-                    (size 0.125 0.125)
-                    (thickness 0.01875))))
-        (property "JLCPCB description" "62.5mW Thick Film Resistors 50V ±100ppm/℃ ±1% 1kΩ 0402 Chip Resistor - Surface Mount ROHS"
+        (property "LCSC" "C2906941"
+            (at 0 0 0)
+            (layer "User.9")
+            (hide yes)
+            (effects
+                (font
+                    (size 0.125 0.125)
+                    (thickness 0.01875))))
+        (property "Partnumber" "FRC0402J472 TS"
+            (at 0 0 0)
+            (layer "User.9")
+            (hide yes)
+            (effects
+                (font
+                    (size 0.125 0.125)
+                    (thickness 0.01875))))
+        (property "Manufacturer" "FOJAN"
+            (at 0 0 0)
+            (layer "User.9")
+            (hide yes)
+            (effects
+                (font
+                    (size 0.125 0.125)
+                    (thickness 0.01875))))
+        (property "JLCPCB description" "62.5mW Thick Film Resistors 50V ±100ppm/℃ ±5% 4.7kΩ 0402  Chip Resistor - Surface Mount ROHS"
             (at 0 0 0)
             (layer "User.9")
@@
             (layers "F.Cu" "F.Paste" "F.Mask")
             (remove_unused_layers no)
-            (net 5 "gnd")))
+            (net 5 "gnd-1")))
     (footprint "lib:IND-SMD_L4.0-W4.0"
         (layer "F.Cu")
@@
                     (size 1 1)
                     (thickness 0.15))))
-        (property "Value" ""
+        (property "Value" "10µH ±20%"
             (at 0 4 0)
             (layer "F.Fab")
@@
             (layers "F.Cu" "F.Paste" "F.Mask")
             (remove_unused_layers no)
-            (net 1 "gnd-1"))))
+            (net 1 "gnd"))))
