File: elec/layout/analog-in/analog-in.kicad_pcb (KiCad board)
At the start: 2 copper layers, 8 parts, among them U2 1µF ±10% 25V X5R, U3 10kΩ ±1% 62.5mW, U4 10kΩ ±1% 62.5mW, U5 BW CMRR Ib Vos GBW Iout SR, U6 10kΩ ±1% 100mW, U7 10kΩ ±1% 100mW

Commit message: HIL Building
Connections:
- net gnd renamed adc-line-2
- D1 pad 1: line-1 -> line-2
- U1 pad 10: line-2 -> line
- U1 pad 2: adc-line-1 -> adc-line-3
- U1 pad 6: adc-line-3 -> adc-line-1
- U1 pad 9: line -> line-3
- U5 pad 3: line-1 -> line-2
- U6 pad 1: line-1 -> line-2
- U7 pad 1: line-3 -> line-1
- U7 pad 2: line-1 -> line-2
Routing:
- net line-2: track 0.00 -> 8.99 mm
- net line-1: track 8.99 -> 0.00 mm
Changed lines of the file:
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@@
     (net 0 "")
     (net 1 "amplifier.opamp.footprint.pins[5].net-net")
-    (net 2 "line-1")
+    (net 2 "line-2")
     (net 3 "amplifier.opamp.footprint.pins[6].net-net")
-    (net 4 "adc-line-3")
+    (net 4 "adc-line-1")
     (net 5 "adc-line-4")
-    (net 6 "line")
-    (net 7 "gnd")
-    (net 8 "line-2")
-    (net 9 "adc-line-1")
+    (net 6 "line-3")
+    (net 7 "adc-line-2")
+    (net 8 "line")
+    (net 9 "adc-line-3")
     (net 10 "amplifier.opamp.footprint.pins[4].net-net")
-    (net 11 "line-3")
+    (net 11 "line-1")
     (net 12 "inverting_input")
     (net 13 "adc-line")
@@
             (layers "F.Cu" "F.Paste" "F.Mask")
             (remove_unused_layers no)
-            (net 7 "gnd"))
+            (net 7 "adc-line-2"))
         (pad "1" smd rect
             (at -2.36 0 90)
@@
             (layers "F.Cu" "F.Paste" "F.Mask")
             (remove_unused_layers no)
-            (net 2 "line-1")))
+            (net 2 "line-2")))
     (footprint "atopile:SOIC-8_L5.0-W4.0-P1.27-LS6.0-BL-294f77"
         (layer "F.Cu")
@@
             (layers "F.Cu" "F.Paste" "F.Mask")
             (remove_unused_layers no)
-            (net 2 "line-1"))
+            (net 2 "line-2"))
         (pad "4" smd oval
             (at 1.9 2.71 90)
@@
             (layers "F.Cu" "F.Paste" "F.Mask")
             (remove_unused_layers no)
-            (net 7 "gnd"))
+            (net 7 "adc-line-2"))
         (pad "5" smd oval
             (at 1.9 -2.71 90)
@@
             (layers "F.Cu" "F.Paste" "F.Mask")
             (remove_unused_layers no)
-            (net 7 "gnd"))
+            (net 7 "adc-line-2"))
         (pad "2" smd rect
             (at 0.43 0 270)
@@
             (layers "F.Cu" "F.Paste" "F.Mask")
             (remove_unused_layers no)
-            (net 2 "line-1"))
+            (net 2 "line-2"))
         (pad "1" smd rect
             (at -0.75 0 90)
@@
             (layers "F.Cu" "F.Paste" "F.Mask")
             (remove_unused_layers no)
-            (net 11 "line-3")))
+            (net 11 "line-1")))
     (footprint "atopile:R0603-ebcab9"
         (layer "F.Cu")
@@
             (layers "F.Cu" "F.Paste" "F.Mask")
             (remove_unused_layers no)
-            (net 7 "gnd"))
+            (net 7 "adc-line-2"))
         (pad "1" smd rect
             (at -0.75 0 90)
@@
             (layers "F.Cu" "F.Paste" "F.Mask")
             (remove_unused_layers no)
-            (net 2 "line-1")))
+            (net 2 "line-2")))
     (footprint "atopile:MSOP-10_L3.0-W3.0-P0.50-LS5.0-BL-752175"
         (layer "F.Cu")
@@
             (layers "F.Cu" "F.Paste" "F.Mask")
             (remove_unused_layers no)
-            (net 7 "gnd"))
+            (net 7 "adc-line-2"))
         (pad "2" smd oval
             (at -0.5 2.11 90)
@@
             (layers "F.Cu" "F.Paste" "F.Mask")
             (remove_unused_layers no)
-            (net 9 "adc-line-1"))
+            (net 9 "adc-line-3"))
         (pad "3" smd oval
             (at 0 2.11 90)
@@
             (layers "F.Cu" "F.Paste" "F.Mask")
             (remove_unused_layers no)
-            (net 7 "gnd"))
+            (net 7 "adc-line-2"))
         (pad "4" smd oval
             (at 0.5 2.11 90)
@@
             (layers "F.Cu" "F.Paste" "F.Mask")
             (remove_unused_layers no)
-            (net 8 "line-2"))
+            (net 8 "line"))
         (pad "9" smd oval
             (at -0.5 -2.11 90)
@@
             (layers "F.Cu" "F.Paste" "F.Mask")
             (remove_unused_layers no)
-            (net 6 "line"))
+            (net 6 "line-3"))
         (pad "8" smd oval
             (at 0 -2.11 90)
@@
             (layers "F.Cu" "F.Paste" "F.Mask")
             (remove_unused_layers no)
-            (net 4 "adc-line-3")))
+            (net 4 "adc-line-1")))
     (footprint "atopile:C0402-b3ef17"
         (layer "F.Cu")
@@
             (layers "F.Cu" "F.Paste" "F.Mask")
             (remove_unused_layers no)
-            (net 7 "gnd")))
+            (net 7 "adc-line-2")))
     (via
         (at 131.8 106.9)
