File: elec/layout/analog-in-4ch/analog-in-4ch.kicad_pcb (KiCad board)
At the start: 2 copper layers, 2 parts, among them U1 100nF ±10% 16V X7R

Commit message: Layout of amplifier-4ch
Connections:
- net dac-line renamed VOUTC
- net dac-line-1 renamed line
Changed lines of the file:
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@@
     (net 1 "VOUTB")
     (net 2 "SDA")
-    (net 3 "dac-line-1")
+    (net 3 "line")
     (net 4 "RDY_BSYh")
     (net 5 "gnd")
-    (net 6 "dac-line")
+    (net 6 "VOUTC")
     (net 7 "VOUTA")
     (net 8 "SCL")
@@
             (layers "F.Cu" "F.Paste" "F.Mask")
             (remove_unused_layers no)
-            (net 6 "dac-line"))
+            (net 6 "VOUTC"))
         (pad "9" smd rect
             (at 2.45 -0.5 0)
@@
             (layers "F.Cu" "F.Paste" "F.Mask")
             (remove_unused_layers no)
-            (net 3 "dac-line-1"))
+            (net 3 "line"))
         (pad "10" smd rect
             (at 2.45 -1 0)

Commit message: update syntax, delete vendored packages
Connections:
- U2 pad 6: VOUTA -> line
- U2 pad 9: line -> VOUTD
Changed lines of the file:
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@@
     (net 1 "VOUTB")
     (net 2 "SDA")
-    (net 3 "line")
+    (net 3 "VOUTD")
     (net 4 "RDY_BSYh")
     (net 5 "gnd")
     (net 6 "VOUTC")
-    (net 7 "VOUTA")
+    (net 7 "line")
     (net 8 "SCL")
     (net 9 "hv")
@@
             (layers "F.Cu" "F.Paste" "F.Mask")
             (remove_unused_layers no)
-            (net 7 "VOUTA"))
+            (net 7 "line"))
         (pad "7" smd rect
             (at 2.45 0.5 0)
@@
             (layers "F.Cu" "F.Paste" "F.Mask")
             (remove_unused_layers no)
-            (net 3 "line"))
+            (net 3 "VOUTD"))
         (pad "10" smd rect
             (at 2.45 -1 0)

Commit message: build and re-link layouts
Connections:
- net VOUTB renamed dac-line-1
- net VOUTC renamed dac-line-2
- net line renamed dac-line
Changed lines of the file:
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@@
             (outputdirectory "")))
     (net 0 "")
-    (net 1 "VOUTB")
+    (net 1 "dac-line-1")
     (net 2 "SDA")
     (net 3 "VOUTD")
     (net 4 "RDY_BSYh")
     (net 5 "gnd")
-    (net 6 "VOUTC")
-    (net 7 "line")
+    (net 6 "dac-line-2")
+    (net 7 "dac-line")
     (net 8 "SCL")
     (net 9 "hv")
@@
             (layers "F.Cu" "F.Paste" "F.Mask")
             (remove_unused_layers no)
-            (net 7 "line"))
+            (net 7 "dac-line"))
         (pad "7" smd rect
             (at 2.45 0.5 0)
@@
             (layers "F.Cu" "F.Paste" "F.Mask")
             (remove_unused_layers no)
-            (net 1 "VOUTB"))
+            (net 1 "dac-line-1"))
         (pad "8" smd rect
             (at 2.45 0 0)
@@
             (layers "F.Cu" "F.Paste" "F.Mask")
             (remove_unused_layers no)
-            (net 6 "VOUTC"))
+            (net 6 "dac-line-2"))
         (pad "9" smd rect
             (at 2.45 -0.5 0)

Commit message: all modules building
Connections:
- net dac-line renamed VOUTA
- net dac-line-1 renamed VOUTB
- net dac-line-2 renamed VOUTC
Changed lines of the file:
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@@
             (outputdirectory "")))
     (net 0 "")
-    (net 1 "dac-line-1")
+    (net 1 "VOUTB")
     (net 2 "SDA")
     (net 3 "VOUTD")
     (net 4 "RDY_BSYh")
     (net 5 "gnd")
-    (net 6 "dac-line-2")
-    (net 7 "dac-line")
+    (net 6 "VOUTC")
+    (net 7 "VOUTA")
     (net 8 "SCL")
     (net 9 "hv")
@@
                     (size 0.125 0.125)
                     (thickness 0.01875))))
+        (property "Datasheet" "https://www.lcsc.com/datasheet/lcsc_datasheet_1811151641_Microchip-Tech-MCP4728-E-UN_C108207.pdf"
+            (at 0 0 0)
+            (layer "User.9")
+            (hide yes)
+            (effects
+                (font
+                    (size 0.125 0.125)
+                    (thickness 0.01875))))
         (attr smd)
         (fp_line
@@
             (layers "F.Cu" "F.Paste" "F.Mask")
             (remove_unused_layers no)
-            (net 7 "dac-line"))
+            (net 7 "VOUTA"))
         (pad "7" smd rect
             (at 2.45 0.5 0)
@@
             (layers "F.Cu" "F.Paste" "F.Mask")
             (remove_unused_layers no)
-            (net 1 "dac-line-1"))
+            (net 1 "VOUTB"))
         (pad "8" smd rect
             (at 2.45 0 0)
@@
             (layers "F.Cu" "F.Paste" "F.Mask")
             (remove_unused_layers no)
-            (net 6 "dac-line-2"))
+            (net 6 "VOUTC"))
         (pad "9" smd rect
             (at 2.45 -0.5 0)

Commit message: HIL Building
Connections:
- net VOUTB renamed dac-line-1
- net VOUTD renamed dac-line
Changed lines of the file:
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@@
             (outputdirectory "")))
     (net 0 "")
-    (net 1 "VOUTB")
+    (net 1 "dac-line-1")
     (net 2 "SDA")
-    (net 3 "VOUTD")
+    (net 3 "dac-line")
     (net 4 "RDY_BSYh")
     (net 5 "gnd")
@@
             (layers "F.Cu" "F.Paste" "F.Mask")
             (remove_unused_layers no)
-            (net 1 "VOUTB"))
+            (net 1 "dac-line-1"))
         (pad "8" smd rect
             (at 2.45 0 0)
@@
             (layers "F.Cu" "F.Paste" "F.Mask")
             (remove_unused_layers no)
-            (net 3 "VOUTD"))
+            (net 3 "dac-line"))
         (pad "10" smd rect
             (at 2.45 -1 0)

Commit message: build with latest main
Parts:
- removed U1: 100nF ±10% 16V X7R, atopile:C0402-b3ef17
- removed U2: , atopile:MSOP-10_L3.0-W3.0-P0.50-LS5.0-TL-ee3c6b
