File: elec/layout/controller-cm4/cm4.kicad_pcb (KiCad board)
At the start: 4 copper layers, 10 parts

Commit message: all modules building
Connections:
- net cm4-line-10 renamed Y
- net cm4.hdi_b-pins[26] renamed pins[26]
- net pins[40] renamed cm4.hdi_b-pins[40]
- net pins[46] renamed cm4-pins[46]-1
- CN1 pad 12: cm4-line-8 -> cm4-line-2
- CN1 pad 15: line-2 -> line
- CN1 pad 17: line-3 -> line-2
- CN1 pad 22: pins[43] -> cm4-line-4
- CN1 pad 23: cm4-line-6 -> pins[45]
- CN1 pad 24: pins[47] -> cm4-line-8
- CN1 pad 25: cm4-line-7 -> cm4-line-6
- CN1 pad 27: line-1 -> line-3
- CN1 pad 28: pins[55] -> cm4-line-5
- CN1 pad 29: cm4-line-1 -> pins[57]
- CN1 pad 75: cm4-line-4 -> pins[50]
- CN1 pad 77: cm4-line-3 -> cm4-pins[46]
- CN1 pad 78: cm4-line-2 -> cm4-line-3
- CN1 pad 80: cm4-line-5 -> cm4-pins[40]
- CN1 pad 82: line -> line-1
- CN1 pad 86: cm4-line-9 -> cm4-line-7
- CN1 pad 87: cm4-pins[26] -> cm4-line-1
- D1 pad 1: cm4-cathode-1 -> cm4-cathode
- D2 pad 1: cm4-cathode -> cm4-cathode-1
- R1 pad 1: cm4-cathode-1 -> cm4-cathode
- R2 pad 1: cm4-cathode -> cm4-cathode-1
- R3 pad 2: rj45-anode -> rj45-anode-1
- R4 pad 2: rj45-anode-1 -> rj45-anode
- RJ1 pad 12: rj45-anode -> rj45-anode-1
- RJ1 pad 13: rj45-anode-1 -> rj45-anode
Changed lines of the file:
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@@
     (net 0 "")
     (net 1 "pins[20]")
-    (net 2 "cm4-line-2")
+    (net 2 "cm4-line-3")
     (net 3 "cm4.hdi_b-pins[62]")
     (net 4 "cm4.hdi_a-pins[74]")
-    (net 5 "pins[43]")
-    (net 6 "pins[47]")
+    (net 5 "cm4-line-4")
+    (net 6 "cm4-line-8")
     (net 7 "cm4.hdi_b-pins[74]")
     (net 8 "cm4.hdi_a-pins[62]")
-    (net 9 "line-1")
+    (net 9 "line-3")
     (net 10 "pins[18]")
-    (net 11 "pins[46]")
+    (net 11 "cm4-pins[46]-1")
     (net 12 "pins[67]")
-    (net 13 "cm4-line-9")
+    (net 13 "cm4-line-7")
     (net 14 "UART_TX")
     (net 15 "pins[5]")
     (net 16 "VCC_5V")
     (net 17 "UART_RX")
-    (net 18 "pins[55]")
+    (net 18 "cm4-line-5")
     (net 19 "HDMI0_D1_N")
     (net 20 "HDMI0_D2_N")
@@
     (net 28 "pins[90]")
     (net 29 "pins[82]")
-    (net 30 "line-2")
+    (net 30 "line")
     (net 31 "pins[58]")
-    (net 32 "cm4-line-1")
+    (net 32 "pins[57]")
     (net 33 "HDMI0_D0_P")
     (net 34 "pins[44]")
@@
     (net 36 "cm4.hdi_a-pins[88]")
     (net 37 "HDMI1_D2_P")
-    (net 38 "line")
+    (net 38 "line-1")
     (net 39 "HDMI1_CK_N")
     (net 40 "pins[79]")
@@
     (net 46 "pins[33]")
     (net 47 "pins[66]")
-    (net 48 "cm4-line-4")
+    (net 48 "pins[50]")
     (net 49 "cm4.hdi_b-pins[88]")
     (net 50 "cm4.hdi_b-pins[92]")
     (net 51 "pins[37]")
-    (net 52 "cm4-line-8")
+    (net 52 "cm4-line-2")
     (net 53 "pins[29]")
     (net 54 "pins[49]")
@@
     (net 67 "HDMI0_D1_P")
     (net 68 "rj45.connector-net-1")
-    (net 70 "cm4-line-10")
-    (net 71 "cm4-cathode-1")
-    (net 73 "cm4-cathode")
-    (net 74 "rj45-anode-1")
+    (net 70 "Y")
+    (net 71 "cm4-cathode")
+    (net 73 "cm4-cathode-1")
+    (net 74 "rj45-anode")
     (net 75 "rj45.connector-net")
     (net 76 "N_C_")
-    (net 77 "rj45-anode")
-    (net 78 "cm4-line-6")
+    (net 77 "rj45-anode-1")
+    (net 78 "pins[45]")
     (net 79 "pins[3]")
     (net 80 "HDMI0_CK_P")
@@
     (net 85 "pins[41]")
     (net 86 "pins[70]")
-    (net 87 "cm4-line-7")
+    (net 87 "cm4-line-6")
     (net 88 "cm4.hdi_a-pins[98]")
     (net 89 "cm4.hdi_b-pins[34]")
@@
     (net 93 "HDMI1_D2_N")
     (net 94 "HDMI0_CEC")
-    (net 95 "pins[40]")
+    (net 95 "cm4.hdi_b-pins[40]")
     (net 96 "pins[91]")
     (net 97 "SCL")
@@
     (net 101 "HDMI1_CK_P")
     (net 102 "I2S_SCK")
-    (net 103 "cm4.hdi_b-pins[26]")
-    (net 104 "cm4-pins[26]")
+    (net 103 "pins[26]")
+    (net 104 "cm4-line-1")
     (net 105 "pins[11]")
     (net 106 "pins[27]")
@@
     (net 121 "HDMI0_D2_P")
     (net 122 "pins[22]")
-    (net 123 "line-3")
+    (net 123 "line-2")
     (net 124 "pins[80]")
     (net 125 "cm4.hdi_b-pins[94]")
@@
     (net 127 "pins[96]")
     (net 128 "pins[14]")
-    (net 129 "cm4-line-3")
+    (net 129 "cm4-pins[46]")
     (net 130 "cm4.hdi_a-pins[94]")
     (net 131 "cm4.hdi_a-pins[34]")
-    (net 132 "cm4-line-5")
+    (net 132 "cm4-pins[40]")
     (net 133 "pins[61]")
     (net 134 "cm4.hdi_b-pins[56]")
@@
             (layers "*.Cu" "*.Mask")
             (remove_unused_layers no)
-            (net 77 "rj45-anode"))
+            (net 77 "rj45-anode-1"))
         (pad "13" thru_hole circle
             (at -4.09 -6.89 90)
@@
             (layers "*.Cu" "*.Mask")
             (remove_unused_layers no)
-            (net 74 "rj45-anode-1"))
+            (net 74 "rj45-anode"))
         (pad "14" thru_hole circle
             (at -6.63 -6.89 90)
@@
             (layers "F.Cu" "F.Paste" "F.Mask")
             (remove_unused_layers no)
-            (net 73 "cm4-cathode"))
+            (net 73 "cm4-cathode-1"))
         (pad "2" smd rect
             (at 0.8 0 180)
@@
             (layers "F.Cu" "F.Paste" "F.Mask")
             (remove_unused_layers no)
-            (net 73 "cm4-cathode"))
+            (net 73 "cm4-cathode-1"))
         (pad "2" smd rect
             (at 0.43 0 270)
@@
             (layers "F.Cu" "F.Paste" "F.Mask")
             (remove_unused_layers no)
-            (net 70 "cm4-line-10")))
+            (net 70 "Y")))
     (footprint "atopile:LED0603-RD-YELLOW-5af84a"
         (layer "F.Cu")
@@
             (layers "F.Cu" "F.Paste" "F.Mask")
             (remove_unused_layers no)
-            (net 71 "cm4-cathode-1"))
+            (net 71 "cm4-cathode"))
         (pad "2" smd rect
             (at 0.8 0 180)
@@
             (layers "F.Cu" "F.Paste" "F.Mask")
             (remove_unused_layers no)
-            (net 70 "cm4-line-10"))
+            (net 70 "Y"))
         (pad "5" smd rect
             (at -1.3 0.95 90)
@@
             (layers "F.Cu" "F.Paste" "F.Mask")
             (remove_unused_layers no)
-            (net 74 "rj45-anode-1")))
+            (net 74 "rj45-anode")))
     (footprint "atopile:CONN-SMD_DF40C-100DS-0.4V-51-ceffa9"
         (layer "F.Cu")
@@
             (layers "F.Cu" "F.Paste" "F.Mask")
             (remove_unused_layers no)
-            (net 11 "pins[46]"))
+            (net 11 "cm4-pins[46]-1"))
         (pad "78" smd rect
             (at 1 -1.6 0)
@@
             (layers "F.Cu" "F.Paste" "F.Mask")
             (remove_unused_layers no)
-            (net 95 "pins[40]"))
+            (net 95 "cm4.hdi_b-pins[40]"))
         (pad "81" smd rect
             (at 2.2 -1.6 0)
@@
             (layers "F.Cu" "F.Paste" "F.Mask")
             (remove_unused_layers no)
-            (net 103 "cm4.hdi_b-pins[26]"))
+            (net 103 "pins[26]"))
         (pad "88" smd rect
             (at 5 -1.6 0)
@@
             (layers "F.Cu" "F.Paste" "F.Mask")
             (remove_unused_layers no)
-            (net 77 "rj45-anode")))
+            (net 77 "rj45-anode-1")))
     (footprint "atopile:R0402-56259e"
         (layer "F.Cu")
@@
             (layers "F.Cu" "F.Paste" "F.Mask")
             (remove_unused_layers no)
-            (net 71 "cm4-cathode-1"))
+            (net 71 "cm4-cathode"))
         (pad "2" smd rect
             (at 0.43 0 270)
@@
             (layers "F.Cu" "F.Paste" "F.Mask")
             (remove_unused_layers no)
-            (net 52 "cm4-line-8"))
+            (net 52 "cm4-line-2"))
         (pad "13" smd rect
             (at 5 1.6 0)
@@
             (layers "F.Cu" "F.Paste" "F.Mask")
             (remove_unused_layers no)
-            (net 30 "line-2"))
+            (net 30 "line"))
         (pad "16" smd rect
             (at 3.8 1.6 0)
@@
             (layers "F.Cu" "F.Paste" "F.Mask")
             (remove_unused_layers no)
-            (net 123 "line-3"))
+            (net 123 "line-2"))
         (pad "18" smd rect
             (at 3 1.6 0)
@@
             (layers "F.Cu" "F.Paste" "F.Mask")
             (remove_unused_layers no)
-            (net 5 "pins[43]"))
+            (net 5 "cm4-line-4"))
         (pad "23" smd rect
             (at 1 1.6 0)
@@
             (layers "F.Cu" "F.Paste" "F.Mask")
             (remove_unused_layers no)
-            (net 78 "cm4-line-6"))
+            (net 78 "pins[45]"))
         (pad "24" smd rect
             (at 0.6 1.6 0)
@@
             (layers "F.Cu" "F.Paste" "F.Mask")
             (remove_unused_layers no)
-            (net 6 "pins[47]"))
+            (net 6 "cm4-line-8"))
         (pad "25" smd rect
             (at 0.2 1.6 0)
@@
             (layers "F.Cu" "F.Paste" "F.Mask")
             (remove_unused_layers no)
-            (net 87 "cm4-line-7"))
+            (net 87 "cm4-line-6"))
         (pad "26" smd rect
             (at -0.2 1.6 0)
@@
             (layers "F.Cu" "F.Paste" "F.Mask")
             (remove_unused_layers no)
-            (net 9 "line-1"))
+            (net 9 "line-3"))
         (pad "28" smd rect
             (at -1 1.6 0)
@@
             (layers "F.Cu" "F.Paste" "F.Mask")
             (remove_unused_layers no)
-            (net 18 "pins[55]"))
+            (net 18 "cm4-line-5"))
         (pad "29" smd rect
             (at -1.4 1.6 0)
@@
             (layers "F.Cu" "F.Paste" "F.Mask")
             (remove_unused_layers no)
-            (net 32 "cm4-line-1"))
+            (net 32 "pins[57]"))
         (pad "30" smd rect
             (at -1.8 1.6 0)
@@
             (layers "F.Cu" "F.Paste" "F.Mask")
             (remove_unused_layers no)
-            (net 48 "cm4-line-4"))
+            (net 48 "pins[50]"))
         (pad "76" smd rect
             (at 0.2 -1.6 0)
@@
             (layers "F.Cu" "F.Paste" "F.Mask")
             (remove_unused_layers no)
-            (net 129 "cm4-line-3"))
+            (net 129 "cm4-pins[46]"))
         (pad "78" smd rect
             (at 1 -1.6 0)
@@
             (layers "F.Cu" "F.Paste" "F.Mask")
             (remove_unused_layers no)
-            (net 2 "cm4-line-2"))
+            (net 2 "cm4-line-3"))
         (pad "79" smd rect
             (at 1.4 -1.6 0)
@@
             (layers "F.Cu" "F.Paste" "F.Mask")
             (remove_unused_layers no)
-            (net 132 "cm4-line-5"))
+            (net 132 "cm4-pins[40]"))
         (pad "81" smd rect
             (at 2.2 -1.6 0)
@@
             (layers "F.Cu" "F.Paste" "F.Mask")
             (remove_unused_layers no)
-            (net 38 "line"))
+            (net 38 "line-1"))
         (pad "83" smd rect
             (at 3 -1.6 0)
@@
             (layers "F.Cu" "F.Paste" "F.Mask")
             (remove_unused_layers no)
-            (net 13 "cm4-line-9"))
+            (net 13 "cm4-line-7"))
         (pad "87" smd rect
             (at 4.6 -1.6 0)
@@
             (layers "F.Cu" "F.Paste" "F.Mask")
             (remove_unused_layers no)
-            (net 104 "cm4-pins[26]"))
+            (net 104 "cm4-line-1"))
         (pad "88" smd rect
             (at 5 -1.6 0)

Commit message: HIL Building
Connections:
- net cm4-line-8 renamed pins[47]
- net cm4-pins[46]-1 renamed pins[46]
- net cm4.hdi_b-pins[40] renamed pins[40]
- net pins[26] renamed cm4.hdi_b-pins[26]
- CN1 pad 12: cm4-line-2 -> cm4-line-3
- CN1 pad 15: line -> line-2
- CN1 pad 17: line-2 -> line-3
- CN1 pad 22: cm4-line-4 -> cm4-line-5
- CN1 pad 25: cm4-line-6 -> cm4-line-1
- CN1 pad 27: line-3 -> line
- CN1 pad 28: cm4-line-5 -> pins[55]
- CN1 pad 77: cm4-pins[46] -> cm4-line-4
- CN1 pad 78: cm4-line-3 -> cm4-line-6
- CN1 pad 80: cm4-pins[40] -> cm4-line-2
- CN1 pad 85: cm4-line -> pins[30]
- CN1 pad 86: cm4-line-7 -> cm4-line
- CN1 pad 87: cm4-line-1 -> cm4-pins[26]
- D1 pad 1: cm4-cathode -> cm4-cathode-1
- D2 pad 1: cm4-cathode-1 -> cm4-cathode
- R1 pad 1: cm4-cathode -> cm4-cathode-1
- R2 pad 1: cm4-cathode-1 -> cm4-cathode
- R3 pad 2: rj45-anode-1 -> rj45-anode
- R4 pad 2: rj45-anode -> rj45-anode-1
- RJ1 pad 12: rj45-anode-1 -> rj45-anode
- RJ1 pad 13: rj45-anode -> rj45-anode-1
- RJ1 pad P1: rj45.connector-net-1 -> rj45.connector-net
- RJ1 pad P10: rj45.connector-net -> rj45.connector-net-1
Changed lines of the file:
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@@
     (net 0 "")
     (net 1 "pins[20]")
-    (net 2 "cm4-line-3")
+    (net 2 "cm4-line-6")
     (net 3 "cm4.hdi_b-pins[62]")
     (net 4 "cm4.hdi_a-pins[74]")
-    (net 5 "cm4-line-4")
-    (net 6 "cm4-line-8")
+    (net 5 "cm4-line-5")
+    (net 6 "pins[47]")
     (net 7 "cm4.hdi_b-pins[74]")
     (net 8 "cm4.hdi_a-pins[62]")
-    (net 9 "line-3")
+    (net 9 "line")
     (net 10 "pins[18]")
-    (net 11 "cm4-pins[46]-1")
+    (net 11 "pins[46]")
     (net 12 "pins[67]")
-    (net 13 "cm4-line-7")
+    (net 13 "cm4-line")
     (net 14 "UART_TX")
     (net 15 "pins[5]")
     (net 16 "VCC_5V")
     (net 17 "UART_RX")
-    (net 18 "cm4-line-5")
+    (net 18 "pins[55]")
     (net 19 "HDMI0_D1_N")
     (net 20 "HDMI0_D2_N")
@@
     (net 28 "pins[90]")
     (net 29 "pins[82]")
-    (net 30 "line")
+    (net 30 "line-2")
     (net 31 "pins[58]")
     (net 32 "pins[57]")
@@
     (net 50 "cm4.hdi_b-pins[92]")
     (net 51 "pins[37]")
-    (net 52 "cm4-line-2")
+    (net 52 "cm4-line-3")
     (net 53 "pins[29]")
     (net 54 "pins[49]")
@@
     (net 66 "cm4.hdi_a-pins[15]")
     (net 67 "HDMI0_D1_P")
-    (net 68 "rj45.connector-net-1")
+    (net 68 "rj45.connector-net")
     (net 70 "Y")
-    (net 71 "cm4-cathode")
-    (net 73 "cm4-cathode-1")
-    (net 74 "rj45-anode")
-    (net 75 "rj45.connector-net")
+    (net 71 "cm4-cathode-1")
+    (net 73 "cm4-cathode")
+    (net 74 "rj45-anode-1")
+    (net 75 "rj45.connector-net-1")
     (net 76 "N_C_")
-    (net 77 "rj45-anode-1")
+    (net 77 "rj45-anode")
     (net 78 "pins[45]")
     (net 79 "pins[3]")
@@
     (net 85 "pins[41]")
     (net 86 "pins[70]")
-    (net 87 "cm4-line-6")
+    (net 87 "cm4-line-1")
     (net 88 "cm4.hdi_a-pins[98]")
     (net 89 "cm4.hdi_b-pins[34]")
@@
     (net 93 "HDMI1_D2_N")
     (net 94 "HDMI0_CEC")
-    (net 95 "cm4.hdi_b-pins[40]")
+    (net 95 "pins[40]")
     (net 96 "pins[91]")
     (net 97 "SCL")
@@
     (net 101 "HDMI1_CK_P")
     (net 102 "I2S_SCK")
-    (net 103 "pins[26]")
-    (net 104 "cm4-line-1")
+    (net 103 "cm4.hdi_b-pins[26]")
+    (net 104 "cm4-pins[26]")
     (net 105 "pins[11]")
     (net 106 "pins[27]")
@@
     (net 118 "pins[72]")
     (net 119 "HDMI0_CK_N")
-    (net 120 "cm4-line")
+    (net 120 "pins[30]")
     (net 121 "HDMI0_D2_P")
     (net 122 "pins[22]")
-    (net 123 "line-2")
+    (net 123 "line-3")
     (net 124 "pins[80]")
     (net 125 "cm4.hdi_b-pins[94]")
@@
     (net 127 "pins[96]")
     (net 128 "pins[14]")
-    (net 129 "cm4-pins[46]")
+    (net 129 "cm4-line-4")
     (net 130 "cm4.hdi_a-pins[94]")
     (net 131 "cm4.hdi_a-pins[34]")
-    (net 132 "cm4-pins[40]")
+    (net 132 "cm4-line-2")
     (net 133 "pins[61]")
     (net 134 "cm4.hdi_b-pins[56]")
@@
             (layers "*.Cu" "*.Mask")
             (remove_unused_layers no)
-            (net 77 "rj45-anode-1"))
+            (net 77 "rj45-anode"))
         (pad "13" thru_hole circle
             (at -4.09 -6.89 90)
@@
             (layers "*.Cu" "*.Mask")
             (remove_unused_layers no)
-            (net 74 "rj45-anode"))
+            (net 74 "rj45-anode-1"))
         (pad "14" thru_hole circle
             (at -6.63 -6.89 90)
@@
             (layers "*.Cu" "*.Mask")
             (remove_unused_layers no)
-            (net 68 "rj45.connector-net-1"))
+            (net 68 "rj45.connector-net"))
         (pad "P2" thru_hole circle
             (at 4.55 4.35 90)
@@
             (layers "*.Cu" "*.Mask")
             (remove_unused_layers no)
-            (net 75 "rj45.connector-net"))
+            (net 75 "rj45.connector-net-1"))
         (pad "SHIELD0" thru_hole circle
             (at -7.74 1.06 90)
@@
             (layers "F.Cu" "F.Paste" "F.Mask")
             (remove_unused_layers no)
-            (net 73 "cm4-cathode-1"))
+            (net 73 "cm4-cathode"))
         (pad "2" smd rect
             (at 0.8 0 180)
@@
             (layers "F.Cu" "F.Paste" "F.Mask")
             (remove_unused_layers no)
-            (net 73 "cm4-cathode-1"))
+            (net 73 "cm4-cathode"))
         (pad "2" smd rect
             (at 0.43 0 270)
@@
             (layers "F.Cu" "F.Paste" "F.Mask")
             (remove_unused_layers no)
-            (net 71 "cm4-cathode"))
+            (net 71 "cm4-cathode-1"))
         (pad "2" smd rect
             (at 0.8 0 180)
@@
             (layers "F.Cu" "F.Paste" "F.Mask")
             (remove_unused_layers no)
-            (net 74 "rj45-anode")))
+            (net 74 "rj45-anode-1")))
     (footprint "atopile:CONN-SMD_DF40C-100DS-0.4V-51-ceffa9"
         (layer "F.Cu")
@@
             (layers "F.Cu" "F.Paste" "F.Mask")
             (remove_unused_layers no)
-            (net 11 "cm4-pins[46]-1"))
+            (net 11 "pins[46]"))
         (pad "78" smd rect
             (at 1 -1.6 0)
@@
             (layers "F.Cu" "F.Paste" "F.Mask")
             (remove_unused_layers no)
-            (net 95 "cm4.hdi_b-pins[40]"))
+            (net 95 "pins[40]"))
         (pad "81" smd rect
             (at 2.2 -1.6 0)
@@
             (layers "F.Cu" "F.Paste" "F.Mask")
             (remove_unused_layers no)
-            (net 103 "pins[26]"))
+            (net 103 "cm4.hdi_b-pins[26]"))
         (pad "88" smd rect
             (at 5 -1.6 0)
@@
             (layers "F.Cu" "F.Paste" "F.Mask")
             (remove_unused_layers no)
-            (net 77 "rj45-anode-1")))
+            (net 77 "rj45-anode")))
     (footprint "atopile:R0402-56259e"
         (layer "F.Cu")
@@
             (layers "F.Cu" "F.Paste" "F.Mask")
             (remove_unused_layers no)
-            (net 71 "cm4-cathode"))
+            (net 71 "cm4-cathode-1"))
         (pad "2" smd rect
             (at 0.43 0 270)
@@
             (layers "F.Cu" "F.Paste" "F.Mask")
             (remove_unused_layers no)
-            (net 52 "cm4-line-2"))
+            (net 52 "cm4-line-3"))
         (pad "13" smd rect
             (at 5 1.6 0)
@@
             (layers "F.Cu" "F.Paste" "F.Mask")
             (remove_unused_layers no)
-            (net 30 "line"))
+            (net 30 "line-2"))
         (pad "16" smd rect
             (at 3.8 1.6 0)
@@
             (layers "F.Cu" "F.Paste" "F.Mask")
             (remove_unused_layers no)
-            (net 123 "line-2"))
+            (net 123 "line-3"))
         (pad "18" smd rect
             (at 3 1.6 0)
@@
             (layers "F.Cu" "F.Paste" "F.Mask")
             (remove_unused_layers no)
-            (net 5 "cm4-line-4"))
+            (net 5 "cm4-line-5"))
         (pad "23" smd rect
             (at 1 1.6 0)
@@
             (layers "F.Cu" "F.Paste" "F.Mask")
             (remove_unused_layers no)
-            (net 6 "cm4-line-8"))
+            (net 6 "pins[47]"))
         (pad "25" smd rect
             (at 0.2 1.6 0)
@@
             (layers "F.Cu" "F.Paste" "F.Mask")
             (remove_unused_layers no)
-            (net 87 "cm4-line-6"))
+            (net 87 "cm4-line-1"))
         (pad "26" smd rect
             (at -0.2 1.6 0)
@@
             (layers "F.Cu" "F.Paste" "F.Mask")
             (remove_unused_layers no)
-            (net 9 "line-3"))
+            (net 9 "line"))
         (pad "28" smd rect
             (at -1 1.6 0)
@@
             (layers "F.Cu" "F.Paste" "F.Mask")
             (remove_unused_layers no)
-            (net 18 "cm4-line-5"))
+            (net 18 "pins[55]"))
         (pad "29" smd rect
             (at -1.4 1.6 0)
@@
             (layers "F.Cu" "F.Paste" "F.Mask")
             (remove_unused_layers no)
-            (net 129 "cm4-pins[46]"))
+            (net 129 "cm4-line-4"))
         (pad "78" smd rect
             (at 1 -1.6 0)
@@
             (layers "F.Cu" "F.Paste" "F.Mask")
             (remove_unused_layers no)
-            (net 2 "cm4-line-3"))
+            (net 2 "cm4-line-6"))
         (pad "79" smd rect
             (at 1.4 -1.6 0)
@@
             (layers "F.Cu" "F.Paste" "F.Mask")
             (remove_unused_layers no)
-            (net 132 "cm4-pins[40]"))
+            (net 132 "cm4-line-2"))
         (pad "81" smd rect
             (at 2.2 -1.6 0)
@@
             (layers "F.Cu" "F.Paste" "F.Mask")
             (remove_unused_layers no)
-            (net 120 "cm4-line"))
+            (net 120 "pins[30]"))
         (pad "86" smd rect
             (at 4.2 -1.6 0)
@@
             (layers "F.Cu" "F.Paste" "F.Mask")
             (remove_unused_layers no)
-            (net 13 "cm4-line-7"))
+            (net 13 "cm4-line"))
         (pad "87" smd rect
             (at 4.6 -1.6 0)
@@
             (layers "F.Cu" "F.Paste" "F.Mask")
             (remove_unused_layers no)
-            (net 104 "cm4-line-1"))
+            (net 104 "cm4-pins[26]"))
         (pad "88" smd rect
             (at 5 -1.6 0)

Commit message: build with latest main
Parts:
- removed CN1, CN2: , atopile:CONN-SMD_DF40C-100DS-0.4V-51-ceffa9
- removed D1: , atopile:LED0603-RD-YELLOW-5af84a
- removed D2: , atopile:LED0603-RD-c81ffb
- removed R1, R2: 10kΩ ±1% 62.5mW, atopile:R0402-56259e
- removed R3, R4: 470Ω ±1% 100mW, atopile:R0603-ebcab9
- removed RJ1: , atopile:RJ45-TH_HR911130A-5845d4
- removed U1: , atopile:SOT-23-5_L3.0-W1.7-P0.95-LS2.8-BR-9d80aa
Routing:
- net ETH_LED_ACTIVITY: track 32.0 -> 0.00 mm, vias 1 -> 0
- net ETH_LED_LINK: track 27.0 -> 0.00 mm, vias 1 -> 0
- net ETH_P0_N: track 21.0 -> 0.00 mm, vias 1 -> 0
- net ETH_P3_P: track 19.4 -> 0.00 mm, vias 1 -> 0
- net ETH_P1_N: track 19.2 -> 0.00 mm, vias 1 -> 0
- net ETH_P3_N: track 18.3 -> 0.00 mm, vias 1 -> 0
- net ETH_P0_P: track 18.0 -> 0.00 mm, vias 1 -> 0
- net ETH_P1_P: track 17.6 -> 0.00 mm, vias 1 -> 0
- net ETH_P2_N: track 16.1 -> 0.00 mm, vias 1 -> 0
- net ETH_P2_P: track 14.7 -> 0.00 mm, vias 1 -> 0
- net PWR_LED: track 8.93 -> 0.00 mm
- net (no net): track 6.43 -> 0.00 mm, vias 5 -> 0
- net pins[19]: track 6.16 -> 0.00 mm, vias 2 -> 0
- net rj45-anode: track 5.94 -> 0.00 mm
- net rj45-anode-1: track 5.90 -> 0.00 mm
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Other:
- copper layers 4 -> 2
