File: elec/layout/multiplexer-i2c-8ch/multiplexer-i2c-8ch.kicad_pcb (KiCad board)
At the start: 2 copper layers, 4 parts

Commit message: build and re-link layouts
Parts:
- C2: value 100nF ±10% 16V X7R -> 1µF ±10% 25V X5R
Connections:
- U1 pad 10: gpio_expander-net-2 -> gpio_expander-net-1
- U1 pad 12: line-6 -> line-4
- U1 pad 13: line-7 -> line-8
- U1 pad 16: gnd -> hv
- U1 pad 2: gpio_expander-net -> gpio_expander-net-2
- U1 pad 9: gpio_expander-net-1 -> gpio_expander-net
- U2 pad 1: line-3 -> line-1
- U2 pad 12: line-4 -> line-9
- U2 pad 14: line-8 -> line-7
- U2 pad 15: line-1 -> line-6
- U2 pad 2: line-5 -> line
- U2 pad 4: line-9 -> line-5
- U2 pad 5: line -> line-3

Commit message: all modules building
Connections:
- U1 pad 10: gpio_expander-net-1 -> gpio_expander-net
- U1 pad 12: line-4 -> line-6
- U1 pad 13: line-8 -> line-4
- U1 pad 2: gpio_expander-net-2 -> gpio_expander-net-1
- U1 pad 9: gpio_expander-net -> gpio_expander-net-2
- U2 pad 1: line-1 -> line-2
- U2 pad 12: line-9 -> line-8
- U2 pad 13: line-2 -> line-9
- U2 pad 14: line-7 -> line-5
- U2 pad 15: line-6 -> line-3
- U2 pad 4: line-5 -> line-1
- U2 pad 5: line-3 -> line-7
Changed lines of the file:
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@@
     (net 0 "")
     (net 1 "INT")
-    (net 2 "gpio_expander-net-2")
-    (net 3 "line-9")
-    (net 4 "line-5")
+    (net 2 "gpio_expander-net-1")
+    (net 3 "line-8")
+    (net 4 "line-1")
     (net 5 "line")
-    (net 6 "line-7")
-    (net 7 "line-1")
-    (net 8 "line-2")
-    (net 9 "line-8")
+    (net 6 "line-5")
+    (net 7 "line-2")
+    (net 8 "line-9")
+    (net 9 "line-4")
     (net 10 "gnd")
-    (net 11 "gpio_expander-net")
-    (net 12 "line-3")
+    (net 11 "gpio_expander-net-2")
+    (net 12 "line-7")
     (net 13 "hv")
-    (net 14 "line-6")
-    (net 15 "gpio_expander-net-1")
+    (net 14 "line-3")
+    (net 15 "gpio_expander-net")
     (net 16 "Eh")
-    (net 17 "line-4")
+    (net 17 "line-6")
     (net 18 "S0")
     (net 19 "S2")
@@
             (layers "F.Cu" "F.Paste" "F.Mask")
             (remove_unused_layers no)
-            (net 2 "gpio_expander-net-2"))
+            (net 2 "gpio_expander-net-1"))
         (pad "3" smd rect
             (at 0.25 1.41 180)
@@
             (layers "F.Cu" "F.Paste" "F.Mask")
             (remove_unused_layers no)
-            (net 11 "gpio_expander-net"))
+            (net 11 "gpio_expander-net-2"))
         (pad "10" smd rect
             (at 0.25 -1.41 180)
@@
             (layers "F.Cu" "F.Paste" "F.Mask")
             (remove_unused_layers no)
-            (net 15 "gpio_expander-net-1"))
+            (net 15 "gpio_expander-net"))
         (pad "11" smd rect
             (at -0.25 -1.41 180)
@@
             (layers "F.Cu" "F.Paste" "F.Mask")
             (remove_unused_layers no)
-            (net 17 "line-4"))
+            (net 17 "line-6"))
         (pad "13" smd rect
             (at -1.41 -0.75 180)
@@
             (layers "F.Cu" "F.Paste" "F.Mask")
             (remove_unused_layers no)
-            (net 9 "line-8"))
+            (net 9 "line-4"))
         (pad "14" smd rect
             (at -1.41 -0.25 180)
@@
             (layers "F.Cu" "F.Paste" "F.Mask")
             (remove_unused_layers no)
-            (net 7 "line-1"))
+            (net 7 "line-2"))
         (pad "2" smd oval
             (at -1.63 2.87 0)
@@
             (layers "F.Cu" "F.Paste" "F.Mask")
             (remove_unused_layers no)
-            (net 4 "line-5"))
+            (net 4 "line-1"))
         (pad "5" smd oval
             (at 0.33 2.87 0)
@@
             (layers "F.Cu" "F.Paste" "F.Mask")
             (remove_unused_layers no)
-            (net 12 "line-3"))
+            (net 12 "line-7"))
         (pad "6" smd oval
             (at 0.98 2.87 0)
@@
             (layers "F.Cu" "F.Paste" "F.Mask")
             (remove_unused_layers no)
-            (net 3 "line-9"))
+            (net 3 "line-8"))
         (pad "13" smd oval
             (at -0.32 -2.87 0)
@@
             (layers "F.Cu" "F.Paste" "F.Mask")
             (remove_unused_layers no)
-            (net 8 "line-2"))
+            (net 8 "line-9"))
         (pad "14" smd oval
             (at -0.98 -2.87 0)
@@
             (layers "F.Cu" "F.Paste" "F.Mask")
             (remove_unused_layers no)
-            (net 6 "line-7"))
+            (net 6 "line-5"))
         (pad "15" smd oval
             (at -1.63 -2.87 0)
@@
             (layers "F.Cu" "F.Paste" "F.Mask")
             (remove_unused_layers no)
-            (net 14 "line-6"))
+            (net 14 "line-3"))
         (pad "16" smd oval
             (at -2.28 -2.87 0)

Commit message: HIL Building
Connections:
- U1 pad 10: gpio_expander-net -> gpio_expander-net-2
- U1 pad 12: line-6 -> line-4
- U1 pad 13: line-4 -> line
- U1 pad 2: gpio_expander-net-1 -> gpio_expander-net
- U1 pad 9: gpio_expander-net-2 -> gpio_expander-net-1
- U2 pad 1: line-2 -> line-8
- U2 pad 12: line-8 -> line-2
- U2 pad 13: line-9 -> line-1
- U2 pad 15: line-3 -> line-6
- U2 pad 2: line -> line-7
- U2 pad 4: line-1 -> line-3
- U2 pad 5: line-7 -> line-9
Changed lines of the file:
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@@
     (net 0 "")
     (net 1 "INT")
-    (net 2 "gpio_expander-net-1")
-    (net 3 "line-8")
-    (net 4 "line-1")
-    (net 5 "line")
+    (net 2 "gpio_expander-net")
+    (net 3 "line-2")
+    (net 4 "line-3")
+    (net 5 "line-7")
     (net 6 "line-5")
-    (net 7 "line-2")
-    (net 8 "line-9")
-    (net 9 "line-4")
+    (net 7 "line-8")
+    (net 8 "line-1")
+    (net 9 "line")
     (net 10 "gnd")
-    (net 11 "gpio_expander-net-2")
-    (net 12 "line-7")
+    (net 11 "gpio_expander-net-1")
+    (net 12 "line-9")
     (net 13 "hv")
-    (net 14 "line-3")
-    (net 15 "gpio_expander-net")
+    (net 14 "line-6")
+    (net 15 "gpio_expander-net-2")
     (net 16 "Eh")
-    (net 17 "line-6")
+    (net 17 "line-4")
     (net 18 "S0")
     (net 19 "S2")
@@
             (layers "F.Cu" "F.Paste" "F.Mask")
             (remove_unused_layers no)
-            (net 2 "gpio_expander-net-1"))
+            (net 2 "gpio_expander-net"))
         (pad "3" smd rect
             (at 0.25 1.41 180)
@@
             (layers "F.Cu" "F.Paste" "F.Mask")
             (remove_unused_layers no)
-            (net 11 "gpio_expander-net-2"))
+            (net 11 "gpio_expander-net-1"))
         (pad "10" smd rect
             (at 0.25 -1.41 180)
@@
             (layers "F.Cu" "F.Paste" "F.Mask")
             (remove_unused_layers no)
-            (net 15 "gpio_expander-net"))
+            (net 15 "gpio_expander-net-2"))
         (pad "11" smd rect
             (at -0.25 -1.41 180)
@@
             (layers "F.Cu" "F.Paste" "F.Mask")
             (remove_unused_layers no)
-            (net 17 "line-6"))
+            (net 17 "line-4"))
         (pad "13" smd rect
             (at -1.41 -0.75 180)
@@
             (layers "F.Cu" "F.Paste" "F.Mask")
             (remove_unused_layers no)
-            (net 9 "line-4"))
+            (net 9 "line"))
         (pad "14" smd rect
             (at -1.41 -0.25 180)
@@
             (layers "F.Cu" "F.Paste" "F.Mask")
             (remove_unused_layers no)
-            (net 7 "line-2"))
+            (net 7 "line-8"))
         (pad "2" smd oval
             (at -1.63 2.87 0)
@@
             (layers "F.Cu" "F.Paste" "F.Mask")
             (remove_unused_layers no)
-            (net 5 "line"))
+            (net 5 "line-7"))
         (pad "3" smd oval
             (at -0.98 2.87 0)
@@
             (layers "F.Cu" "F.Paste" "F.Mask")
             (remove_unused_layers no)
-            (net 4 "line-1"))
+            (net 4 "line-3"))
         (pad "5" smd oval
             (at 0.33 2.87 0)
@@
             (layers "F.Cu" "F.Paste" "F.Mask")
             (remove_unused_layers no)
-            (net 12 "line-7"))
+            (net 12 "line-9"))
         (pad "6" smd oval
             (at 0.98 2.87 0)
@@
             (layers "F.Cu" "F.Paste" "F.Mask")
             (remove_unused_layers no)
-            (net 3 "line-8"))
+            (net 3 "line-2"))
         (pad "13" smd oval
             (at -0.32 -2.87 0)
@@
             (layers "F.Cu" "F.Paste" "F.Mask")
             (remove_unused_layers no)
-            (net 8 "line-9"))
+            (net 8 "line-1"))
         (pad "14" smd oval
             (at -0.98 -2.87 0)
@@
             (layers "F.Cu" "F.Paste" "F.Mask")
             (remove_unused_layers no)
-            (net 14 "line-3"))
+            (net 14 "line-6"))
         (pad "16" smd oval
             (at -2.28 -2.87 0)

Commit message: build with latest main
Parts:
- removed C1: 100nF ±10% 16V X7R, atopile:C0402-b3ef17
- removed C2: 1µF ±10% 25V X5R, atopile:C0402-b3ef17
- removed U1: , atopile:QFN-16_L3.0-W3.0-P0.50-BL-EP1.7-3a4c56
- removed U2: , atopile:TSSOP-16_L5.0-W4.4-P0.65-LS6.4-BL-4f6acc
Routing:
- net gnd: track 10.3 -> 0.00 mm, vias 5 -> 0
- net hv: track 7.10 -> 0.00 mm, vias 2 -> 0
- net A: track 5.74 -> 0.00 mm
- net S0: track 3.85 -> 0.00 mm
- net S2: track 3.82 -> 0.00 mm
- net Eh: track 3.79 -> 0.00 mm
- net S1: track 3.46 -> 0.00 mm
