File: elec/layout/controller-cm5/cm4.kicad_pcb (KiCad board)
At the start: 4 copper layers, 14 parts

Commit message: update layout
Connections:
- CN1 pad 12: cm5-line-4 -> cm5-line-7
- CN1 pad 15: line-4 -> line-1
- CN1 pad 19: cm5-line-6 -> cm5-line-4
- CN1 pad 23: cm5-line-7 -> cm5-line-5
- CN1 pad 25: cm5-line-8 -> cm5-line-2
- CN1 pad 27: line-1 -> line-7
- CN1 pad 40: line-7 -> line-3
- CN1 pad 41: line -> line-4
- CN1 pad 78: cm5-line-1 -> cm5-line-3
- CN1 pad 80: cm5-line-5 -> cm5-line-1
- CN1 pad 81: line-3 -> line
- CN1 pad 85: cm5-line-2 -> cm5-line
- CN1 pad 86: cm5-line-3 -> cm5-line-6
- D1 pad 1: cm5-cathode-1 -> cm5-cathode
- D2 pad 1: cm5-cathode -> cm5-cathode-1
- R1 pad 1: cm5-cathode-1 -> cm5-cathode
- R2 pad 1: cm5-cathode -> cm5-cathode-1
- R2 pad 2: cm5-line -> Y
- R3 pad 2: rj45-anode-1 -> rj45-anode
- R4 pad 2: rj45-anode -> rj45-anode-1
- RJ1 pad 11: rj45-anode-1 -> rj45-anode
- RJ1 pad 14: rj45-anode -> rj45-anode-1
- RJ1 pad P1: rj45.connector-net-1 -> rj45.connector-net
- RJ1 pad P10: rj45.connector-net -> rj45.connector-net-1
- U1 pad 4: cm5-line -> Y
Routing:
- net cm5-line: track 1.86 -> 0.00 mm
- net Y: track 0.00 -> 1.86 mm
Changed lines of the file:
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@@
 	(net 0 "")
 	(net 1 "pins[20]")
-	(net 2 "cm5-line-1")
+	(net 2 "cm5-line-3")
 	(net 3 "cm5-pins[62]")
 	(net 4 "cm5.hdi_a-pins[74]")
@@
 	(net 7 "cm5.hdi_b-pins[74]")
 	(net 8 "cm5.hdi_a-pins[62]")
-	(net 9 "line-1")
+	(net 9 "line-7")
 	(net 10 "pins[18]")
 	(net 11 "cm5-pins[46]")
 	(net 12 "pins[67]")
-	(net 13 "cm5-line-3")
+	(net 13 "cm5-line-6")
 	(net 14 "UART_TX")
 	(net 15 "pins[5]")
@@
 	(net 22 "cm5.hdi_a-pins[68]")
 	(net 23 "cm5.hdi_a-pins[92]")
-	(net 24 "line")
+	(net 24 "line-4")
 	(net 25 "pins[8]")
 	(net 26 "pins[1]")
@@
 	(net 28 "pins[90]")
 	(net 29 "pins[82]")
-	(net 30 "line-4")
+	(net 30 "line-1")
 	(net 31 "pins[58]")
 	(net 32 "SDA")
@@
 	(net 38 "line-5")
 	(net 39 "HDMI1_CK_N")
-	(net 40 "line-7")
+	(net 40 "line-3")
 	(net 41 "pins[86]")
 	(net 42 "cm5-pins[99]")
@@
 	(net 49 "cm5.hdi_b-pins[88]")
 	(net 50 "cm5.hdi_b-pins[92]")
-	(net 51 "cm5-line-6")
-	(net 52 "cm5-line-4")
+	(net 51 "cm5-line-4")
+	(net 52 "cm5-line-7")
 	(net 53 "pins[29]")
 	(net 54 "pins[49]")
@@
 	(net 65 "cm5.hdi_a-pins[15]")
 	(net 66 "HDMI0_D1_P")
-	(net 67 "rj45.connector-net-1")
-	(net 68 "cm5-line")
-	(net 69 "cm5-cathode-1")
-	(net 70 "cm5-cathode")
-	(net 71 "rj45.connector-net")
+	(net 67 "rj45.connector-net")
+	(net 68 "Y")
+	(net 69 "cm5-cathode")
+	(net 70 "cm5-cathode-1")
+	(net 71 "rj45.connector-net-1")
 	(net 72 "N_C_")
-	(net 73 "cm5-line-7")
+	(net 73 "cm5-line-5")
 	(net 74 "pins[3]")
 	(net 75 "HDMI0_CK_P")
@@
 	(net 80 "pins[41]")
 	(net 81 "pins[70]")
-	(net 82 "cm5-line-8")
+	(net 82 "cm5-line-2")
 	(net 83 "cm5.hdi_a-pins[98]")
 	(net 84 "cm5.hdi_b-pins[34]")
@@
 	(net 113 "pins[72]")
 	(net 114 "HDMI0_CK_N")
-	(net 115 "cm5-line-2")
+	(net 115 "cm5-line")
 	(net 116 "HDMI0_D2_P")
 	(net 117 "pins[22]")
@@
 	(net 125 "cm5.hdi_a-pins[94]")
 	(net 126 "cm5.hdi_a-pins[34]")
-	(net 127 "cm5-line-5")
+	(net 127 "cm5-line-1")
 	(net 128 "pins[61]")
 	(net 129 "cm5-pins[56]")
@@
 	(net 133 "pins[32]")
 	(net 134 "cm5.hdi_b-pins[93]")
-	(net 135 "line-3")
+	(net 135 "line")
 	(net 136 "cm5-pins[98]")
 	(net 137 "ETH_P0_P")
@@
 	(net 161 "stud3.footprint.pins[2].net-net")
 	(net 162 "stud1.footprint.pins[3].net-net")
-	(net 163 "rj45-anode")
+	(net 163 "rj45-anode-1")
 	(net 164 "ETH_LED_LINK")
-	(net 165 "rj45-anode-1")
+	(net 165 "rj45-anode")
 	(net 166 "ETH_LED_ACTIVITY")
 	(footprint "atopile:SMD_BD5.6-D4.1-12eb58"
@@
 			)
 			(remove_unused_layers no)
-			(net 165 "rj45-anode-1")
+			(net 165 "rj45-anode")
 		)
 		(pad "12" thru_hole circle
@@
 			)
 			(remove_unused_layers no)
-			(net 163 "rj45-anode")
+			(net 163 "rj45-anode-1")
 		)
 		(pad "P1" thru_hole rect
@@
 			)
 			(remove_unused_layers no)
-			(net 67 "rj45.connector-net-1")
+			(net 67 "rj45.connector-net")
 		)
 		(pad "P2" thru_hole circle
@@
 			)
 			(remove_unused_layers no)
-			(net 71 "rj45.connector-net")
+			(net 71 "rj45.connector-net-1")
 		)
 		(pad "SHIELD0" thru_hole circle
@@
 			(size 0.8 0.8)
 			(layers "F.Cu" "F.Paste" "F.Mask")
-			(net 70 "cm5-cathode")
+			(net 70 "cm5-cathode-1")
 		)
 		(pad "2" smd rect
@@
 			(size 0.57 0.54)
 			(layers "F.Cu" "F.Paste" "F.Mask")
-			(net 70 "cm5-cathode")
+			(net 70 "cm5-cathode-1")
 		)
 		(pad "2" smd rect
@@
 			(size 0.57 0.54)
 			(layers "F.Cu" "F.Paste" "F.Mask")
-			(net 68 "cm5-line")
+			(net 68 "Y")
 		)
 	)
@@
 			(size 0.8 0.8)
 			(layers "F.Cu" "F.Paste" "F.Mask")
-			(net 69 "cm5-cathode-1")
+			(net 69 "cm5-cathode")
 		)
 		(pad "2" smd rect
@@
 			(size 1.1 0.6)
 			(layers "F.Cu" "F.Paste" "F.Mask")
-			(net 68 "cm5-line")
+			(net 68 "Y")
 		)
 		(pad "5" smd rect
@@
 			(size 0.81 0.86)
 			(layers "F.Cu" "F.Paste" "F.Mask")
-			(net 163 "rj45-anode")
+			(net 163 "rj45-anode-1")
 		)
 	)
@@
 			(size 0.81 0.86)
 			(layers "F.Cu" "F.Paste" "F.Mask")
-			(net 165 "rj45-anode-1")
+			(net 165 "rj45-anode")
 		)
 	)
@@
 			(size 0.57 0.54)
 			(layers "F.Cu" "F.Paste" "F.Mask")
-			(net 69 "cm5-cathode-1")
+			(net 69 "cm5-cathode")
 		)
 		(pad "2" smd rect
@@
 			(size 0.2 0.7)
 			(layers "F.Cu" "F.Paste" "F.Mask")
-			(net 52 "cm5-line-4")
+			(net 52 "cm5-line-7")
 		)
 		(pad "13" smd rect
@@
 			(size 0.2 0.7)
 			(layers "F.Cu" "F.Paste" "F.Mask")
-			(net 30 "line-4")
+			(net 30 "line-1")
 		)
 		(pad "16" smd rect
@@
 			(size 0.2 0.7)
 			(layers "F.Cu" "F.Paste" "F.Mask")
-			(net 51 "cm5-line-6")
+			(net 51 "cm5-line-4")
 		)
 		(pad "20" smd rect
@@
 			(size 0.2 0.7)
 			(layers "F.Cu" "F.Paste" "F.Mask")
-			(net 73 "cm5-line-7")
+			(net 73 "cm5-line-5")
 		)
 		(pad "24" smd rect
@@
 			(size 0.2 0.7)
 			(layers "F.Cu" "F.Paste" "F.Mask")
-			(net 82 "cm5-line-8")
+			(net 82 "cm5-line-2")
 		)
 		(pad "26" smd rect
@@
 			(size 0.2 0.7)
 			(layers "F.Cu" "F.Paste" "F.Mask")
-			(net 9 "line-1")
+			(net 9 "line-7")
 		)
 		(pad "28" smd rect
@@
 			(size 0.2 0.7)
 			(layers "F.Cu" "F.Paste" "F.Mask")
-			(net 40 "line-7")
+			(net 40 "line-3")
 		)
 		(pad "41" smd rect
@@
 			(size 0.2 0.7)
 			(layers "F.Cu" "F.Paste" "F.Mask")
-			(net 24 "line")
+			(net 24 "line-4")
 		)
 		(pad "42" smd rect
@@
 			(size 0.2 0.7)
 			(layers "F.Cu" "F.Paste" "F.Mask")
-			(net 2 "cm5-line-1")
+			(net 2 "cm5-line-3")
 		)
 		(pad "79" smd rect
@@
 			(size 0.2 0.7)
 			(layers "F.Cu" "F.Paste" "F.Mask")
-			(net 127 "cm5-line-5")
+			(net 127 "cm5-line-1")
 		)
 		(pad "81" smd rect
@@
 			(size 0.2 0.7)
 			(layers "F.Cu" "F.Paste" "F.Mask")
-			(net 135 "line-3")
+			(net 135 "line")
 		)
 		(pad "82" smd rect
@@
 			(size 0.2 0.7)
 			(layers "F.Cu" "F.Paste" "F.Mask")
-			(net 115 "cm5-line-2")
+			(net 115 "cm5-line")
 		)
 		(pad "86" smd rect
@@
 			(size 0.2 0.7)
 			(layers "F.Cu" "F.Paste" "F.Mask")
-			(net 13 "cm5-line-3")
+			(net 13 "cm5-line-6")
 		)
 		(pad "87" smd rect
