File: elec/layout/controller-cm5/cm5.kicad_pcb (KiCad board)
At the start: 4 copper layers, 16 parts

Commit message: building frozen
Connections:
- net MDI3plus renamed pins[2]-1
- net cm5-pins[87] renamed pins[87]
- net cm5-pins[87]-1 renamed cm5-pins[89]-1
- net pins[89] renamed cm5-pins[89]
- CN1 pad 15: line -> line-1
- CN1 pad 18: pins[35]-1 -> pins[35]
- CN1 pad 2: MDI1plus -> pins[3]
- CN1 pad 27: cm5-pins[53] -> cm5-pins[53]-1
- CN1 pad 3: pins[5] -> MDI1_
- CN1 pad 57: pins[78] -> pins[76]
- CN1 pad 58: pins[78] -> pins[76]
- CN1 pad 59: pins[78] -> pins[76]
- CN1 pad 6: MDI0plus -> pins[11]
- CN1 pad 60: pins[78] -> pins[76]
- CN1 pad 61: pins[78] -> pins[76]
- CN1 pad 62: pins[78] -> pins[76]
- CN1 pad 76: cm5-pins[48]-1 -> cm5-pins[48]
- CN1 pad 78: cm5-pins[44]-1 -> cm5-pins[44]
- CN1 pad 81: pins[38] -> line-2
- CN1 pad 82: line-1 -> pins[36]
- CN1 pad 87: pins[26] -> line
- CN1 pad 96: MDI2_ -> pins[8]
- CN2 pad 18: pins[35] -> pins[35]-1
- CN2 pad 2: pins[3] -> cm5.hdi_b-pins[3]
- CN2 pad 27: cm5-pins[53]-1 -> cm5-pins[53]
- CN2 pad 3: cm5.hdi_b-pins[5] -> pins[5]
- CN2 pad 6: pins[11] -> cm5.hdi_b-pins[11]
- CN2 pad 62: pins[76] -> cm5.hdi_b-pins[76]
- CN2 pad 76: cm5-pins[48] -> cm5-pins[48]-1
- CN2 pad 78: cm5-pins[44] -> cm5-pins[44]-1
- CN2 pad 81: cm5.hdi_b-pins[38] -> pins[38]
- CN2 pad 87: cm5.hdi_b-pins[26] -> pins[26]
- CN2 pad 96: pins[8] -> cm5.hdi_b-pins[8]
- D1 pad 1: cm5-cathode-1 -> cm5-cathode
- D2 pad 1: cm5-cathode -> cm5-cathode-1
- R1 pad 1: cm5-cathode-1 -> cm5-cathode
- R2 pad 1: cm5-cathode -> cm5-cathode-1
- R3 pad 2: rj45-anode -> rj45-anode-1
- R4 pad 2: rj45-anode-1 -> rj45-anode
- RJ1 pad 11: rj45-anode -> rj45-anode-1
- RJ1 pad 14: rj45-anode-1 -> rj45-anode
- RJ1 pad P1: rj45.connector-net-1 -> rj45.connector-net
- RJ1 pad P10: rj45.connector-net -> rj45.connector-net-1
- RJ1 pad P2: MDI0plus -> pins[11]
- RJ1 pad P4: MDI1plus -> pins[3]
- RJ1 pad P6: MDI2_ -> pins[8]
- RJ1 pad P7: pins[5] -> MDI1_
Routing:
- net pins[5]: track 18.8 -> 0.00 mm, vias 1 -> 0
- net MDI1_: track 0.00 -> 18.8 mm, vias 0 -> 1
- net pins[3]: track 0.00 -> 17.3 mm, vias 0 -> 1
- net MDI1plus: track 17.3 -> 0.00 mm, vias 1 -> 0
- net pins[11]: track 0.00 -> 16.5 mm, vias 0 -> 1
- net MDI0plus: track 16.5 -> 0.00 mm, vias 1 -> 0
- net pins[8]: track 0.00 -> 14.7 mm, vias 0 -> 1
- net MDI2_: track 14.7 -> 0.00 mm, vias 1 -> 0

Commit message: building locally to fix frozen builds
Connections:
- net cm5-pins[89] renamed pins[89]
- net cm5-pins[89]-1 renamed cm5-pins[87]-1
- net pins[2]-1 renamed MDI3plus
- net pins[4]-1 renamed MDI3_
- net pins[87] renamed cm5-pins[87]
- CN1 pad 15: line-1 -> cm5-pins[29]
- CN1 pad 18: pins[35] -> pins[35]-1
- CN1 pad 2: pins[3] -> MDI1plus
- CN1 pad 24: cm5-pins[47] -> cm5-pins[47]-1
- CN1 pad 5: MDI0_ -> pins[9]
- CN1 pad 76: cm5-pins[48] -> cm5-pins[48]-1
- CN1 pad 81: line-2 -> line
- CN1 pad 87: line -> line-1
- CN1 pad 96: pins[8] -> MDI2_
- CN2 pad 18: pins[35]-1 -> pins[35]
- CN2 pad 2: cm5.hdi_b-pins[3] -> pins[3]
- CN2 pad 24: cm5-pins[47]-1 -> cm5-pins[47]
- CN2 pad 5: pins[9] -> cm5.hdi_b-pins[9]
- CN2 pad 76: cm5-pins[48]-1 -> cm5-pins[48]
- CN2 pad 96: cm5.hdi_b-pins[8] -> pins[8]
- R3 pad 2: rj45-anode-1 -> rj45-anode
- R4 pad 2: rj45-anode -> rj45-anode-1
- RJ1 pad 11: rj45-anode-1 -> rj45-anode
- RJ1 pad 14: rj45-anode -> rj45-anode-1
- RJ1 pad P3: MDI0_ -> pins[9]
- RJ1 pad P4: pins[3] -> MDI1plus
- RJ1 pad P6: pins[8] -> MDI2_
Routing:
- net pins[9]: track 0.00 -> 19.6 mm, vias 0 -> 1
- net MDI0_: track 19.6 -> 0.00 mm, vias 1 -> 0
- net pins[3]: track 17.3 -> 0.00 mm, vias 1 -> 0
- net MDI1plus: track 0.00 -> 17.3 mm, vias 0 -> 1
- net pins[8]: track 14.7 -> 0.00 mm, vias 1 -> 0
- net MDI2_: track 0.00 -> 14.7 mm, vias 0 -> 1
