File: elec/layout/usb2-hub/usb2-hub.kicad_pcb (KiCad board)
At the start: 2 copper layers, 4 parts

Commit message: assemble
Parts:
- added C10: 100nF ±10% 16V X7R, atopile:C0402-b3ef17, F.Cu at (62.8, 36.4)
- added C11: 10µF ±10% 10V X5R, atopile:C0603-bd72f6, F.Cu at (118.5, 33.6)
- added C12: 10µF ±10% 10V X5R, atopile:C0603-bd72f6, F.Cu at (125.8, 31.9)
- added C13: 10µF ±10% 10V X5R, atopile:C0603-bd72f6, F.Cu at (125.9, 34.7)
- added C14: 10µF ±10% 10V X5R, atopile:C0603-bd72f6, F.Cu at (127.3, 31.9)
- added C15: 10µF ±10% 10V X5R, atopile:C0603-bd72f6, F.Cu at (124.4, 31.9)
- added C16: 10µF ±10% 10V X5R, atopile:C0603-bd72f6, F.Cu at (124.5, 34.7)
- added C3: 10µF ±10% 10V X5R, atopile:C0603-bd72f6, F.Cu at (68.1, 38.0)
- added C4: 10µF ±10% 10V X5R, atopile:C0603-bd72f6, F.Cu at (55.1, 46.9)
- added C5: 100nF ±10% 16V X7R, atopile:C0402-b3ef17, F.Cu at (59.6, 36.4)
- added C6: 100nF ±10% 16V X7R, atopile:C0402-b3ef17, F.Cu at (68.2, 42.6)
- added C7: 100nF ±10% 16V X7R, atopile:C0402-b3ef17, F.Cu at (57.6, 36.5)
- added C8: 100nF ±10% 16V X7R, atopile:C0402-b3ef17, F.Cu at (68.2, 43.6)
- added C9: 100nF ±10% 16V X7R, atopile:C0402-b3ef17, F.Cu at (67.9, 40.9)
- added D1: , atopile:SOT-143_L2.9-W1.3-P1.92-LS2.3-BR-44397f, F.Cu at (58.7, 46.7)
- added D2: , atopile:SOT-143_L2.9-W1.3-P1.92-LS2.3-BR-44397f, F.Cu at (61.9, 46.8)
- added D3: , atopile:SOT-143_L2.9-W1.3-P1.92-LS2.3-BR-44397f, F.Cu at (65.2, 46.7)
- added D4: , atopile:SOT-143_L2.9-W1.3-P1.92-LS2.3-BR-44397f, F.Cu at (68.5, 46.7)
- added D5: , atopile:SOT-143_L2.9-W1.3-P1.92-LS2.3-BR-44397f, F.Cu at (55.6, 38.6)
- added R1: 33kΩ ±1% 62.5mW, atopile:R0402-56259e, F.Cu at (61.8, 36.2)
- added R2: 33kΩ ±1% 62.5mW, atopile:R0402-56259e, F.Cu at (63.8, 36.2)
- added R3: 12kΩ ±1% 62.5mW, atopile:R0402-56259e, F.Cu at (58.5, 44.1)
- added R4: 33kΩ ±1% 62.5mW, atopile:R0402-56259e, F.Cu at (60.8, 36.2)
- added R5: 33kΩ ±1% 62.5mW, atopile:R0402-56259e, F.Cu at (58.6, 36.2)
- added R6: 15kΩ ±1% 62.5mW, atopile:R0402-56259e, F.Cu at (120.6, 36.1)
- added U2: , atopile:SOT-23-6_L2.9-W1.6-P0.95-LS2.8-BR-bfc73b, F.Cu at (121.5, 33.9)
- moved C1 79.8 mm to (55.6, 45.5), turned to 180 degrees
- moved U1 75.2 mm to (62.8, 41.3)
- moved C2 68.2 mm to (53.4, 42.6), turned to -90 degrees
- moved X1 62.4 mm to (55.7, 42.5), turned to 90 degrees
Connections:
- net PRTPWR1_BC_EN1 renamed line-7
- U1 pad 1: hub-line -> line-5
- U1 pad 10: VDDA33 -> hv-1
- U1 pad 15: VDD33 -> hv-1
- U1 pad 2: hub-line-2 -> line-9
- U1 pad 22: SDA_SMBBATA_NON_REM1 -> hub-line-1
- U1 pad 23: VDD33 -> hv-1
- U1 pad 24: SCL_SMBCLK_CFG_SEL0 -> hub-line
- U1 pad 27: VBUS_DET -> hv-1
- U1 pad 29: VDDA33 -> hv-1
- U1 pad 3: hub-line-4 -> line-4
- U1 pad 30: USBDM_UP -> line-8
- U1 pad 31: USBDP_UP -> line-10
- U1 pad 32: XTALOUT -> xout
- U1 pad 33: XTALIN_CLKIN -> xin
- U1 pad 36: VDDA33 -> hv-1
- U1 pad 37: EP -> gnd
- U1 pad 4: hub-line-1 -> line-1
- U1 pad 5: VDDA33 -> hv-1
- U1 pad 6: hub-line-6 -> line-2
- U1 pad 7: hub-line-3 -> line
- U1 pad 8: hub-line-7 -> line-6
- U1 pad 9: hub-line-5 -> line-3
Routing:
- net gnd-1: track 0.00 -> 19.8 mm, vias 0 -> 10
- net hv-1: track 0.00 -> 15.6 mm, vias 0 -> 7
- net hv: track 0.00 -> 11.0 mm, vias 0 -> 4
- net xout: track 0.00 -> 7.75 mm
- net line-3: track 0.00 -> 7.56 mm
- net line-6: track 0.00 -> 7.14 mm
- net gnd: track 0.00 -> 7.13 mm, vias 0 -> 4
- net line-8: track 0.00 -> 6.77 mm
- net line-10: track 0.00 -> 6.19 mm
- net xin: track 0.00 -> 6.12 mm
- net line-5: track 0.00 -> 5.66 mm
- net line-9: track 0.00 -> 5.59 mm
- net line: track 0.00 -> 5.28 mm
- net line-1: track 0.00 -> 3.90 mm
- net line-4: track 0.00 -> 3.90 mm
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
Commit message: Fix gnd issue
Parts:
- moved C14 56.4 mm to (71.2, 38.2), turned to 180 degrees
- moved C12 55.2 mm to (71.2, 39.6), turned to 180 degrees
- moved C15 54.0 mm to (71.2, 41.0), turned to 180 degrees
- moved C13 52.1 mm to (74.0, 39.5), turned to 0 degrees
- moved C16 50.9 mm to (74.0, 41.0), turned to 0 degrees
- moved U2 49.4 mm to (73.2, 44.0), turned to -90 degrees
- moved C11 47.5 mm to (72.9, 47.0), turned to 0 degrees
- moved R6 46.1 mm to (75.4, 44.9), turned to -90 degrees
Connections:
- C11 pad 2: gnd-1 -> gnd
- C12 pad 2: gnd-1 -> gnd
- C13 pad 2: gnd-1 -> gnd
- C14 pad 2: gnd-1 -> gnd
- C15 pad 2: gnd-1 -> gnd
- C16 pad 2: gnd-1 -> gnd
- D1 pad 1: gnd-1 -> gnd
- D1 pad 2: line-5 -> line-2
- D1 pad 3: line-9 -> line-3
- D2 pad 1: gnd-1 -> gnd
- D2 pad 2: line-4 -> line-7
- D2 pad 3: line-1 -> line-4
- D3 pad 1: gnd-1 -> gnd
- D3 pad 2: line-2 -> line-5
- D3 pad 3: line -> line-10
- D4 pad 1: gnd-1 -> gnd
- D4 pad 3: line-3 -> line-9
- D5 pad 1: gnd-1 -> gnd
- D5 pad 2: line-8 -> line-1
- D5 pad 3: line-10 -> line
- R6 pad 2: gnd-1 -> gnd
- U1 pad 1: line-5 -> line-2
- U1 pad 12: line-7 -> line-8
- U1 pad 2: line-9 -> line-3
- U1 pad 3: line-4 -> line-7
- U1 pad 30: line-8 -> line-1
- U1 pad 31: line-10 -> line
- U1 pad 4: line-1 -> line-4
- U1 pad 6: line-2 -> line-5
- U1 pad 7: line -> line-10
- U1 pad 9: line-3 -> line-9
- U2 pad 2: gnd-1 -> gnd
- U2 pad 3: EN_ENh -> line-8
Routing:
- net hv: track 11.0 -> 40.8 mm, vias 4 -> 6
- net gnd: track 7.13 -> 34.9 mm, vias 4 -> 20
- net gnd-1: track 19.8 -> 0.00 mm, vias 10 -> 0
- net line-8: track 6.77 -> 16.9 mm
- net line-7: track 0.00 -> 3.90 mm
- net line-1: track 3.90 -> 6.77 mm
- net line-9: track 5.59 -> 7.56 mm
- net line-3: track 7.56 -> 5.59 mm
- net line-5: track 5.66 -> 3.83 mm
- net line-2: track 3.83 -> 5.66 mm
- net line-10: track 6.19 -> 5.28 mm
- net line: track 5.28 -> 6.19 mm

Commit message: layout tidyup
Routing:
- net line-8: track 16.9 -> 10.3 mm
- net gnd: track 34.9 -> 31.2 mm
Changed lines of the file:
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@@
 	)
 	(segment
-		(start 74.925 47.475)
-		(end 74.925 46.075)
+		(start 73.625 44.125)
+		(end 74.15 44.65)
+		(width 0.15)
+		(layer "F.Cu")
+		(net 34)
+	)
+	(segment
+		(start 66.785 42.3)
+		(end 67.005 42.08)
+		(width 0.15)
+		(layer "F.Cu")
+		(net 34)
+	)
+	(segment
+		(start 74.15 44.65)
+		(end 74.15 45.3)
+		(width 0.15)
+		(layer "F.Cu")
+		(net 34)
+	)
+	(segment
+		(start 65.66 42.3)
+		(end 66.785 42.3)
 		(width 0.15)
 		(layer "F.Cu")
@@
 	)
 	(segment
-		(start 65.66 42.3)
-		(end 66.785 42.3)
-		(width 0.15)
-		(layer "F.Cu")
-		(net 34)
-	)
-	(segment
-		(start 74.925 46.075)
-		(end 74.15 45.3)
-		(width 0.15)
-		(layer "F.Cu")
-		(net 34)
-	)
-	(segment
 		(start 71.3 44.125)
-		(end 71.3 47.3)
-		(width 0.15)
-		(layer "F.Cu")
-		(net 34)
-	)
-	(segment
-		(start 66.785 42.3)
-		(end 67.005 42.08)
-		(width 0.15)
-		(layer "F.Cu")
-		(net 34)
-	)
-	(segment
-		(start 73.8 48.6)
-		(end 74.925 47.475)
-		(width 0.15)
-		(layer "F.Cu")
-		(net 34)
-	)
-	(segment
-		(start 71.3 47.3)
-		(end 72.6 48.6)
-		(width 0.15)
-		(layer "F.Cu")
-		(net 34)
-	)
-	(segment
-		(start 72.6 48.6)
-		(end 73.8 48.6)
+		(end 73.625 44.125)
 		(width 0.15)
 		(layer "F.Cu")
@@
 	)
 	(segment
-		(start 73.2 45.3)
-		(end 73.2 44.2)
-		(width 0.5)
-		(layer "F.Cu")
-		(net 35)
-	)
-	(segment
 		(start 69.575 43.575)
 		(end 69.775 43.775)
@@
 	)
 	(segment
-		(start 73.2 44.2)
-		(end 73.175 44.175)
-		(width 0.2)
-		(layer "F.Cu")
-		(net 35)
-	)
-	(segment
 		(start 63.825 35.025)
 		(end 63.775 34.975)
@@
 	)
 	(segment
-		(start 75.028192 45.03)
-		(end 74.805 45.03)
-		(width 0.2)
-		(layer "F.Cu")
-		(net 35)
-	)
-	(segment
 		(start 70.5 38.25)
 		(end 70.525 38.275)
@@
 	)
 	(segment
-		(start 74.805 45.03)
-		(end 74.75 44.975)
-		(width 0.2)
-		(layer "F.Cu")
-		(net 35)
-	)
-	(segment
 		(start 64.05 46.9)
 		(end 64.075 46.925)
@@
 	)
 	(segment
-		(start 74.75 44.625)
-		(end 74.3 44.175)
-		(width 0.2)
-		(layer "F.Cu")
-		(net 35)
-	)
-	(segment
 		(start 56.375 38.05)
 		(end 56.625 38.3)
@@
 	)
 	(segment
-		(start 75.375 45.305)
-		(end 75.303192 45.305)
+		(start 73.2 44.65)
+		(end 73.35 44.5)
+		(width 0.2)
+		(layer "F.Cu")
+		(net 35)
+	)
+	(segment
+		(start 75.303192 45.305)
+		(end 75.375 45.305)
 		(width 0.2)
 		(layer "F.Cu")
@@
 	)
 	(segment
-		(start 74.3 44.175)
-		(end 73.175 44.175)
-		(width 0.2)
-		(layer "F.Cu")
-		(net 35)
-	)
-	(segment
 		(start 67.35 45.975)
 		(end 67.35 46.25)
@@
 	)
 	(segment
-		(start 74.75 44.975)
-		(end 74.75 44.625)
-		(width 0.2)
-		(layer "F.Cu")
-		(net 35)
-	)
-	(segment
-		(start 75.303192 45.305)
-		(end 75.028192 45.03)
-		(width 0.2)
-		(layer "F.Cu")
-		(net 35)
-	)
-	(segment
 		(start 58.025 46.125)
 		(end 58.25 46.125)
@@
 	)
 	(via
-		(at 73.175 44.175)
+		(at 73.2 44.65)
 		(size 0.6)
 		(drill 0.3)
@@
 			"19d6b2d6-e1f5-4d9a-be19-5b2c2a3370ec" "1caa8069-fdd2-4083-be2d-496adf27ed24"
 			"24a15252-b06b-42e4-be44-e97aea6cce9d" "250bb4a9-76f4-46a7-b905-28574023cd18"
-			"2b0928c8-e0a5-41a7-8d62-b19e1bc4b049" "320fda52-bb4d-4832-af60-f1a24642524b"
-			"3ce7b724-c8f5-4102-a2d2-682a90efb5f7" "3fe76845-367e-4038-a962-19be70e7466a"
-			"4c8ac7e3-4541-4ea5-aa7a-77124642524b" "50af49e7-91c7-4afe-947e-093fbf0e2c32"
-			"520adedb-770c-4812-89e0-f2d850ca9332" "53abb1c0-a5e1-441a-86f3-8e10b7b41787"
-			"545cb2e8-3342-47e0-ad08-2aff955b2bd9" "6751a11b-2354-489b-ac09-ef946b8ed0f2"
+			"320fda52-bb4d-4832-af60-f1a24642524b" "3ce7b724-c8f5-4102-a2d2-682a90efb5f7"
+			"3fe76845-367e-4038-a962-19be70e7466a" "4c8ac7e3-4541-4ea5-aa7a-77124642524b"
+			"50af49e7-91c7-4afe-947e-093fbf0e2c32" "520adedb-770c-4812-89e0-f2d850ca9332"
+			"53abb1c0-a5e1-441a-86f3-8e10b7b41787" "6751a11b-2354-489b-ac09-ef946b8ed0f2"
 			"6e807abb-dee8-4361-be8d-bbc0fce6f106" "70ffdc75-84b2-4898-ad9d-cb404642524b"
 			"72b8d446-b06d-484f-ae6b-2813e45056a7" "787d10f5-3a14-4e3b-9b3b-a6254759d8b7"
 			"7d8be784-f945-4483-bf90-93b45ce9000f" "7f809a95-357a-4cc1-9cec-d7f59badd4d6"
 			"88bf4f8a-1fe8-4878-87a2-6811513dc1ab" "8a4ce1df-d803-42c2-a86b-b064ae2d7fb2"
-			"8ee1e9d1-e100-465c-9616-e4267e9db160" "93e238b7-2744-4046-8e8c-6e5c659bfed1"
-			"94c5fe95-0152-4650-8b49-39e6685b9a4b" "98a13876-8285-4467-af73-25801a5dd471"
-			"9a5094c3-48bd-4b2d-957b-796fc0a2e0dc" "a514afd4-e723-466f-a70a-7f51415c208f"
-			"a56281f5-49c5-4f37-9af4-9139737ea795" "a5d1fb4c-a6d7-4b11-8e34-e52162e899ce"
-			"a8dde44c-e7eb-44d9-a023-ea8ff5af35fd" "ac682d2d-3417-4f63-9478-cab84642524b"
-			"b0d39839-f2e1-43d3-88c9-21b3a3394873" "b26a0593-86b5-419c-85ec-1cec1d92305d"
-			"b644a5bf-ffdf-4843-aa5e-3b874642524b" "b7167853-deaa-47ef-87f9-ec6ea9904719"
-			"b96687d7-0d85-4c56-b34a-83528a6dda19" "c0d8d115-b219-4ac3-a0b0-7e0d5a971e92"
-			"c37b2f76-d4f8-4a6c-81ea-2a3d7cfa1fe4" "c6ef68c7-6aa7-4f9e-b738-03f24642524b"
-			"c88ebe01-0a66-4393-b7f3-75533eb7aefa" "cf6d58a1-e0ef-4b66-ae41-426dd4f71788"
-			"d59df8bb-0ea0-435d-8643-74beea1d536f" "d5c9afb2-63bb-4b6a-bcc9-21ba488ff25b"
-			"d7bd9189-246a-447e-a41e-96ec05379fc0" "e164c668-c0f8-4624-8626-b660edbff0b0"
-			"e687e546-3299-4663-ba08-2e9086e6ce2b" "ef4dfe4b-e8ac-4405-a760-dbc7eef1e6cb"
-			"f454287c-8860-4d4c-bc26-299b4642524b" "f4fbb93a-aa3d-4643-b892-c67fce11121e"
-			"f5b948fd-ea96-450e-a968-342a4642524b" "f7375d91-51cd-4745-aa53-07687198f48b"
-			"f8b57edc-de4e-4066-886c-d93c86a18c98" "fad56a40-fa8e-479f-aa7d-3c1247a24d21"
-			"fec68bbb-3478-4dc0-9c3b-938ead3dc96b"
+			"8ee1e9d1-e100-465c-9616-e4267e9db160" "94c5fe95-0152-4650-8b49-39e6685b9a4b"
+			"98a13876-8285-4467-af73-25801a5dd471" "9a5094c3-48bd-4b2d-957b-796fc0a2e0dc"
+			"a514afd4-e723-466f-a70a-7f51415c208f" "a56281f5-49c5-4f37-9af4-9139737ea795"
+			"a5d1fb4c-a6d7-4b11-8e34-e52162e899ce" "a8dde44c-e7eb-44d9-a023-ea8ff5af35fd"
+			"ac682d2d-3417-4f63-9478-cab84642524b" "b0d39839-f2e1-43d3-88c9-21b3a3394873"
+			"b26a0593-86b5-419c-85ec-1cec1d92305d" "b644a5bf-ffdf-4843-aa5e-3b874642524b"
+			"b7167853-deaa-47ef-87f9-ec6ea9904719" "b96687d7-0d85-4c56-b34a-83528a6dda19"
+			"c0d8d115-b219-4ac3-a0b0-7e0d5a971e92" "c37b2f76-d4f8-4a6c-81ea-2a3d7cfa1fe4"
+			"c6ef68c7-6aa7-4f9e-b738-03f24642524b" "cf6d58a1-e0ef-4b66-ae41-426dd4f71788"
+			"d5c9afb2-63bb-4b6a-bcc9-21ba488ff25b" "d94a344d-7c1f-4d43-a2ef-c9bbeaba5530"
+			"dccf4e25-a992-40e4-a520-1e9e4226aee5" "e164c668-c0f8-4624-8626-b660edbff0b0"
+			"e687e546-3299-4663-ba08-2e9086e6ce2b" "f454287c-8860-4d4c-bc26-299b4642524b"
+			"f4fbb93a-aa3d-4643-b892-c67fce11121e" "f5b948fd-ea96-450e-a968-342a4642524b"
+			"f7375d91-51cd-4745-aa53-07687198f48b" "f8b57edc-de4e-4066-886c-d93c86a18c98"
 		)
 	)
