File: elec/layout/cellsim-16ch/cellsim-16ch.kicad_pcb (KiCad board)
At the start: 6 copper layers, 1.5 x 9.6 mm, 1266 parts, among them U244 10µH ±20%

Commit message: fix build warnings
Parts:
- moved C1 3.77 mm to (62.6, 41.3)
- moved C4 3.77 mm to (52.1, 41.0)
- moved U1 3.77 mm to (60.6, 37.8)
- moved U4 3.77 mm to (60.6, 24.1)
- moved C2 3.77 mm to (59.8, 29.1)
- moved C3 3.77 mm to (59.5, 34.6)
- moved C5 3.77 mm to (51.9, 18.9)
- moved C6 3.77 mm to (55.8, 16.8)
- moved C7 3.77 mm to (63.0, 29.5)
- moved C8 3.77 mm to (59.2, 19.6)
- moved D1 3.77 mm to (60.0, 16.7)
- moved R1 3.77 mm to (57.4, 16.9)
- moved R2 3.77 mm to (62.4, 16.9)
- moved U2 3.77 mm to (59.9, 32.0)
- moved U3 3.77 mm to (51.5, 31.2)
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Routing:
- net hil_core-line-6: track 58.7 -> 60.2 mm
- net hil_core-line-13: track 53.8 -> 55.3 mm
