File: elec/layout/usb251b/usb251b.kicad_pcb (KiCad board)
At the start: 2 copper layers, 17 parts

Commit message: building frozen
Connections:
- net line renamed USBDP_DN4_PRT_DIS_P4
- net line-1 renamed SDA_SMBBATA_NON_REM1
- net line-2 renamed SCL_SMBCLK_CFG_SEL0
