File: elec/layout/micro-vault/micro-vault.kicad_pcb (KiCad board)
At the start: 2 copper layers, 28 x 20 mm, 32 parts

Commit message: Build everything with ordered params to fix frozen builds
Connections:
- net IN1minus renamed TEMP
- C1 pad 1: hv-3 -> hv
- C2 pad 1: hv-3 -> hv
- C8 pad 1: hv -> hv-3
- R12 pad 1: heater_controller-net -> heater_controller-net-3
- R12 pad 2: heater_controller-net-4 -> heater_controller-net-2
- R13 pad 1: heater_controller-net-4 -> heater_controller-net-2
- R13 pad 2: heater_controller-net-1 -> heater_controller-net
- R14 pad 1: heater_controller-net-1 -> heater_controller-net
- R2 pad 1: hv -> hv-3
- R2 pad 2: heater_controller-net-2 -> heater_controller-net-4
- R3 pad 1: heater_controller-net-2 -> heater_controller-net-4
- R3 pad 2: heater_controller-net-3 -> heater_controller-net-1
- R4 pad 1: heater_controller-net-3 -> heater_controller-net-1
- R5 pad 2: heater_controller-net -> heater_controller-net-3
- U2 pad 1: hv-3 -> hv
- U3 pad 12: hv-3 -> hv
- U7 pad 1: hv -> hv-3
- U7 pad 3: hv -> hv-3
Routing:
- net hv-3: track 7.33 -> 20.6 mm
- net hv: track 20.6 -> 7.33 mm
- net heater_controller-net-1: track 10.5 -> 3.62 mm, vias 2 -> 0
- net heater_controller-net: track 4.25 -> 10.5 mm, vias 0 -> 2
- net heater_controller-net-4: track 4.99 -> 6.47 mm
- net heater_controller-net-2: track 6.47 -> 4.99 mm
- net heater_controller-net-3: track 3.62 -> 4.25 mm
