File: elec/layout/saleae-header/saleae-header.kicad_pcb (KiCad board)
At the start: 2 copper layers, 5 parts

Commit message: Build everything with ordered params to fix frozen builds
Connections:
- R1 pad 1: line -> line-1
- R1 pad 2: net -> net-3
- R2 pad 1: line-3 -> line-2
- R2 pad 2: net-2 -> net-1
- R3 pad 1: line-2 -> line-3
- R3 pad 2: net-1 -> net-2
- R4 pad 1: line-1 -> line
- R4 pad 2: net-3 -> net
- U1 pad 1: net -> net-3
- U1 pad 3: net-2 -> net-1
- U1 pad 5: net-1 -> net-2
- U1 pad 7: net-3 -> net
Changed lines of the file:
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@@
     )
     (net 0 "")
-    (net 1 "net")
-    (net 2 "line-3")
-    (net 3 "line-2")
-    (net 4 "net-3")
-    (net 5 "net-1")
-    (net 6 "line-1")
+    (net 1 "net-3")
+    (net 2 "line-2")
+    (net 3 "line-3")
+    (net 4 "net")
+    (net 5 "net-2")
+    (net 6 "line")
     (net 7 "gnd")
-    (net 8 "line")
-    (net 9 "net-2")
+    (net 8 "line-1")
+    (net 9 "net-1")
     (footprint "atopile:R0402-56259e"
         (layer "F.Cu")
@@
             )
         )
+        (property "PARAM_max_power" "{\"type\": \"Quantity_Set_Discrete\", \"data\": {\"intervals\": {\"type\": \"Numeric_Interval_Disjoint\", \"data\": {\"intervals\": [{\"type\": \"Numeric_Interval\", \"data\": {\"min\": 0.0625, \"max\": 0.0625}}]}}, \"unit\": \"watt\"}}"
+            (at 0 0 0)
+            (layer "User.9")
+            (hide yes)
+            (effects
+                (font
+                    (size 0.125 0.125)
+                    (thickness 0.01875)
+                )
+            )
+        )
+        (property "PARAM_resistance" "{\"type\": \"Quantity_Interval_Disjoint\", \"data\": {\"intervals\": {\"type\": \"Numeric_Interval_Disjoint\", \"data\": {\"intervals\": [{\"type\": \"Numeric_Interval\", \"data\": {\"min\": 99.00000002235174, \"max\": 100.99999997764826}}]}}, \"unit\": \"ohm\"}}"
+            (at 0 0 0)
+            (layer "User.9")
+            (hide yes)
+            (effects
+                (font
+                    (size 0.125 0.125)
+                    (thickness 0.01875)
+                )
+            )
+        )
+        (property "PARAM_max_voltage" "{\"type\": \"Quantity_Set_Discrete\", \"data\": {\"intervals\": {\"type\": \"Numeric_Interval_Disjoint\", \"data\": {\"intervals\": [{\"type\": \"Numeric_Interval\", \"data\": {\"min\": 50.0, \"max\": 50.0}}]}}, \"unit\": \"volt\"}}"
+            (at 0 0 0)
+            (layer "User.9")
+            (hide yes)
+            (effects
+                (font
+                    (size 0.125 0.125)
+                    (thickness 0.01875)
+                )
+            )
+        )
         (attr smd)
         (fp_line
@@
             (size 0.57 0.54)
             (layers "F.Cu" "F.Mask" "F.Paste")
-            (net 6 "line-1")
+            (net 6 "line")
         )
         (pad "2" smd rect
@@
             (size 0.57 0.54)
             (layers "F.Cu" "F.Mask" "F.Paste")
-            (net 4 "net-3")
+            (net 4 "net")
         )
         (embedded_fonts no)
@@
             )
         )
+        (property "PARAM_max_power" "{\"type\": \"Quantity_Set_Discrete\", \"data\": {\"intervals\": {\"type\": \"Numeric_Interval_Disjoint\", \"data\": {\"intervals\": [{\"type\": \"Numeric_Interval\", \"data\": {\"min\": 0.0625, \"max\": 0.0625}}]}}, \"unit\": \"watt\"}}"
+            (at 0 0 0)
+            (layer "User.9")
+            (hide yes)
+            (effects
+                (font
+                    (size 0.125 0.125)
+                    (thickness 0.01875)
+                )
+            )
+        )
+        (property "PARAM_resistance" "{\"type\": \"Quantity_Interval_Disjoint\", \"data\": {\"intervals\": {\"type\": \"Numeric_Interval_Disjoint\", \"data\": {\"intervals\": [{\"type\": \"Numeric_Interval\", \"data\": {\"min\": 99.00000002235174, \"max\": 100.99999997764826}}]}}, \"unit\": \"ohm\"}}"
+            (at 0 0 0)
+            (layer "User.9")
+            (hide yes)
+            (effects
+                (font
+                    (size 0.125 0.125)
+                    (thickness 0.01875)
+                )
+            )
+        )
+        (property "PARAM_max_voltage" "{\"type\": \"Quantity_Set_Discrete\", \"data\": {\"intervals\": {\"type\": \"Numeric_Interval_Disjoint\", \"data\": {\"intervals\": [{\"type\": \"Numeric_Interval\", \"data\": {\"min\": 50.0, \"max\": 50.0}}]}}, \"unit\": \"volt\"}}"
+            (at 0 0 0)
+            (layer "User.9")
+            (hide yes)
+            (effects
+                (font
+                    (size 0.125 0.125)
+                    (thickness 0.01875)
+                )
+            )
+        )
         (attr smd)
         (fp_line
@@
             (size 0.57 0.54)
             (layers "F.Cu" "F.Mask" "F.Paste")
-            (net 8 "line")
+            (net 8 "line-1")
         )
         (pad "2" smd rect
@@
             (size 0.57 0.54)
             (layers "F.Cu" "F.Mask" "F.Paste")
-            (net 1 "net")
+            (net 1 "net-3")
         )
         (embedded_fonts no)
@@
             (size 1.27 2.8)
             (layers "F.Cu" "F.Mask" "F.Paste")
-            (net 1 "net")
+            (net 1 "net-3")
         )
         (pad "2" smd rect
@@
             (size 1.27 2.8)
             (layers "F.Cu" "F.Mask" "F.Paste")
-            (net 9 "net-2")
+            (net 9 "net-1")
         )
         (pad "4" smd rect
@@
             (size 1.27 2.8)
             (layers "F.Cu" "F.Mask" "F.Paste")
-            (net 5 "net-1")
+            (net 5 "net-2")
         )
         (pad "6" smd rect
@@
             (size 1.27 2.8)
             (layers "F.Cu" "F.Mask" "F.Paste")
-            (net 4 "net-3")
+            (net 4 "net")
         )
         (pad "8" smd rect
@@
             )
         )
+        (property "PARAM_max_power" "{\"type\": \"Quantity_Set_Discrete\", \"data\": {\"intervals\": {\"type\": \"Numeric_Interval_Disjoint\", \"data\": {\"intervals\": [{\"type\": \"Numeric_Interval\", \"data\": {\"min\": 0.0625, \"max\": 0.0625}}]}}, \"unit\": \"watt\"}}"
+            (at 0 0 0)
+            (layer "User.9")
+            (hide yes)
+            (effects
+                (font
+                    (size 0.125 0.125)
+                    (thickness 0.01875)
+                )
+            )
+        )
+        (property "PARAM_resistance" "{\"type\": \"Quantity_Interval_Disjoint\", \"data\": {\"intervals\": {\"type\": \"Numeric_Interval_Disjoint\", \"data\": {\"intervals\": [{\"type\": \"Numeric_Interval\", \"data\": {\"min\": 99.00000002235174, \"max\": 100.99999997764826}}]}}, \"unit\": \"ohm\"}}"
+            (at 0 0 0)
+            (layer "User.9")
+            (hide yes)
+            (effects
+                (font
+                    (size 0.125 0.125)
+                    (thickness 0.01875)
+                )
+            )
+        )
+        (property "PARAM_max_voltage" "{\"type\": \"Quantity_Set_Discrete\", \"data\": {\"intervals\": {\"type\": \"Numeric_Interval_Disjoint\", \"data\": {\"intervals\": [{\"type\": \"Numeric_Interval\", \"data\": {\"min\": 50.0, \"max\": 50.0}}]}}, \"unit\": \"volt\"}}"
+            (at 0 0 0)
+            (layer "User.9")
+            (hide yes)
+            (effects
+                (font
+                    (size 0.125 0.125)
+                    (thickness 0.01875)
+                )
+            )
+        )
         (attr smd)
         (fp_line
@@
             (size 0.57 0.54)
             (layers "F.Cu" "F.Mask" "F.Paste")
-            (net 3 "line-2")
+            (net 3 "line-3")
         )
         (pad "2" smd rect
@@
             (size 0.57 0.54)
             (layers "F.Cu" "F.Mask" "F.Paste")
-            (net 5 "net-1")
+            (net 5 "net-2")
         )
         (embedded_fonts no)
@@
             )
         )
+        (property "PARAM_max_power" "{\"type\": \"Quantity_Set_Discrete\", \"data\": {\"intervals\": {\"type\": \"Numeric_Interval_Disjoint\", \"data\": {\"intervals\": [{\"type\": \"Numeric_Interval\", \"data\": {\"min\": 0.0625, \"max\": 0.0625}}]}}, \"unit\": \"watt\"}}"
+            (at 0 0 0)
+            (layer "User.9")
+            (hide yes)
+            (effects
+                (font
+                    (size 0.125 0.125)
+                    (thickness 0.01875)
+                )
+            )
+        )
+        (property "PARAM_resistance" "{\"type\": \"Quantity_Interval_Disjoint\", \"data\": {\"intervals\": {\"type\": \"Numeric_Interval_Disjoint\", \"data\": {\"intervals\": [{\"type\": \"Numeric_Interval\", \"data\": {\"min\": 99.00000002235174, \"max\": 100.99999997764826}}]}}, \"unit\": \"ohm\"}}"
+            (at 0 0 0)
+            (layer "User.9")
+            (hide yes)
+            (effects
+                (font
+                    (size 0.125 0.125)
+                    (thickness 0.01875)
+                )
+            )
+        )
+        (property "PARAM_max_voltage" "{\"type\": \"Quantity_Set_Discrete\", \"data\": {\"intervals\": {\"type\": \"Numeric_Interval_Disjoint\", \"data\": {\"intervals\": [{\"type\": \"Numeric_Interval\", \"data\": {\"min\": 50.0, \"max\": 50.0}}]}}, \"unit\": \"volt\"}}"
+            (at 0 0 0)
+            (layer "User.9")
+            (hide yes)
+            (effects
+                (font
+                    (size 0.125 0.125)
+                    (thickness 0.01875)
+                )
+            )
+        )
         (attr smd)
         (fp_line
@@
             (size 0.57 0.54)
             (layers "F.Cu" "F.Mask" "F.Paste")
-            (net 2 "line-3")
+            (net 2 "line-2")
         )
         (pad "2" smd rect
@@
             (size 0.57 0.54)
             (layers "F.Cu" "F.Mask" "F.Paste")
-            (net 9 "net-2")
+            (net 9 "net-1")
         )
         (embedded_fonts no)

Commit message: Update saleae header resistance
Parts:
- R1, R2, R3, R4: value 100Ω ±1% 62.5mW -> 1kΩ ±1% 62.5mW
Connections:
- R1 pad 1: line-1 -> line-2
- R1 pad 2: net-3 -> net
- R2 pad 1: line-2 -> line-3
- R3 pad 1: line-3 -> line
- R3 pad 2: net-2 -> net-3
- R4 pad 1: line -> line-1
- R4 pad 2: net -> net-2
- U1 pad 1: net-3 -> net
- U1 pad 5: net-2 -> net-3
- U1 pad 7: net -> net-2

Commit message: checkin
Connections:
- R1 pad 2: net -> net-2
- R2 pad 1: line-3 -> line-1
- R2 pad 2: net-1 -> net-3
- R3 pad 1: line -> line-3
- R3 pad 2: net-3 -> net
- R4 pad 1: line-1 -> line
- R4 pad 2: net-2 -> net-1
- U1 pad 1: net -> net-2
- U1 pad 3: net-1 -> net-3
- U1 pad 5: net-3 -> net
- U1 pad 7: net-2 -> net-1
