File: elec/layout/black-magic-debugger/black-magic-debugger.kicad_pcb (KiCad board)
At the start: 2 copper layers, 52 parts

Commit message: build with excluded checks
Connections:
- net S2 renamed S1
- C15 pad 1: line -> line-10
- D1 pad 1: anode-1 -> anode
- D2 pad 1: anode -> anode-1
- R10 pad 1: line-14 -> line-13
- R14 pad 2: line-10 -> line-8
- R15 pad 1: B2 -> B2-1
- R15 pad 2: line-5 -> line-4
- R16 pad 2: line-13 -> line-5
- R17 pad 2: line-1 -> line-14
- R18 pad 2: line-13 -> line-5
- R2 pad 1: line-9 -> line-3
- R20 pad 1: line-6 -> line-11
- R21 pad 2: line-6 -> line-11
- R22 pad 1: line -> line-10
- R23 pad 2: line -> line-10
- R25 pad 1: B2-2 -> B2
- R25 pad 2: line-4 -> line-7
- R26 pad 1: B2-1 -> B2-2
- R26 pad 2: line-15 -> line-6
- R3 pad 1: line-14 -> line-13
- U1 pad 13: line-2 -> line-9
- U1 pad 14: line-11 -> line-15
- U1 pad 15: line-12 -> line-1
- U1 pad 16: line-8 -> line
- U1 pad 18: line -> line-10
- U1 pad 20: anode-1 -> anode
- U1 pad 21: anode -> anode-1
- U1 pad 26: line-6 -> line-11
- U1 pad 30: line-3 -> line-12
- U1 pad 31: line-7 -> line-2
- U2 pad 3: line-3 -> line-12
- U2 pad 6: B2-1 -> B2-2
- U3 pad 2: line-12 -> line-1
- U3 pad 3: line-2 -> line-9
- U3 pad 6: B2 -> B2-1
- U4 pad 2: line-8 -> line
- U4 pad 3: line-7 -> line-2
- U4 pad 6: B2-2 -> B2
- U5 pad 3: line-11 -> line-15
Routing:
- net line-5: track 0.00 -> 23.7 mm, vias 0 -> 2
- net line-7: track 19.9 -> 0.00 mm, vias 2 -> 0
- net line-3: track 22.2 -> 3.41 mm, vias 2 -> 0
- net line-8: track 17.1 -> 0.00 mm
- net line-15: track 0.00 -> 16.5 mm, vias 0 -> 2
- net line-1: track 0.00 -> 14.1 mm, vias 0 -> 2
- net line-11: track 16.5 -> 2.58 mm, vias 2 -> 0
- net line-13: track 23.7 -> 10.5 mm
- net line-14: track 10.5 -> 0.00 mm, vias 2 -> 0
- net line: track 7.33 -> 17.1 mm
- net line-2: track 10.8 -> 19.9 mm
- net line-12: track 14.1 -> 22.2 mm
- net line-9: track 3.41 -> 10.8 mm, vias 0 -> 2
- net line-10: track 0.00 -> 7.33 mm
- net line-6: track 2.58 -> 0.00 mm
Changed lines of the file:
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@@
     (net 0 "")
     (net 1 "PC14_OSC32_IN")
-    (net 2 "line-9")
+    (net 2 "line-3")
     (net 3 "NRST")
     (net 4 "PB8")
@@
     (net 16 "xout")
     (net 17 "PA11")
-    (net 19 "line")
+    (net 19 "line-10")
     (net 20 "gnd")
     (net 21 "hv-1")
@@
     (net 24 "PB4")
     (net 25 "PB5")
-    (net 26 "line-1")
-    (net 27 "line-13")
-    (net 28 "S2")
-    (net 29 "line-6")
+    (net 26 "line-14")
+    (net 27 "line-5")
+    (net 28 "S1")
+    (net 29 "line-11")
     (net 30 "G2")
     (net 31 "D1")
     (net 32 "PB3")
     (net 33 "B1")
-    (net 34 "B2")
+    (net 34 "B2-1")
     (net 35 "B1-1")
     (net 36 "D2")
-    (net 37 "line-5")
+    (net 37 "line-4")
     (net 38 "PA8")
-    (net 39 "line-14")
-    (net 40 "line-8")
-    (net 41 "line-11")
+    (net 39 "line-13")
+    (net 40 "line")
+    (net 41 "line-15")
     (net 42 "VCCB")
-    (net 43 "line-10")
+    (net 43 "line-8")
     (net 44 "PB12")
     (net 45 "hv-2")
     (net 46 "PB6")
-    (net 47 "line-2")
-    (net 48 "line-12")
+    (net 47 "line-9")
+    (net 48 "line-1")
     (net 49 "B2-3")
     (net 50 "anode-2")
     (net 51 "led2-cathode")
     (net 52 "led1-cathode")
-    (net 53 "anode")
+    (net 53 "anode-1")
     (net 54 "G1")
     (net 55 "led0-cathode")
-    (net 56 "anode-1")
-    (net 57 "B2-1")
+    (net 56 "anode")
+    (net 57 "B2-2")
     (net 58 "PA13")
-    (net 59 "line-7")
-    (net 60 "line-4")
-    (net 61 "line-15")
-    (net 62 "line-3")
-    (net 63 "B2-2")
+    (net 59 "line-2")
+    (net 60 "line-7")
+    (net 61 "line-6")
+    (net 62 "line-12")
+    (net 63 "B2")
     (net 64 "PA14")
     (net 65 "G1-1")
@@
             (size 0.57 0.54)
             (layers "F.Cu" "F.Mask" "F.Paste")
-            (net 19 "line")
+            (net 19 "line-10")
         )
         (pad "2" smd rect
@@
             (size 0.57 0.54)
             (layers "F.Cu" "F.Mask" "F.Paste")
-            (net 39 "line-14")
+            (net 39 "line-13")
         )
         (pad "2" smd rect
@@
             (size 0.57 0.54)
             (layers "F.Cu" "F.Mask" "F.Paste")
-            (net 27 "line-13")
+            (net 27 "line-5")
         )
         (embedded_fonts no)
@@
             (size 0.9 0.28)
             (layers "F.Cu" "F.Mask" "F.Paste")
-            (net 47 "line-2")
+            (net 47 "line-9")
         )
         (pad "14" smd oval
@@
             (size 0.9 0.28)
             (layers "F.Cu" "F.Mask" "F.Paste")
-            (net 41 "line-11")
+            (net 41 "line-15")
         )
         (pad "15" smd oval
@@
             (size 0.9 0.28)
             (layers "F.Cu" "F.Mask" "F.Paste")
-            (net 48 "line-12")
+            (net 48 "line-1")
         )
         (pad "16" smd oval
@@
             (size 0.9 0.28)
             (layers "F.Cu" "F.Mask" "F.Paste")
-            (net 40 "line-8")
+            (net 40 "line")
         )
         (pad "17" smd oval
@@
             (size 0.9 0.28)
             (layers "F.Cu" "F.Mask" "F.Paste")
-            (net 19 "line")
+            (net 19 "line-10")
         )
         (pad "19" smd oval
@@
             (size 0.9 0.28)
             (layers "F.Cu" "F.Mask" "F.Paste")
-            (net 56 "anode-1")
+            (net 56 "anode")
         )
         (pad "21" smd oval
@@
             (size 0.9 0.28)
             (layers "F.Cu" "F.Mask" "F.Paste")
-            (net 53 "anode")
+            (net 53 "anode-1")
         )
         (pad "22" smd oval
@@
             (size 0.28 0.9)
             (layers "F.Cu" "F.Mask" "F.Paste")
-            (net 29 "line-6")
+            (net 29 "line-11")
         )
         (pad "27" smd oval
@@
             (size 0.28 0.9)
             (layers "F.Cu" "F.Mask" "F.Paste")
-            (net 62 "line-3")
+            (net 62 "line-12")
         )
         (pad "31" smd oval
@@
             (size 0.28 0.9)
             (layers "F.Cu" "F.Mask" "F.Paste")
-            (net 59 "line-7")
+            (net 59 "line-2")
         )
         (pad "32" smd oval
@@
             (size 0.75 0.25)
             (layers "F.Cu" "F.Mask" "F.Paste")
-            (net 48 "line-12")
+            (net 48 "line-1")
         )
         (pad "3" smd oval
@@
             (size 0.75 0.25)
             (layers "F.Cu" "F.Mask" "F.Paste")
-            (net 47 "line-2")
+            (net 47 "line-9")
         )
         (pad "4" smd oval
@@
             (size 0.75 0.25)
             (layers "F.Cu" "F.Mask" "F.Paste")
-            (net 34 "B2")
+            (net 34 "B2-1")
         )
         (pad "7" smd oval
@@
             (size 0.57 0.54)
             (layers "F.Cu" "F.Mask" "F.Paste")
-            (net 29 "line-6")
+            (net 29 "line-11")
         )
         (embedded_fonts no)
@@
             (size 0.57 0.54)
             (layers "F.Cu" "F.Mask" "F.Paste")
-            (net 26 "line-1")
+            (net 26 "line-14")
         )
         (embedded_fonts no)
@@
             (size 0.57 0.54)
             (layers "F.Cu" "F.Mask" "F.Paste")
-            (net 29 "line-6")
+            (net 29 "line-11")
         )
         (pad "2" smd rect
@@
             (size 0.57 0.54)
             (layers "F.Cu" "F.Mask" "F.Paste")
-            (net 27 "line-13")
+            (net 27 "line-5")
         )
         (embedded_fonts no)
@@
             (size 0.57 0.54)
             (layers "F.Cu" "F.Mask" "F.Paste")
-            (net 43 "line-10")
+            (net 43 "line-8")
         )
         (embedded_fonts no)
@@
             (size 0.75 0.6)
             (layers "F.Cu" "F.Mask" "F.Paste")
-            (net 53 "anode")
+            (net 53 "anode-1")
         )
         (pad "2" smd rect
@@
             (size 0.57 0.54)
             (layers "F.Cu" "F.Mask" "F.Paste")
-            (net 34 "B2")
+            (net 34 "B2-1")
         )
         (pad "2" smd rect
@@
             (size 0.57 0.54)
             (layers "F.Cu" "F.Mask" "F.Paste")
-            (net 37 "line-5")
+            (net 37 "line-4")
         )
         (embedded_fonts no)
@@
             (size 0.57 0.54)
             (layers "F.Cu" "F.Mask" "F.Paste")
-            (net 57 "B2-1")
+            (net 57 "B2-2")
         )
         (pad "2" smd rect
@@
             (size 0.57 0.54)
             (layers "F.Cu" "F.Mask" "F.Paste")
-            (net 61 "line-15")
+            (net 61 "line-6")
         )
         (embedded_fonts no)
@@
             (size 0.75 0.25)
             (layers "F.Cu" "F.Mask" "F.Paste")
-            (net 41 "line-11")
+            (net 41 "line-15")
         )
         (pad "4" smd oval
@@
             (size 0.28 0.68)
             (layers "F.Cu" "F.Mask" "F.Paste")
-            (net 28 "S2")
+            (net 28 "S1")
         )
         (pad "2" smd rect
@@
             (size 0.28 0.68)
             (layers "F.Cu" "F.Mask" "F.Paste")
-            (net 28 "S2")
+            (net 28 "S1")
         )
         (pad "5" smd rect
@@
             (size 0.57 0.54)
             (layers "F.Cu" "F.Mask" "F.Paste")
-            (net 19 "line")
+            (net 19 "line-10")
         )
         (embedded_fonts no)
@@
             (size 0.57 0.54)
             (layers "F.Cu" "F.Mask" "F.Paste")
-            (net 28 "S2")
+            (net 28 "S1")
         )
         (embedded_fonts no)
@@
             (size 0.57 0.54)
             (layers "F.Cu" "F.Mask" "F.Paste")
-            (net 2 "line-9")
+            (net 2 "line-3")
         )
         (pad "2" smd rect
@@
             (size 0.75 0.6)
             (layers "F.Cu" "F.Mask" "F.Paste")
-            (net 56 "anode-1")
+            (net 56 "anode")
         )
         (pad "2" smd rect
@@
             (size 0.79 0.54)
             (layers "F.Cu" "F.Mask" "F.Paste")
-            (net 19 "line")
+            (net 19 "line-10")
         )
         (pad "2" smd rect
@@
             (size 0.57 0.54)
             (layers "F.Cu" "F.Mask" "F.Paste")
-            (net 63 "B2-2")
+            (net 63 "B2")
         )
         (pad "2" smd rect
@@
             (size 0.57 0.54)
             (layers "F.Cu" "F.Mask" "F.Paste")
-            (net 60 "line-4")
+            (net 60 "line-7")
         )
         (embedded_fonts no)
@@
             (size 0.57 0.54)
             (layers "F.Cu" "F.Mask" "F.Paste")
-            (net 39 "line-14")
+            (net 39 "line-13")
         )
         (pad "2" smd rect
@@
             (size 0.75 0.25)
             (layers "F.Cu" "F.Mask" "F.Paste")
-            (net 62 "line-3")
+            (net 62 "line-12")
         )
         (pad "4" smd oval
@@
             (size 0.75 0.25)
             (layers "F.Cu" "F.Mask" "F.Paste")
-            (net 57 "B2-1")
+            (net 57 "B2-2")
         )
         (pad "7" smd oval
@@
             (size 0.75 0.25)
             (layers "F.Cu" "F.Mask" "F.Paste")
-            (net 40 "line-8")
+            (net 40 "line")
         )
         (pad "3" smd oval
@@
             (size 0.75 0.25)
             (layers "F.Cu" "F.Mask" "F.Paste")
-            (net 59 "line-7")
+            (net 59 "line-2")
         )
         (pad "4" smd oval
@@
             (size 0.75 0.25)
             (layers "F.Cu" "F.Mask" "F.Paste")
-            (net 63 "B2-2")
+            (net 63 "B2")
         )
         (pad "7" smd oval
