File: elec/layout/block-tester/block-tester.kicad_pcb (KiCad board)
At the start: 2 copper layers, 389 x 279 mm, 164 parts

Commit message: checkin
Parts:
- added C47: 100nF ±10% 16V X7R, atopile:C0402-b3ef17, F.Cu at (158.2, -23.0)
- added C48: 2.2µF ±10% 16V X5R, atopile:C0603-bd72f6, F.Cu at (158.1, -24.3)
- added C49: 100nF ±10% 16V X7R, atopile:C0402-b3ef17, F.Cu at (176.7, -178.1)
- added C50: 2.2µF ±10% 16V X5R, atopile:C0603-bd72f6, F.Cu at (176.7, -179.5)
- added C51: 100nF ±10% 16V X7R, atopile:C0402-b3ef17, F.Cu at (179.1, -119.5)
- added C52: 2.2µF ±10% 16V X5R, atopile:C0603-bd72f6, F.Cu at (179.1, -120.8)
- added C53: 100nF ±10% 16V X7R, atopile:C0402-b3ef17, F.Cu at (534.4, -75.1)
- added C54: 2.2µF ±10% 16V X5R, atopile:C0603-bd72f6, F.Cu at (534.4, -76.4)
- added C55: 100nF ±10% 16V X7R, atopile:C0402-b3ef17, F.Cu at (542.5, -16.8)
- added C56: 2.2µF ±10% 16V X5R, atopile:C0603-bd72f6, F.Cu at (542.5, -18.1)
- added R100: 10kΩ ±1% 62.5mW, atopile:R0402-56259e, F.Cu at (527.9, -83.3)
- added R101: 10kΩ ±1% 62.5mW, atopile:R0402-56259e, F.Cu at (527.9, -80.2)
- added R102: 10kΩ ±1% 62.5mW, atopile:R0402-56259e, F.Cu at (527.9, -81.2)
- added R103: 10kΩ ±1% 62.5mW, atopile:R0402-56259e, F.Cu at (527.9, -78.1)
- added R104: 10kΩ ±1% 62.5mW, atopile:R0402-56259e, F.Cu at (527.9, -79.1)
- added R105: 10kΩ ±1% 62.5mW, atopile:R0402-56259e, F.Cu at (540.3, -77.0)
- added R106: 10kΩ ±1% 62.5mW, atopile:R0402-56259e, F.Cu at (548.4, -20.9)
- added R107: 10kΩ ±1% 62.5mW, atopile:R0402-56259e, F.Cu at (548.4, -19.8)
- added R108: 10kΩ ±1% 62.5mW, atopile:R0402-56259e, F.Cu at (548.4, -23.0)
- added R109: 10kΩ ±1% 62.5mW, atopile:R0402-56259e, F.Cu at (548.4, -22.0)
- added R110: 10kΩ ±1% 62.5mW, atopile:R0402-56259e, F.Cu at (548.4, -25.2)
- added R111: 10kΩ ±1% 62.5mW, atopile:R0402-56259e, F.Cu at (548.4, -24.1)
- added R112: 10kΩ ±1% 62.5mW, atopile:R0402-56259e, F.Cu at (548.4, -27.3)
- added R113: 10kΩ ±1% 62.5mW, atopile:R0402-56259e, F.Cu at (548.4, -26.3)
- added R114: 10kΩ ±1% 62.5mW, atopile:R0402-56259e, F.Cu at (536.1, -26.1)
- added R115: 10kΩ ±1% 62.5mW, atopile:R0402-56259e, F.Cu at (536.1, -27.2)
- added R116: 10kΩ ±1% 62.5mW, atopile:R0402-56259e, F.Cu at (536.1, -24.0)
- added R117: 10kΩ ±1% 62.5mW, atopile:R0402-56259e, F.Cu at (536.1, -25.1)
- added R118: 10kΩ ±1% 62.5mW, atopile:R0402-56259e, F.Cu at (536.1, -21.9)
- added R119: 10kΩ ±1% 62.5mW, atopile:R0402-56259e, F.Cu at (536.1, -23.0)
- added R120: 10kΩ ±1% 62.5mW, atopile:R0402-56259e, F.Cu at (536.1, -19.9)
- added R121: 10kΩ ±1% 62.5mW, atopile:R0402-56259e, F.Cu at (536.1, -20.9)
- added R122: 10kΩ ±1% 62.5mW, atopile:R0402-56259e, F.Cu at (548.4, -18.7)
- added R38: 10kΩ ±1% 62.5mW, atopile:R0402-56259e, F.Cu at (164.1, -27.1)
- added R39: 10kΩ ±1% 62.5mW, atopile:R0402-56259e, F.Cu at (164.1, -26.0)
- added R40: 10kΩ ±1% 62.5mW, atopile:R0402-56259e, F.Cu at (164.1, -29.2)
- added R41: 10kΩ ±1% 62.5mW, atopile:R0402-56259e, F.Cu at (164.1, -28.1)
- added R42: 10kΩ ±1% 62.5mW, atopile:R0402-56259e, F.Cu at (164.1, -31.4)
- added R43: 10kΩ ±1% 62.5mW, atopile:R0402-56259e, F.Cu at (164.1, -30.3)
- added R44: 10kΩ ±1% 62.5mW, atopile:R0402-56259e, F.Cu at (164.1, -33.5)
- added R45: 10kΩ ±1% 62.5mW, atopile:R0402-56259e, F.Cu at (164.1, -32.4)
- added R46: 10kΩ ±1% 62.5mW, atopile:R0402-56259e, F.Cu at (151.7, -32.3)
- added R47: 10kΩ ±1% 62.5mW, atopile:R0402-56259e, F.Cu at (151.7, -33.3)
- added R48: 10kΩ ±1% 62.5mW, atopile:R0402-56259e, F.Cu at (151.7, -30.2)
- added R49: 10kΩ ±1% 62.5mW, atopile:R0402-56259e, F.Cu at (151.7, -31.3)
- added R50: 10kΩ ±1% 62.5mW, atopile:R0402-56259e, F.Cu at (151.7, -28.1)
- added R51: 10kΩ ±1% 62.5mW, atopile:R0402-56259e, F.Cu at (151.7, -29.2)
- added R52: 10kΩ ±1% 62.5mW, atopile:R0402-56259e, F.Cu at (151.7, -26.0)
- added R53: 10kΩ ±1% 62.5mW, atopile:R0402-56259e, F.Cu at (151.7, -27.1)
- added R54: 10kΩ ±1% 62.5mW, atopile:R0402-56259e, F.Cu at (164.1, -24.9)
- added R55: 10kΩ ±1% 62.5mW, atopile:R0402-56259e, F.Cu at (182.6, -182.2)
- added R56: 10kΩ ±1% 62.5mW, atopile:R0402-56259e, F.Cu at (182.6, -181.1)
- added R57: 10kΩ ±1% 62.5mW, atopile:R0402-56259e, F.Cu at (182.6, -184.4)
- added R58: 10kΩ ±1% 62.5mW, atopile:R0402-56259e, F.Cu at (182.6, -183.3)
- added R59: 10kΩ ±1% 62.5mW, atopile:R0402-56259e, F.Cu at (182.6, -186.5)
- added R60: 10kΩ ±1% 62.5mW, atopile:R0402-56259e, F.Cu at (182.6, -185.4)
- added R61: 10kΩ ±1% 62.5mW, atopile:R0402-56259e, F.Cu at (182.6, -188.7)
- added R62: 10kΩ ±1% 62.5mW, atopile:R0402-56259e, F.Cu at (182.6, -187.6)
- added R63: 10kΩ ±1% 62.5mW, atopile:R0402-56259e, F.Cu at (170.2, -187.4)
- added R64: 10kΩ ±1% 62.5mW, atopile:R0402-56259e, F.Cu at (170.2, -188.5)
- added R65: 10kΩ ±1% 62.5mW, atopile:R0402-56259e, F.Cu at (170.2, -185.4)
- added R66: 10kΩ ±1% 62.5mW, atopile:R0402-56259e, F.Cu at (170.2, -186.4)
- added R67: 10kΩ ±1% 62.5mW, atopile:R0402-56259e, F.Cu at (170.2, -183.3)
- added R68: 10kΩ ±1% 62.5mW, atopile:R0402-56259e, F.Cu at (170.2, -184.3)
- added R69: 10kΩ ±1% 62.5mW, atopile:R0402-56259e, F.Cu at (170.2, -181.2)
- added R70: 10kΩ ±1% 62.5mW, atopile:R0402-56259e, F.Cu at (170.2, -182.2)
- added R71: 10kΩ ±1% 62.5mW, atopile:R0402-56259e, F.Cu at (182.6, -180.1)
- added R72: 10kΩ ±1% 62.5mW, atopile:R0402-56259e, F.Cu at (185.1, -123.6)
- added R73: 10kΩ ±1% 62.5mW, atopile:R0402-56259e, F.Cu at (185.1, -122.5)
- added R74: 10kΩ ±1% 62.5mW, atopile:R0402-56259e, F.Cu at (185.1, -125.7)
- added R75: 10kΩ ±1% 62.5mW, atopile:R0402-56259e, F.Cu at (185.1, -124.7)
- added R76: 10kΩ ±1% 62.5mW, atopile:R0402-56259e, F.Cu at (185.1, -127.9)
- added R77: 10kΩ ±1% 62.5mW, atopile:R0402-56259e, F.Cu at (185.1, -126.8)
- added R78: 10kΩ ±1% 62.5mW, atopile:R0402-56259e, F.Cu at (185.1, -130.0)
- added R79: 10kΩ ±1% 62.5mW, atopile:R0402-56259e, F.Cu at (185.1, -129.0)
- added R80: 10kΩ ±1% 62.5mW, atopile:R0402-56259e, F.Cu at (172.7, -128.8)
- added R81: 10kΩ ±1% 62.5mW, atopile:R0402-56259e, F.Cu at (172.7, -129.9)
- added R82: 10kΩ ±1% 62.5mW, atopile:R0402-56259e, F.Cu at (172.7, -126.7)
- added R83: 10kΩ ±1% 62.5mW, atopile:R0402-56259e, F.Cu at (172.7, -127.8)
- added R84: 10kΩ ±1% 62.5mW, atopile:R0402-56259e, F.Cu at (172.7, -124.6)
- added R85: 10kΩ ±1% 62.5mW, atopile:R0402-56259e, F.Cu at (172.7, -125.7)
- added R86: 10kΩ ±1% 62.5mW, atopile:R0402-56259e, F.Cu at (172.7, -122.6)
- added R87: 10kΩ ±1% 62.5mW, atopile:R0402-56259e, F.Cu at (172.7, -123.6)
- added R88: 10kΩ ±1% 62.5mW, atopile:R0402-56259e, F.Cu at (185.1, -121.4)
- added R89: 10kΩ ±1% 62.5mW, atopile:R0402-56259e, F.Cu at (540.3, -79.1)
- added R90: 10kΩ ±1% 62.5mW, atopile:R0402-56259e, F.Cu at (540.3, -78.1)
- added R91: 10kΩ ±1% 62.5mW, atopile:R0402-56259e, F.Cu at (540.3, -81.3)
- added R92: 10kΩ ±1% 62.5mW, atopile:R0402-56259e, F.Cu at (540.3, -80.2)
- added R93: 10kΩ ±1% 62.5mW, atopile:R0402-56259e, F.Cu at (540.3, -83.4)
- added R94: 10kΩ ±1% 62.5mW, atopile:R0402-56259e, F.Cu at (540.3, -82.4)
- added R95: 10kΩ ±1% 62.5mW, atopile:R0402-56259e, F.Cu at (540.3, -85.6)
- added R96: 10kΩ ±1% 62.5mW, atopile:R0402-56259e, F.Cu at (540.3, -84.5)
- added R97: 10kΩ ±1% 62.5mW, atopile:R0402-56259e, F.Cu at (527.9, -84.4)
- added R98: 10kΩ ±1% 62.5mW, atopile:R0402-56259e, F.Cu at (527.9, -85.4)
- added R99: 10kΩ ±1% 62.5mW, atopile:R0402-56259e, F.Cu at (527.9, -82.3)
- added U63: , atopile:HDR-TH_10P-P2.54-V-F-f96416, F.Cu at (530.4, -58.1)
- added U64: , atopile:HDR-TH_10P-P2.54-V-F-f96416, F.Cu at (530.4, -104.1)
- added U65: , atopile:QFN-16_L3.0-W3.0-P0.50-BL-EP1.7-3a4c56, F.Cu at (485.8, -76.3)
- added U66: , atopile:QFN-16_L3.0-W3.0-P0.50-BL-EP1.7-3a4c56, F.Cu at (485.8, -86.3)
- added U67: , lib:TSSOP-24_L7.8-W4.4-P0.65-LS6.4-BL, F.Cu at (534.2, -81.5)
- added U68: , atopile:HDR-TH_10P-P2.54-V-F-f96416, F.Cu at (329.3, 0.28)
- added U69: , atopile:HDR-TH_10P-P2.54-V-F-f96416, F.Cu at (329.3, -45.7)
- added U70: , atopile:HDR-TH_10P-P2.54-V-F-f96416, F.Cu at (382.9, 0.70)
- added U71: , atopile:HDR-TH_10P-P2.54-V-F-f96416, F.Cu at (382.9, -45.3)
- added U72: , atopile:HDR-TH_10P-P2.54-V-F-f96416, F.Cu at (434.9, 0.60)
- added U73: , atopile:HDR-TH_10P-P2.54-V-F-f96416, F.Cu at (434.9, -45.4)
- added U74: , atopile:HDR-TH_10P-P2.54-V-F-f96416, F.Cu at (486.8, 0.33)
- added U75: , atopile:HDR-TH_10P-P2.54-V-F-f96416, F.Cu at (486.8, -45.7)
- added U76: , atopile:HDR-TH_10P-P2.54-V-F-f96416, F.Cu at (538.5, 0.15)
- added U77: , atopile:HDR-TH_10P-P2.54-V-F-f96416, F.Cu at (538.5, -45.9)
- added U78: , atopile:QFN-16_L3.0-W3.0-P0.50-BL-EP1.7-3a4c56, F.Cu at (493.9, -18.1)
- added U79: , atopile:QFN-16_L3.0-W3.0-P0.50-BL-EP1.7-3a4c56, F.Cu at (493.9, -28.1)
- added U80: , lib:TSSOP-24_L7.8-W4.4-P0.65-LS6.4-BL, F.Cu at (542.3, -23.2)
- added U81: , atopile:PWRM-TH_L69.5-W39.0_LD30-23B05R2-a2c477, F.Cu at (223.6, 153.8)
- added U82: , atopile:PWRM-TH_L69.5-W39.0_LD30-23B05R2-a2c477, F.Cu at (223.5, 114.5)
- R15: value 10kΩ ±1% 62.5mW -> 560Ω ±1% 62.5mW
- R16: value 18kΩ ±1% 62.5mW -> 1kΩ ±1% 62.5mW
- U1, U2, U3: footprint atopile:HDR-TH_10P-P2.54-V-F-f96416 -> lib:SMD_BD5.6-D4.1-12eb58
- U14, U15, U27, U28, U40, U41: footprint atopile:HDR-TH_10P-P2.54-V-F-f96416 -> atopile:QFN-16_L3.0-W3.0-P0.50-BL-EP1.7-3a4c56
- U16, U29, U42: footprint atopile:HDR-TH_10P-P2.54-V-F-f96416 -> lib:TSSOP-24_L7.8-W4.4-P0.65-LS6.4-BL
- moved U43 429.2 mm to (321.2, -58.0)
- moved U44 429.2 mm to (321.2, -104.0)
- moved U45 427.8 mm to (374.7, -57.5)
- moved U46 427.8 mm to (374.7, -103.5)
- moved U47 425.6 mm to (426.8, -57.6)
- moved U48 425.6 mm to (426.8, -103.7)
- moved U49 423.4 mm to (478.7, -57.9)
- moved U50 423.4 mm to (478.7, -103.9)
- moved U41 396.8 mm to (130.6, -130.8)
- moved U42 382.5 mm to (178.9, -125.9), turned to 90 degrees
- moved U2 375.9 mm to (274.6, 107.4)
- moved U1 366.2 mm to (274.6, 128.6)
- moved U3 322.2 mm to (274.2, 144.1)
- moved U31 309.0 mm to (-34.1, -148.4)
- moved U33 308.5 mm to (19.5, -148.0)
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Connections:
- net DN2 renamed DN1
- net DP2 renamed A6
- net MDI0_ renamed hil_core.controller-pins[9]
- net MDI2_ renamed hil_core.controller-pins[8]
- net base_1_2-line renamed column_0.gpio_expander_2-net-2
- net base_1_2-line-2 renamed column_0.gpio_expander_2-net-1
- net base_1_2-line-3 renamed column_0.gpio_expander_2-net-3
- net base_1_2-line-4 renamed column_0.gpio_expander_2-net-7
- net base_1_2-line-5 renamed column_0.gpio_expander_2-net-5
- net base_1_3-gnd renamed column_1.base_0-gnd
- net base_1_3-hv renamed column_1.base_0-hv-2
- net base_1_3-hv-1 renamed column_1.base_0-hv
- net base_1_3-hv-2 renamed column_1.base_0-hv-1
- net base_1_3-line renamed column_1.base_0-line-5
- net base_1_3-line-1 renamed column_1.base_0-line
- net base_1_3-line-2 renamed column_1.base_0-line-4
- net base_1_3-line-3 renamed column_1.base_0-line-2
- net base_1_3-line-4 renamed column_1.base_0-line-1
- net base_1_3-line-5 renamed column_1.base_0-line-3
- net base_1_4-gnd renamed column_1.base_1-gnd
- net base_1_4-hv renamed column_1.base_1-hv-2
- net base_1_4-hv-1 renamed column_1.base_1-hv
- net base_1_4-hv-2 renamed column_1.base_1-hv-1
- net base_1_4-line renamed column_1.base_1-line-2
- net base_1_4-line-1 renamed column_1.base_1-line-4
- net base_1_4-line-2 renamed column_1.base_1-line
- net base_1_4-line-3 renamed column_1.base_1-line-1
- net base_1_4-line-4 renamed column_1.base_1-line-5
- net base_1_4-line-5 renamed column_1.base_1-line-3
- net base_2_0-gnd renamed column_1.base_2-gnd
- net base_2_0-hv renamed column_1.base_2-hv-1
- net base_2_0-hv-1 renamed column_1.base_2-hv
- net base_2_0-hv-2 renamed column_1.base_2-hv-2
- net base_2_0-line renamed column_1.base_2-line
- net base_2_0-line-1 renamed column_1.base_2-line-5
- net base_2_0-line-2 renamed column_1.base_2-line-2
- net base_2_0-line-3 renamed column_1.base_2-line-3
- net base_2_0-line-4 renamed column_1.base_2-line-1
- net base_2_0-line-5 renamed column_1.base_2-line-4
- net base_2_1-gnd renamed column_1.base_3-gnd
- net base_2_1-hv renamed column_1.base_3-hv-1
- net base_2_1-hv-1 renamed column_1.base_3-hv
- net base_2_1-hv-2 renamed column_1.base_3-hv-2
- net base_2_1-line renamed column_1.base_3-line-3
- net base_2_1-line-1 renamed column_1.base_3-line-1
- net base_2_1-line-2 renamed column_1.base_3-line-2
- net base_2_1-line-3 renamed column_1.base_3-line
- net base_2_1-line-4 renamed column_1.base_3-line-4
- net base_2_1-line-5 renamed column_1.base_3-line-5
- net base_2_2-gnd renamed column_1.base_4-gnd
- net base_2_2-hv renamed column_1.base_4-hv-1
- net base_2_2-hv-1 renamed column_1.base_4-hv-2
- net base_2_2-hv-2 renamed column_1.base_4-hv
- net base_2_2-line renamed column_1.base_4-line-1
- net base_2_2-line-1 renamed column_1.base_4-line-4
- net base_2_2-line-2 renamed column_1.base_4-line-2
- net base_2_2-line-3 renamed column_1.base_4-line-3
- net base_2_2-line-4 renamed column_1.base_4-line
- net base_2_2-line-5 renamed column_1.base_4-line-5
- net base_2_3-line renamed column_1.gpio_expander_1-net-3
- net base_2_3-line-2 renamed column_1.gpio_expander_1-net-2
- net base_2_3-line-3 renamed column_1.gpio_expander_1-net-4
- net base_2_3-line-4 renamed column_1.gpio_expander_1-net
- net base_2_3-line-5 renamed column_1.gpio_expander_1-net-5
- net base_4_0-line renamed column_2.gpio_expander_2-net-6
- net base_4_0-line-1 renamed column_2.gpio_expander_2-net-5
- net base_4_0-line-2 renamed column_2.gpio_expander_2-net-1
- net base_4_0-line-3 renamed column_2.gpio_expander_2-net
- net base_4_0-line-5 renamed column_2.gpio_expander_2-net-7
- net base_4_1-gnd renamed column_3.base_0-gnd
- net base_4_1-hv renamed column_3.base_0-hv-2
- net base_4_1-hv-1 renamed column_3.base_0-hv
- net base_4_1-hv-2 renamed column_3.base_0-hv-1
- net base_4_1-line renamed column_3.base_0-line-3
- net base_4_1-line-1 renamed column_3.base_0-line-5
- net base_4_1-line-2 renamed column_3.base_0-line-4
- net base_4_1-line-3 renamed column_3.base_0-line-2
- net base_4_1-line-4 renamed column_3.base_0-line-1
- net base_4_1-line-5 renamed column_3.base_0-line
- net base_4_2-gnd renamed column_3.base_1-gnd
- net base_4_2-hv renamed column_3.base_1-hv-1
- net base_4_2-hv-1 renamed column_3.base_1-hv-2
- net base_4_2-hv-2 renamed column_3.base_1-hv
- net base_4_2-line renamed column_3.base_1-line
- net base_4_2-line-1 renamed column_3.base_1-line-3
- net base_4_2-line-2 renamed column_3.base_1-line-5
- net base_4_2-line-3 renamed column_3.base_1-line-4
- net base_4_2-line-4 renamed column_3.base_1-line-2
- net base_4_2-line-5 renamed column_3.base_1-line-1
- net base_4_3-gnd renamed column_3.base_2-gnd
- net base_4_3-hv renamed column_3.base_2-hv
- net base_4_3-hv-1 renamed column_3.base_2-hv-1
- net base_4_3-hv-2 renamed column_3.base_2-hv-2
- net base_4_3-line renamed column_3.base_2-line-1
- net base_4_3-line-1 renamed column_3.base_2-line-3
- net base_4_3-line-2 renamed column_3.base_2-line
- net base_4_3-line-3 renamed column_3.base_2-line-4
- net base_4_3-line-4 renamed column_3.base_2-line-5
- net base_4_3-line-5 renamed column_3.base_2-line-2
- net base_4_4-gnd renamed column_3.base_3-gnd
- net base_4_4-hv renamed column_3.base_3-hv-1
- net base_4_4-hv-1 renamed column_3.base_3-hv-2
- net base_4_4-hv-2 renamed column_3.base_3-hv
- net base_4_4-line renamed column_3.base_3-line-1
- net base_4_4-line-1 renamed column_3.base_3-line-2
- net base_4_4-line-2 renamed column_3.base_3-line-5
- net base_4_4-line-3 renamed column_3.base_3-line
- net base_4_4-line-4 renamed column_3.base_3-line-3
- net base_4_4-line-5 renamed column_3.base_3-line-4
- net hil_core-pins[4] renamed pins[4]
- net hil_core.controller-pins[3] renamed MDI1plus
- net hil_core.controller-pins[4] renamed MDI3_
- net hil_core.controller.cm5.hdi_b-pins[3] renamed pins[3]
- net hil_core.usb_connector.connector-A2 renamed A2
- net hil_core.usb_connector.connector-A3 renamed A3
- net hil_core.usb_connector.connector-A8 renamed A8
- net hil_core.usb_connector.connector-B10 renamed B10
- net hil_core.usb_connector.connector-B11 renamed B11
- net hil_core.usb_connector.connector-B2 renamed SSTXP2
- net hil_core.usbpd.usb_connector-A2 renamed SSTXP1
- net hil_core.usbpd.usb_connector-A3 renamed SSTXN1
- net hil_core.usbpd.usb_connector-A8 renamed SBU1
- net hil_core.usbpd.usb_connector-B10 renamed SSRXN1
- net hil_core.usbpd.usb_connector-B11 renamed SSRXP1
- net hil_core.usbpd.usb_connector-B2 renamed B2
- net hv renamed hv-5
- net pins[8] renamed hil_core.controller.cm5.hdi_b-pins[8]
- net pins[9] renamed hil_core.controller.cm5.hdi_b-pins[9]
- C23 pad 1: hv-2 -> hv-6
- C39 pad 1: hv-3 -> hv-2
- C40 pad 1: hv-3 -> hv-2
- C44 pad 2: hil_core.usbpd.pd_controller-hv-1 -> hil_core.usbpd.pd_controller-hv
- C45 pad 2: hil_core.usbpd.pd_controller-hv -> hil_core.usbpd.pd_controller-hv-1
- CN1 pad 23: hil_core-line-3 -> hil_core-line-1
- CN1 pad 25: hil_core-line-1 -> hil_core-line-5
- CN1 pad 27: hil_core.controller.cm5-pins[53]-1 -> hil_core.controller.cm5-pins[53]
- CN1 pad 44: hil_core.controller.cm5-pins[89] -> hil_core.controller.cm5-pins[89]-1
- CN1 pad 45: hil_core.controller.cm5-pins[89] -> hil_core.controller.cm5-pins[89]-1
- CN1 pad 73: hil_core-line-4 -> hil_core-line-2
- CN1 pad 75: hil_core-line-2 -> hil_core-line-4
- CN1 pad 77: hil_core-line -> hil_core-line-3
- CN1 pad 86: hil_core-line-5 -> hil_core-line
- CN2 pad 27: hil_core.controller.cm5-pins[53] -> hil_core.controller.cm5-pins[53]-1
- CN2 pad 45: hil_core.controller.cm5-pins[89]-1 -> hil_core.controller.cm5-pins[89]
- D3 pad 1: hil_core.controller.cm5-cathode-1 -> hil_core.controller.cm5-cathode
- D4 pad 1: hil_core.controller.cm5-cathode -> hil_core.controller.cm5-cathode-1
- D5 pad 2: hil_core.usbpd-line -> hil_core.usbpd-line-3
- OLED1 pad 10: hil_core-line -> hil_core-line-3
- OLED1 pad 11: hil_core-line-3 -> hil_core-line-1
- OLED1 pad 5: hv-2 -> hv-6
- R10 pad 1: hil_core.controller.cm5-cathode -> hil_core.controller.cm5-cathode-1
- R11 pad 2: hil_core.controller.rj45-anode-1 -> hil_core.controller.rj45-anode
- R12 pad 2: hil_core.controller.rj45-anode -> hil_core.controller.rj45-anode-1
- R13 pad 1: hil_core-line -> hil_core-line-3
- R14 pad 1: hil_core-line-3 -> hil_core-line-1
- R19 pad 1: hv-2 -> hv-6
- R33 pad 1: hil_core.usbpd-line-3 -> hil_core.usbpd-line
- R9 pad 1: hil_core.controller.cm5-cathode-1 -> hil_core.controller.cm5-cathode
- RJ1 pad 11: hil_core.controller.rj45-anode-1 -> hil_core.controller.rj45-anode
- RJ1 pad 14: hil_core.controller.rj45-anode -> hil_core.controller.rj45-anode-1
- U1 pad 1: base_0_0-gnd -> ac_in_chassis-net
- U1 pad 2: base_0_0-line-3 -> ac_in_chassis-net
- U1 pad 3: base_0_0-line-5 -> ac_in_chassis-net
- U1 pad 4: base_0_0-gnd -> ac_in_chassis-net
- U10 pad 1: base_0_4-gnd -> column_0.base_3-gnd
- U10 pad 10: base_0_4-gnd -> column_0.base_3-gnd
- U10 pad 2: base_0_4-hv-1 -> column_0.base_3-line-4
- U10 pad 3: base_0_4-hv-1 -> column_0.base_3-line
- U10 pad 4: base_0_4-gnd -> column_0.base_3-gnd
- U10 pad 5: base_0_4-hv-2 -> column_0.base_3-line-1
- U10 pad 6: base_0_4-hv-2 -> column_0.base_3-line-3
- U10 pad 7: base_0_4-gnd -> column_0.base_3-gnd
- U10 pad 8: base_0_4-hv -> column_0.base_3-line-2
- U10 pad 9: base_0_4-hv -> column_0.base_3-line-5
- U11 pad 1: base_1_0-gnd -> column_0.base_3-gnd
- U11 pad 10: base_1_0-gnd -> column_0.base_3-gnd
- U11 pad 2: base_1_0-line -> column_0.base_3-hv-1
- U11 pad 3: base_1_0-line-2 -> column_0.base_3-hv-1
- U11 pad 4: base_1_0-gnd -> column_0.base_3-gnd
- U11 pad 5: base_1_0-line-4 -> column_0.base_3-hv-2
- U11 pad 6: base_1_0-line-5 -> column_0.base_3-hv-2
- U11 pad 7: base_1_0-gnd -> column_0.base_3-gnd
- U11 pad 8: base_1_0-line-1 -> column_0.base_3-hv
- U11 pad 9: base_1_0-line-3 -> column_0.base_3-hv
- U12 pad 1: base_1_0-gnd -> column_0.base_4-gnd
- U12 pad 10: base_1_0-gnd -> column_0.base_4-gnd
- U12 pad 2: base_1_0-hv -> column_0.base_4-line-3
- U12 pad 3: base_1_0-hv -> column_0.base_4-line-5
- U12 pad 4: base_1_0-gnd -> column_0.base_4-gnd
- U12 pad 5: base_1_0-hv-1 -> column_0.base_4-line
- U12 pad 6: base_1_0-hv-1 -> column_0.base_4-line-2
- U12 pad 7: base_1_0-gnd -> column_0.base_4-gnd
- U12 pad 8: base_1_0-hv-2 -> column_0.base_4-line-1
- U12 pad 9: base_1_0-hv-2 -> column_0.base_4-line-4
- U13 pad 1: base_1_1-gnd -> column_0.base_4-gnd
- U13 pad 10: base_1_1-gnd -> column_0.base_4-gnd
- U13 pad 2: base_1_1-line-4 -> column_0.base_4-hv
- U13 pad 3: base_1_1-line -> column_0.base_4-hv
- U13 pad 4: base_1_1-gnd -> column_0.base_4-gnd
- U13 pad 5: base_1_1-line-3 -> column_0.base_4-hv-2
- U13 pad 6: base_1_1-line-5 -> column_0.base_4-hv-2
- U13 pad 7: base_1_1-gnd -> column_0.base_4-gnd
- U13 pad 8: base_1_1-line-2 -> column_0.base_4-hv-1
- U13 pad 9: base_1_1-line-1 -> column_0.base_4-hv-1
- U14 pad 1: base_1_1-gnd -> column_0.gpio_expander_1-VCCI
- U14 pad 10: base_1_1-gnd -> column_0.gpio_expander_1-net-7
- U14 pad 2: base_1_1-hv-2 -> column_0.gpio_expander_1-net-4
- U14 pad 3: base_1_1-hv-2 -> column_0.gpio_expander_1-net-1
- U14 pad 4: base_1_1-gnd -> column_0.gpio_expander_1-net-5
- U14 pad 5: base_1_1-hv -> column_0.gpio_expander_1-net
- U14 pad 6: base_1_1-hv -> column_0.gpio_expander_1-gnd
- U14 pad 7: base_1_1-gnd -> column_0.gpio_expander_1-net-6
- U14 pad 8: base_1_1-hv-1 -> column_0.gpio_expander_1-net-2
- U14 pad 9: base_1_1-hv-1 -> column_0.gpio_expander_1-net-3
- U15 pad 1: base_1_2-gnd -> column_0.gpio_expander_2-RESET
- U15 pad 10: base_1_2-gnd -> column_0.gpio_expander_2-net-4
- U15 pad 4: base_1_2-gnd -> column_0.gpio_expander_2-net
- U15 pad 6: base_1_2-line-1 -> column_0.gpio_expander_2-gnd
- U15 pad 7: base_1_2-gnd -> column_0.gpio_expander_2-net-6
- U16 pad 1: base_1_2-gnd -> gnd-3
- U16 pad 10: base_1_2-gnd -> column_0.i2c_mux-SD3
- U16 pad 2: base_1_2-hv-1 -> gnd-3
- U16 pad 3: base_1_2-hv-1 -> column_0.i2c_mux-RESET_
- U16 pad 4: base_1_2-gnd -> column_0.i2c_mux-SD0
- U16 pad 5: base_1_2-hv-2 -> column_0.i2c_mux-SC0
- U16 pad 6: base_1_2-hv-2 -> column_0.i2c_mux-SD1
- U16 pad 7: base_1_2-gnd -> column_0.i2c_mux-SC1
- U16 pad 8: base_1_2-hv -> column_0.i2c_mux-SD2
- U16 pad 9: base_1_2-hv -> column_0.i2c_mux-SC2
- U2 pad 1: base_0_0-gnd -> ac_in_line-net
- U2 pad 2: base_0_0-hv -> ac_in_line-net
- U2 pad 3: base_0_0-hv -> ac_in_line-net
- U2 pad 4: base_0_0-gnd -> ac_in_line-net
- U27 pad 1: base_2_3-gnd -> column_1.gpio_expander_1-RESET
- U27 pad 10: base_2_3-gnd -> column_1.gpio_expander_1-net-1
- U27 pad 4: base_2_3-gnd -> column_1.gpio_expander_1-net-7
- U27 pad 6: base_2_3-line-1 -> column_1.gpio_expander_1-gnd
- U27 pad 7: base_2_3-gnd -> column_1.gpio_expander_1-net-6
- U28 pad 1: base_2_3-gnd -> column_1.gpio_expander_2-VCCP
- U28 pad 10: base_2_3-gnd -> column_1.gpio_expander_2-net-7
- U28 pad 2: base_2_3-hv-1 -> column_1.gpio_expander_2-net-2
- U28 pad 3: base_2_3-hv-1 -> column_1.gpio_expander_2-net-3
- U28 pad 4: base_2_3-gnd -> column_1.gpio_expander_2-net-1
- U28 pad 5: base_2_3-hv -> column_1.gpio_expander_2-net
- U28 pad 6: base_2_3-hv -> column_1.gpio_expander_2-gnd
- U28 pad 7: base_2_3-gnd -> column_1.gpio_expander_2-net-4
- U28 pad 8: base_2_3-hv-2 -> column_1.gpio_expander_2-net-5
- U28 pad 9: base_2_3-hv-2 -> column_1.gpio_expander_2-net-6
- U29 pad 1: base_2_4-gnd -> gnd-1
- U29 pad 10: base_2_4-gnd -> column_1.i2c_mux-SD3
- U29 pad 2: base_2_4-line-5 -> gnd-1
- U29 pad 3: base_2_4-line-2 -> column_1.i2c_mux-RESET_
- U29 pad 4: base_2_4-gnd -> column_1.i2c_mux-SD0
- U29 pad 5: base_2_4-line -> column_1.i2c_mux-SC0
- U29 pad 6: base_2_4-line-4 -> column_1.i2c_mux-SD1
- U29 pad 7: base_2_4-gnd -> column_1.i2c_mux-SC1
- U29 pad 8: base_2_4-line-1 -> column_1.i2c_mux-SD2
- U29 pad 9: base_2_4-line-3 -> column_1.i2c_mux-SC2
- U3 pad 1: base_0_1-gnd -> ac_in_neutral-net
- U3 pad 2: base_0_1-line-1 -> ac_in_neutral-net
- U3 pad 3: base_0_1-line-3 -> ac_in_neutral-net
- U3 pad 4: base_0_1-gnd -> ac_in_neutral-net
- U30 pad 1: base_2_4-gnd -> column_2.base_0-gnd
- U30 pad 10: base_2_4-gnd -> column_2.base_0-gnd
- U30 pad 2: base_2_4-hv -> column_2.base_0-line-5
- U30 pad 3: base_2_4-hv -> column_2.base_0-line
- U30 pad 4: base_2_4-gnd -> column_2.base_0-gnd
- U30 pad 5: base_2_4-hv-1 -> column_2.base_0-line-4
- U30 pad 6: base_2_4-hv-1 -> column_2.base_0-line-2
- U30 pad 7: base_2_4-gnd -> column_2.base_0-gnd
- U30 pad 8: base_2_4-hv-2 -> column_2.base_0-line-1
- U30 pad 9: base_2_4-hv-2 -> column_2.base_0-line-3
- U31 pad 1: base_3_0-gnd -> column_2.base_0-gnd
- U31 pad 10: base_3_0-gnd -> column_2.base_0-gnd
- U31 pad 2: base_3_0-line-5 -> column_2.base_0-hv
- U31 pad 3: base_3_0-line-1 -> column_2.base_0-hv
- U31 pad 4: base_3_0-gnd -> column_2.base_0-gnd
- U31 pad 5: base_3_0-line -> column_2.base_0-hv-1
- U31 pad 6: base_3_0-line-3 -> column_2.base_0-hv-1
- U31 pad 7: base_3_0-gnd -> column_2.base_0-gnd
- U31 pad 8: base_3_0-line-4 -> column_2.base_0-hv-2
- U31 pad 9: base_3_0-line-2 -> column_2.base_0-hv-2
- U32 pad 1: base_3_0-gnd -> column_2.base_1-gnd
- U32 pad 10: base_3_0-gnd -> column_2.base_1-gnd
- U32 pad 2: base_3_0-hv -> column_2.base_1-line-1
- U32 pad 3: base_3_0-hv -> column_2.base_1-line-3
- U32 pad 4: base_3_0-gnd -> column_2.base_1-gnd
- U32 pad 5: base_3_0-hv-1 -> column_2.base_1-line-5
- U32 pad 6: base_3_0-hv-1 -> column_2.base_1-line
- U32 pad 7: base_3_0-gnd -> column_2.base_1-gnd
- U32 pad 8: base_3_0-hv-2 -> column_2.base_1-line-4
- U32 pad 9: base_3_0-hv-2 -> column_2.base_1-line-2
- U33 pad 1: base_3_1-gnd -> column_2.base_1-gnd
- U33 pad 10: base_3_1-gnd -> column_2.base_1-gnd
- U33 pad 2: base_3_1-line-4 -> column_2.base_1-hv
- U33 pad 3: base_3_1-line-3 -> column_2.base_1-hv
- U33 pad 4: base_3_1-gnd -> column_2.base_1-gnd
- U33 pad 5: base_3_1-line-2 -> column_2.base_1-hv-1
- U33 pad 6: base_3_1-line-5 -> column_2.base_1-hv-1
- U33 pad 7: base_3_1-gnd -> column_2.base_1-gnd
- U33 pad 8: base_3_1-line-1 -> column_2.base_1-hv-2
- U33 pad 9: base_3_1-line -> column_2.base_1-hv-2
- U34 pad 1: base_3_1-gnd -> column_2.base_2-gnd
- U34 pad 10: base_3_1-gnd -> column_2.base_2-gnd
- U34 pad 2: base_3_1-hv-1 -> column_2.base_2-line-4
- U34 pad 3: base_3_1-hv-1 -> column_2.base_2-line-2
- U34 pad 4: base_3_1-gnd -> column_2.base_2-gnd
- U34 pad 5: base_3_1-hv -> column_2.base_2-line-3
- U34 pad 6: base_3_1-hv -> column_2.base_2-line
- U34 pad 7: base_3_1-gnd -> column_2.base_2-gnd
- U34 pad 8: base_3_1-hv-2 -> column_2.base_2-line-1
- U34 pad 9: base_3_1-hv-2 -> column_2.base_2-line-5
- U35 pad 1: base_3_2-gnd -> column_2.base_2-gnd
- U35 pad 10: base_3_2-gnd -> column_2.base_2-gnd
- U35 pad 2: base_3_2-line-5 -> column_2.base_2-hv-1
- U35 pad 3: base_3_2-line -> column_2.base_2-hv-1
- U35 pad 4: base_3_2-gnd -> column_2.base_2-gnd
- U35 pad 5: base_3_2-line-1 -> column_2.base_2-hv
- U35 pad 6: base_3_2-line-3 -> column_2.base_2-hv
- U35 pad 7: base_3_2-gnd -> column_2.base_2-gnd
- U35 pad 8: base_3_2-line-4 -> column_2.base_2-hv-2
- U35 pad 9: base_3_2-line-2 -> column_2.base_2-hv-2
- U36 pad 1: base_3_2-gnd -> column_2.base_3-gnd
- U36 pad 10: base_3_2-gnd -> column_2.base_3-gnd
- U36 pad 2: base_3_2-hv -> column_2.base_3-line-1
- U36 pad 3: base_3_2-hv -> column_2.base_3-line-4
- U36 pad 4: base_3_2-gnd -> column_2.base_3-gnd
- U36 pad 5: base_3_2-hv-2 -> column_2.base_3-line-3
- U36 pad 6: base_3_2-hv-2 -> column_2.base_3-line-2
- U36 pad 7: base_3_2-gnd -> column_2.base_3-gnd
- U36 pad 8: base_3_2-hv-1 -> column_2.base_3-line-5
- U36 pad 9: base_3_2-hv-1 -> column_2.base_3-line
- U37 pad 1: base_3_3-gnd -> column_2.base_3-gnd
- U37 pad 10: base_3_3-gnd -> column_2.base_3-gnd
- U37 pad 2: base_3_3-line-4 -> column_2.base_3-hv-2
- U37 pad 3: base_3_3-line-1 -> column_2.base_3-hv-2
- U37 pad 4: base_3_3-gnd -> column_2.base_3-gnd
- U37 pad 5: base_3_3-line-3 -> column_2.base_3-hv-1
- U37 pad 6: base_3_3-line-5 -> column_2.base_3-hv-1
- U37 pad 7: base_3_3-gnd -> column_2.base_3-gnd
- U37 pad 8: base_3_3-line-2 -> column_2.base_3-hv
- U37 pad 9: base_3_3-line -> column_2.base_3-hv
- U38 pad 1: base_3_3-gnd -> column_2.base_4-gnd
- U38 pad 10: base_3_3-gnd -> column_2.base_4-gnd
- U38 pad 2: base_3_3-hv-1 -> column_2.base_4-line-5
- U38 pad 3: base_3_3-hv-1 -> column_2.base_4-line-3
- U38 pad 4: base_3_3-gnd -> column_2.base_4-gnd
- U38 pad 5: base_3_3-hv-2 -> column_2.base_4-line-4
- U38 pad 6: base_3_3-hv-2 -> column_2.base_4-line-1
- U38 pad 7: base_3_3-gnd -> column_2.base_4-gnd
- U38 pad 8: base_3_3-hv -> column_2.base_4-line
- U38 pad 9: base_3_3-hv -> column_2.base_4-line-2
- U39 pad 1: base_3_4-gnd -> column_2.base_4-gnd
- U39 pad 10: base_3_4-gnd -> column_2.base_4-gnd
- U39 pad 2: base_3_4-line-4 -> column_2.base_4-hv-2
- U39 pad 3: base_3_4-line-2 -> column_2.base_4-hv-2
- U39 pad 4: base_3_4-gnd -> column_2.base_4-gnd
- U39 pad 5: base_3_4-line-1 -> column_2.base_4-hv
- U39 pad 6: base_3_4-line-5 -> column_2.base_4-hv
- U39 pad 7: base_3_4-gnd -> column_2.base_4-gnd
- U39 pad 8: base_3_4-line -> column_2.base_4-hv-1
- U39 pad 9: base_3_4-line-3 -> column_2.base_4-hv-1
- U4 pad 1: base_0_1-gnd -> column_0.base_0-gnd
- U4 pad 10: base_0_1-gnd -> column_0.base_0-gnd
- U4 pad 2: base_0_1-hv-1 -> column_0.base_0-line-2
- U4 pad 3: base_0_1-hv-1 -> column_0.base_0-line-3
- U4 pad 4: base_0_1-gnd -> column_0.base_0-gnd
- U4 pad 5: base_0_1-hv-2 -> column_0.base_0-line-4
- U4 pad 6: base_0_1-hv-2 -> column_0.base_0-line
- U4 pad 7: base_0_1-gnd -> column_0.base_0-gnd
- U4 pad 8: base_0_1-hv -> column_0.base_0-line-5
- U4 pad 9: base_0_1-hv -> column_0.base_0-line-1
- U40 pad 1: base_3_4-gnd -> column_2.gpio_expander_1-VCCI
- U40 pad 10: base_3_4-gnd -> column_2.gpio_expander_1-net-5
- U40 pad 2: base_3_4-hv-1 -> column_2.gpio_expander_1-net-7
- U40 pad 3: base_3_4-hv-1 -> column_2.gpio_expander_1-net-4
- U40 pad 4: base_3_4-gnd -> column_2.gpio_expander_1-net-2
- U40 pad 5: base_3_4-hv -> column_2.gpio_expander_1-net-6
- U40 pad 6: base_3_4-hv -> column_2.gpio_expander_1-gnd
- U40 pad 7: base_3_4-gnd -> column_2.gpio_expander_1-net
- U40 pad 8: base_3_4-hv-2 -> column_2.gpio_expander_1-net-3
- U40 pad 9: base_3_4-hv-2 -> column_2.gpio_expander_1-net-1
- U41 pad 1: base_4_0-gnd -> column_2.gpio_expander_2-VCCP
- U41 pad 10: base_4_0-gnd -> column_2.gpio_expander_2-net-2
- U41 pad 4: base_4_0-gnd -> column_2.gpio_expander_2-net-4
- U41 pad 6: base_4_0-line-4 -> column_2.gpio_expander_2-gnd
- U41 pad 7: base_4_0-gnd -> column_2.gpio_expander_2-net-3
- U42 pad 1: base_4_0-gnd -> gnd
- U42 pad 10: base_4_0-gnd -> column_2.i2c_mux-SD3
- U42 pad 2: base_4_0-hv-1 -> gnd
- U42 pad 3: base_4_0-hv-1 -> column_2.i2c_mux-RESET_
- U42 pad 4: base_4_0-gnd -> column_2.i2c_mux-SD0
- U42 pad 5: base_4_0-hv -> column_2.i2c_mux-SC0
- U42 pad 6: base_4_0-hv -> column_2.i2c_mux-SD1
- U42 pad 7: base_4_0-gnd -> column_2.i2c_mux-SC1
- U42 pad 8: base_4_0-hv-2 -> column_2.i2c_mux-SD2
- U42 pad 9: base_4_0-hv-2 -> column_2.i2c_mux-SC2
- U5 pad 1: base_0_2-gnd -> column_0.base_0-gnd
- U5 pad 10: base_0_2-gnd -> column_0.base_0-gnd
- U5 pad 2: base_0_2-line-3 -> column_0.base_0-hv-2
- U5 pad 3: base_0_2-line-1 -> column_0.base_0-hv-2
- U5 pad 4: base_0_2-gnd -> column_0.base_0-gnd
- U5 pad 5: base_0_2-line-5 -> column_0.base_0-hv
- U5 pad 6: base_0_2-line-2 -> column_0.base_0-hv
- U5 pad 7: base_0_2-gnd -> column_0.base_0-gnd
- U5 pad 8: base_0_2-line-4 -> column_0.base_0-hv-1
- U5 pad 9: base_0_2-line -> column_0.base_0-hv-1
- U59 pad 5: hv-2 -> hv-6
- U6 pad 1: base_0_2-gnd -> column_0.base_1-gnd
- U6 pad 10: base_0_2-gnd -> column_0.base_1-gnd
- U6 pad 2: base_0_2-hv -> column_0.base_1-line-2
- U6 pad 3: base_0_2-hv -> column_0.base_1-line-3
- U6 pad 4: base_0_2-gnd -> column_0.base_1-gnd
- U6 pad 5: base_0_2-hv-2 -> column_0.base_1-line-1
- U6 pad 6: base_0_2-hv-2 -> column_0.base_1-line
- U6 pad 7: base_0_2-gnd -> column_0.base_1-gnd
- U6 pad 8: base_0_2-hv-1 -> column_0.base_1-line-4
- U6 pad 9: base_0_2-hv-1 -> column_0.base_1-line-5
- U61 pad 23: hil_core-line-1 -> hil_core-line-5
- U61 pad 24: hil_core-line-5 -> hil_core-line
- U61 pad 25: hil_core-line-4 -> hil_core-line-2
- U61 pad 26: hil_core-line-2 -> hil_core-line-4
- U61 pad 7: hv-3 -> hv-2
- U61 pad 8: hv-3 -> hv-2
- U62 pad 21: hil_core.usbpd.pd_controller-hv-1 -> hil_core.usbpd.pd_controller-hv
- U62 pad 23: hil_core.usbpd.pd_controller-hv -> hil_core.usbpd.pd_controller-hv-1
- U62 pad 4: hil_core.usbpd-line -> hil_core.usbpd-line-3
- U62 pad 5: hil_core.usbpd-line -> hil_core.usbpd-line-3
- U62 pad 8: hil_core.usbpd-line-3 -> hil_core.usbpd-line
- U7 pad 1: base_0_3-gnd -> column_0.base_1-gnd
- U7 pad 10: base_0_3-gnd -> column_0.base_1-gnd
- U7 pad 2: base_0_3-line-5 -> column_0.base_1-hv-2
- U7 pad 3: base_0_3-line -> column_0.base_1-hv-2
- U7 pad 4: base_0_3-gnd -> column_0.base_1-gnd
- U7 pad 5: base_0_3-line-4 -> column_0.base_1-hv-1
- U7 pad 6: base_0_3-line-2 -> column_0.base_1-hv-1
- U7 pad 7: base_0_3-gnd -> column_0.base_1-gnd
- U7 pad 8: base_0_3-line-3 -> column_0.base_1-hv
- U7 pad 9: base_0_3-line-1 -> column_0.base_1-hv
- U8 pad 1: base_0_3-gnd -> column_0.base_2-gnd
- U8 pad 10: base_0_3-gnd -> column_0.base_2-gnd
- U8 pad 2: base_0_3-hv-1 -> column_0.base_2-line-2
- U8 pad 3: base_0_3-hv-1 -> column_0.base_2-line-1
- U8 pad 4: base_0_3-gnd -> column_0.base_2-gnd
- U8 pad 5: base_0_3-hv -> column_0.base_2-line
- U8 pad 6: base_0_3-hv -> column_0.base_2-line-3
- U8 pad 7: base_0_3-gnd -> column_0.base_2-gnd
- U8 pad 8: base_0_3-hv-2 -> column_0.base_2-line-4
- U8 pad 9: base_0_3-hv-2 -> column_0.base_2-line-5
- U9 pad 1: base_0_4-gnd -> column_0.base_2-gnd
- U9 pad 10: base_0_4-gnd -> column_0.base_2-gnd
- U9 pad 2: base_0_4-line-1 -> column_0.base_2-hv-1
- U9 pad 3: base_0_4-line-5 -> column_0.base_2-hv-1
- U9 pad 4: base_0_4-gnd -> column_0.base_2-gnd
- U9 pad 5: base_0_4-line-4 -> column_0.base_2-hv-2
- U9 pad 6: base_0_4-line-2 -> column_0.base_2-hv-2
- U9 pad 7: base_0_4-gnd -> column_0.base_2-gnd
- U9 pad 8: base_0_4-line -> column_0.base_2-hv
- U9 pad 9: base_0_4-line-3 -> column_0.base_2-hv
- USB1 pad A4: hv-3 -> hv-2
- USB1 pad A9: hv-3 -> hv-2
- USB1 pad B4: hv-3 -> hv-2
- USB1 pad B9: hv-3 -> hv-2
- USB2 pad B5: hil_core.usbpd-line -> hil_core.usbpd-line-3
Routing:
- net hil_core-line: track 28.9 -> 75.5 mm
- net hv-2: track 16.7 -> 50.6 mm, vias 1 -> 3
- net hil_core-line-1: track 64.8 -> 31.8 mm, vias 2 -> 3
- net hv-3: track 50.6 -> 23.8 mm
- net hv: track 0.00 -> 23.8 mm, vias 0 -> 3
- net hv-8: track 0.00 -> 23.8 mm, vias 0 -> 3
- net hv-4: track 0.00 -> 23.8 mm, vias 0 -> 3
- net hv-7: track 0.00 -> 23.8 mm, vias 0 -> 3
- net hv-6: track 0.00 -> 16.7 mm, vias 0 -> 1
- net hil_core-line-5: track 75.5 -> 64.8 mm, vias 3 -> 2
- net hil_core.usbpd-line-3: track 4.26 -> 13.0 mm, vias 0 -> 2
- net hil_core.usbpd-line: track 13.0 -> 4.26 mm, vias 2 -> 0
- net gnd-2: track 0.00 -> 7.64 mm, vias 0 -> 3
- net gnd-4: track 0.00 -> 7.64 mm, vias 0 -> 3
- net gnd-1: track 0.00 -> 7.64 mm, vias 0 -> 3
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Other:
- outline, holes or cut-outs redrawn
