File: elec/layout/cell/cell.kicad_pcb (KiCad board)
At the start: 4 copper layers, 79.5 x 8 mm, 65 parts

Commit message: Cleanup layout for usb hub and usb-uart, add CM5 controller heatsink outline
Connections:
- C1 pad 1: hv-3 -> hv-7
- C1 pad 2: gnd-3 -> gnd
- C10 pad 2: gnd-8 -> gnd-5
- C11 pad 2: gnd-8 -> gnd-5
- C12 pad 1: hv -> hv-8
- C12 pad 2: gnd-8 -> gnd-5
- C13 pad 2: gnd -> gnd-8
- C14 pad 2: gnd -> gnd-8
- C15 pad 2: gnd-8 -> gnd-5
- C16 pad 2: gnd-8 -> gnd-5
- C2 pad 2: gnd-8 -> gnd-5
- C3 pad 2: gnd-8 -> gnd-5
- C4 pad 2: gnd-8 -> gnd-5
- C5 pad 2: gnd-8 -> gnd-5
- C6 pad 1: hv-6 -> hv-1
- C6 pad 2: gnd-8 -> gnd-5
- C7 pad 1: hv-6 -> hv-1
- C7 pad 2: gnd-8 -> gnd-5
- C8 pad 1: hv-6 -> hv-1
- C8 pad 2: gnd-8 -> gnd-5
- L1 pad 2: hv-6 -> hv-1
- L2 pad 2: hv -> hv-8
- Q1 pad 2: gnd-8 -> gnd-5
- Q2 pad 2: gnd -> gnd-8
- Q3 pad 2: gnd-8 -> gnd-5
- Q3 pad 3: gnd-5 -> gnd-3
- Q4 pad 3: gnd-4 -> gnd-7
- R10 pad 1: hv -> hv-8
- R10 pad 2: hv-8 -> hv-9
- R11 pad 2: gnd-8 -> gnd-5
- R12 pad 1: line-2 -> line-8
- R13 pad 1: line-2 -> line-8
- R13 pad 2: gnd-8 -> gnd-5
- R15 pad 1: line-4 -> line-9
- R16 pad 1: line-4 -> line-9
- R16 pad 2: gnd -> gnd-8
- R17 pad 1: line-1 -> line-2
- R18 pad 1: line-1 -> line-2
- R18 pad 2: gnd-8 -> gnd-5
- R19 pad 1: hv -> hv-8
- R19 pad 2: gnd-5 -> gnd-3
- R20 pad 1: line-7 -> line-4
- R21 pad 1: line-8 -> line-1
- R22 pad 1: line-11 -> line-3
- R23 pad 1: line-11 -> line-3
- R24 pad 2: hv-9 -> hv
- R25 pad 1: gnd-7 -> gnd-4
- R26 pad 1: hv-7 -> hv-6
- R26 pad 2: gnd-4 -> gnd-7
- R3 pad 1: hv-6 -> hv-1
- R4 pad 2: gnd-8 -> gnd-5
- R5 pad 1: line-6 -> line-11
- R8 pad 2: gnd-8 -> gnd-5
- R9 pad 1: line-3 -> line-7
- U1 pad 1: hv-3 -> hv-7
- U1 pad 2: gnd-3 -> gnd
- U1 pad 4: gnd-8 -> gnd-5
- U10 pad 10: gpio-net -> gpio-net-2
- U10 pad 12: line-8 -> line-1
- U10 pad 13: line-7 -> line-4
- U10 pad 16: gnd-8 -> gnd-5
- U10 pad 17: gnd-8 -> gnd-5
- U10 pad 3: gpio-net-2 -> gpio-net
- U10 pad 4: line-6 -> line-11
- U10 pad 5: line-3 -> line-7
- U10 pad 6: gnd-8 -> gnd-5
- U10 pad 7: line-1 -> line-2
- U10 pad 8: line-2 -> line-8
- U10 pad 9: line-11 -> line-3
- U11 pad 1: hv-1 -> hv-3
- U11 pad 2: line -> line-10
- U11 pad 3: line-5 -> line-6
- U11 pad 5: gnd-8 -> gnd-5
- U11 pad 6: line-8 -> line-1
- U11 pad 7: line-7 -> line-4
- U12 pad 3: gnd -> gnd-8
- U12 pad 4: line-10 -> line
- U13 pad 2: line-10 -> line
- U13 pad 3: gnd -> gnd-8
- U14 pad 1: gnd-8 -> gnd-5
- U2 pad 1: gnd-8 -> gnd-5
- U2 pad 10: line-8 -> line-1
- U2 pad 3: gnd-8 -> gnd-5
- U2 pad 4: hv-6 -> hv-1
- U2 pad 6: line-9 -> line-5
- U2 pad 7: hv-8 -> hv-9
- U2 pad 9: line-7 -> line-4
- U3 pad 2: gnd-8 -> gnd-5
- U3 pad 4: line-7 -> line-4
- U3 pad 5: line-8 -> line-1
- U4 pad 1: gnd-8 -> gnd-5
- U5 pad 2: gnd-8 -> gnd-5
- U5 pad 4: line-7 -> line-4
- U5 pad 5: line-8 -> line-1
- U5 pad 6: gnd-8 -> gnd-5
- U6 pad 3: gnd-8 -> gnd-5
- U6 pad 6: hv-6 -> hv-1
- U6 pad 7: gnd-8 -> gnd-5
- U7 pad 1: line-9 -> line-5
- U7 pad 2: gnd-8 -> gnd-5
- U7 pad 3: hv -> hv-8
- U7 pad 4: hv-8 -> hv-9
- U7 pad 5: gnd-8 -> gnd-5
- U8 pad 4: gnd-8 -> gnd-5
- U8 pad 5: hv-8 -> hv-9
- U8 pad 6: hv-7 -> hv-6
- U9 pad 3: gnd-7 -> gnd-4
- U9 pad 4: gnd-8 -> gnd-5
- U9 pad 5: hv-8 -> hv-9
Routing:
- net gnd-8: track 105.5 -> 0.00 mm, vias 31 -> 0
- net gnd-5: track 3.42 -> 105.5 mm, vias 0 -> 31
- net line-4: track 1.44 -> 44.5 mm, vias 0 -> 4
- net line-7: track 44.5 -> 7.72 mm, vias 4 -> 2
- net line-1: track 13.5 -> 43.5 mm, vias 2 -> 5
- net hv-9: track 0.00 -> 27.5 mm, vias 0 -> 1
- net hv-1: track 0.00 -> 24.3 mm, vias 0 -> 2
- net line-3: track 7.72 -> 31.7 mm
- net line-11: track 31.7 -> 12.8 mm
- net line-2: track 30.4 -> 13.5 mm
- net hv-8: track 27.5 -> 13.2 mm, vias 1 -> 2
- net hv: track 13.2 -> 0.00 mm, vias 2 -> 0
- net line-8: track 43.5 -> 30.4 mm, vias 5 -> 2
- net line-6: track 12.8 -> 0.00 mm, vias 2 -> 0
- net gnd: track 0.00 -> 10.8 mm, vias 0 -> 1
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- added copper zone on B.Cu, net gnd-5
- added copper zone on F.Cu, net gnd-5
- added copper zone on In2.Cu, net gnd-5
- removed copper zone on B.Cu, net gnd-8
- removed copper zone on F.Cu, net gnd-8
- removed copper zone on In2.Cu, net gnd-8

Commit message: checkin
Connections:
- C1 pad 1: hv-7 -> hv-6
- C10 pad 1: hv-5 -> hv-2
- C10 pad 2: gnd-5 -> gnd-1
- C11 pad 1: hv-5 -> hv-2
- C11 pad 2: gnd-5 -> gnd-1
- C12 pad 1: hv-8 -> hv
- C12 pad 2: gnd-5 -> gnd-1
- C13 pad 1: hv-2 -> hv-9
- C13 pad 2: gnd-8 -> gnd-5
- C14 pad 1: hv-2 -> hv-9
- C14 pad 2: gnd-8 -> gnd-5
- C15 pad 2: gnd-5 -> gnd-1
- C16 pad 2: gnd-5 -> gnd-1
- C2 pad 2: gnd-5 -> gnd-1
- C3 pad 2: gnd-5 -> gnd-1
- C4 pad 2: gnd-5 -> gnd-1
- C5 pad 2: gnd-5 -> gnd-1
- C6 pad 1: hv-1 -> hv-3
- C6 pad 2: gnd-5 -> gnd-1
- C7 pad 1: hv-1 -> hv-3
- C7 pad 2: gnd-5 -> gnd-1
- C8 pad 1: hv-1 -> hv-3
- C8 pad 2: gnd-5 -> gnd-1
- L1 pad 2: hv-1 -> hv-3
- L2 pad 1: hv-5 -> hv-2
- L2 pad 2: hv-8 -> hv
- LED3 pad 2: hv-2 -> hv-9
- Q1 pad 2: gnd-5 -> gnd-1
- Q2 pad 2: gnd-8 -> gnd-5
- Q3 pad 2: gnd-5 -> gnd-1
- Q3 pad 3: gnd-3 -> gnd-2
- Q4 pad 2: gnd-2 -> gnd-6
- Q4 pad 3: gnd-7 -> gnd-4
- R10 pad 1: hv-8 -> hv
- R10 pad 2: hv-9 -> hv-7
- R11 pad 2: gnd-5 -> gnd-1
- R12 pad 1: line-8 -> line-2
- R13 pad 1: line-8 -> line-2
- R13 pad 2: gnd-5 -> gnd-1
- R15 pad 1: line-9 -> line-4
- R16 pad 1: line-9 -> line-4
- R16 pad 2: gnd-8 -> gnd-5
- R17 pad 1: line-2 -> line-5
- R18 pad 1: line-2 -> line-5
- R18 pad 2: gnd-5 -> gnd-1
- R19 pad 1: hv-8 -> hv
- R19 pad 2: gnd-3 -> gnd-2
- R20 pad 1: line-4 -> line-9
- R22 pad 1: line-3 -> line-8
- R23 pad 1: line-3 -> line-8
- R23 pad 2: gnd-2 -> gnd-6
- R24 pad 2: hv -> hv-5
- R25 pad 1: gnd-4 -> gnd-7
- R25 pad 2: gnd-1 -> gnd-3
- R26 pad 1: hv-6 -> hv-8
- R26 pad 2: gnd-7 -> gnd-4
- R3 pad 1: hv-1 -> hv-3
- R4 pad 2: gnd-5 -> gnd-1
- R5 pad 1: line-11 -> line-7
- R7 pad 1: hv-5 -> hv-2
- R8 pad 2: gnd-5 -> gnd-1
- R9 pad 1: line-7 -> line-3
- U1 pad 1: hv-7 -> hv-6
- U1 pad 4: gnd-5 -> gnd-1
- U10 pad 10: gpio-net-2 -> gpio-net
- U10 pad 13: line-4 -> line-9
- U10 pad 16: gnd-5 -> gnd-1
- U10 pad 17: gnd-5 -> gnd-1
- U10 pad 3: gpio-net -> gpio-net-2
- U10 pad 4: line-11 -> line-7
- U10 pad 5: line-7 -> line-3
- U10 pad 6: gnd-5 -> gnd-1
- U10 pad 7: line-2 -> line-5
- U10 pad 8: line-8 -> line-2
- U10 pad 9: line-3 -> line-8
- U11 pad 1: hv-3 -> hv-1
- U11 pad 3: line-6 -> line
- U11 pad 4: gnd-6 -> gnd-8
- U11 pad 5: gnd-5 -> gnd-1
- U11 pad 7: line-4 -> line-9
- U12 pad 1: hv-2 -> hv-9
- U12 pad 3: gnd-8 -> gnd-5
- U12 pad 4: line -> line-11
- U13 pad 1: hv-2 -> hv-9
- U13 pad 2: line -> line-11
- U13 pad 3: gnd-8 -> gnd-5
- U14 pad 1: gnd-5 -> gnd-1
- U2 pad 1: gnd-5 -> gnd-1
- U2 pad 3: gnd-5 -> gnd-1
- U2 pad 4: hv-1 -> hv-3
- U2 pad 5: hv-5 -> hv-2
- U2 pad 6: line-5 -> line-6
- U2 pad 7: hv-9 -> hv-7
- U2 pad 9: line-4 -> line-9
- U3 pad 2: gnd-5 -> gnd-1
- U3 pad 4: line-4 -> line-9
- U4 pad 1: gnd-5 -> gnd-1
- U5 pad 2: gnd-5 -> gnd-1
- U5 pad 4: line-4 -> line-9
- U5 pad 6: gnd-5 -> gnd-1
- U6 pad 1: hv-5 -> hv-2
- U6 pad 3: gnd-5 -> gnd-1
- U6 pad 6: hv-1 -> hv-3
- U6 pad 7: gnd-5 -> gnd-1
- U7 pad 1: line-5 -> line-6
- U7 pad 2: gnd-5 -> gnd-1
- U7 pad 3: hv-8 -> hv
- U7 pad 4: hv-9 -> hv-7
- U7 pad 5: gnd-5 -> gnd-1
- U8 pad 3: gnd-2 -> gnd-6
- U8 pad 4: gnd-5 -> gnd-1
- U8 pad 5: hv-9 -> hv-7
- U8 pad 6: hv-6 -> hv-8
- U9 pad 1: hv-2 -> hv-9
- U9 pad 3: gnd-4 -> gnd-7
- U9 pad 4: gnd-5 -> gnd-1
- U9 pad 5: hv-9 -> hv-7
Routing:
- net gnd-5: track 105.5 -> 0.00 mm, vias 31 -> 0
- net gnd-1: track 0.00 -> 105.5 mm, vias 0 -> 31
- net line-9: track 1.44 -> 44.5 mm, vias 0 -> 4
- net line-4: track 44.5 -> 1.44 mm, vias 4 -> 0
- net hv-9: track 27.5 -> 0.00 mm, vias 1 -> 0
- net hv-3: track 0.00 -> 24.3 mm, vias 0 -> 2
- net hv-1: track 24.3 -> 0.00 mm, vias 2 -> 0
- net line-3: track 31.7 -> 7.72 mm
- net hv-7: track 4.33 -> 27.5 mm, vias 0 -> 1
- net line-2: track 13.5 -> 30.4 mm
- net hv-5: track 15.6 -> 0.00 mm
- net hv-2: track 0.00 -> 15.6 mm
- net hv: track 0.00 -> 13.2 mm, vias 0 -> 2
- net line-11: track 12.8 -> 2.29 mm, vias 2 -> 0
- net hv-6: track 14.3 -> 4.33 mm, vias 1 -> 0
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- added copper zone on B.Cu, net gnd-1
- added copper zone on F.Cu, net gnd-1
- added copper zone on In2.Cu, net gnd-1
- removed copper zone on B.Cu, net gnd-5
- removed copper zone on F.Cu, net gnd-5
- removed copper zone on In2.Cu, net gnd-5

Commit message: build with excluded checks
Connections:
- C1 pad 1: hv-6 -> hv-1
- C1 pad 2: gnd -> gnd-8
- C10 pad 1: hv-2 -> hv-6
- C10 pad 2: gnd-1 -> gnd
- C11 pad 1: hv-2 -> hv-6
- C11 pad 2: gnd-1 -> gnd
- C12 pad 1: hv -> hv-4
- C12 pad 2: gnd-1 -> gnd
- C13 pad 2: gnd-5 -> gnd-4
- C14 pad 2: gnd-5 -> gnd-4
- C15 pad 2: gnd-1 -> gnd
- C16 pad 2: gnd-1 -> gnd
- C2 pad 2: gnd-1 -> gnd
- C3 pad 2: gnd-1 -> gnd
- C4 pad 2: gnd-1 -> gnd
- C5 pad 2: gnd-1 -> gnd
- C6 pad 2: gnd-1 -> gnd
- C7 pad 2: gnd-1 -> gnd
- C8 pad 2: gnd-1 -> gnd
- L2 pad 1: hv-2 -> hv-6
- L2 pad 2: hv -> hv-4
- Q1 pad 2: gnd-1 -> gnd
- Q2 pad 2: gnd-5 -> gnd-4
- Q3 pad 2: gnd-1 -> gnd
- Q3 pad 3: gnd-2 -> gnd-5
- Q4 pad 2: gnd-6 -> gnd-2
- Q4 pad 3: gnd-4 -> gnd-6
- R10 pad 1: hv -> hv-4
- R10 pad 2: hv-7 -> hv-8
- R11 pad 2: gnd-1 -> gnd
- R12 pad 1: line-2 -> line-11
- R13 pad 1: line-2 -> line-11
- R13 pad 2: gnd-1 -> gnd
- R15 pad 1: line-4 -> line
- R16 pad 1: line-4 -> line
- R16 pad 2: gnd-5 -> gnd-4
- R17 pad 1: line-5 -> line-4
- R18 pad 1: line-5 -> line-4
- R18 pad 2: gnd-1 -> gnd
- R19 pad 1: hv -> hv-4
- R19 pad 2: gnd-2 -> gnd-5
- R20 pad 1: line-9 -> line-7
- R21 pad 1: line-1 -> line-3
- R22 pad 1: line-8 -> line-6
- R23 pad 1: line-8 -> line-6
- R23 pad 2: gnd-6 -> gnd-2
- R24 pad 1: hv-4 -> hv-7
- R25 pad 2: gnd-3 -> gnd-1
- R26 pad 1: hv-8 -> hv-2
- R26 pad 2: gnd-4 -> gnd-6
- R4 pad 2: gnd-1 -> gnd
- R5 pad 1: line-7 -> line-2
- R7 pad 1: hv-2 -> hv-6
- R8 pad 2: gnd-1 -> gnd
- R9 pad 1: line-3 -> line-1
- U1 pad 1: hv-6 -> hv-1
- U1 pad 2: gnd -> gnd-8
- U1 pad 4: gnd-1 -> gnd
- U10 pad 12: line-1 -> line-3
- U10 pad 13: line-9 -> line-7
- U10 pad 16: gnd-1 -> gnd
- U10 pad 17: gnd-1 -> gnd
- U10 pad 4: line-7 -> line-2
- U10 pad 5: line-3 -> line-1
- U10 pad 6: gnd-1 -> gnd
- U10 pad 7: line-5 -> line-4
- U10 pad 8: line-2 -> line-11
- U10 pad 9: line-8 -> line-6
- U11 pad 1: hv-1 -> hv
- U11 pad 2: line-10 -> line-9
- U11 pad 3: line -> line-10
- U11 pad 4: gnd-8 -> gnd-3
- U11 pad 5: gnd-1 -> gnd
- U11 pad 6: line-1 -> line-3
- U11 pad 7: line-9 -> line-7
- U12 pad 3: gnd-5 -> gnd-4
- U12 pad 4: line-11 -> line-5
- U13 pad 2: line-11 -> line-5
- U13 pad 3: gnd-5 -> gnd-4
- U14 pad 1: gnd-1 -> gnd
- U2 pad 1: gnd-1 -> gnd
- U2 pad 10: line-1 -> line-3
- U2 pad 3: gnd-1 -> gnd
- U2 pad 5: hv-2 -> hv-6
- U2 pad 6: line-6 -> line-8
- U2 pad 7: hv-7 -> hv-8
- U2 pad 9: line-9 -> line-7
- U3 pad 2: gnd-1 -> gnd
- U3 pad 4: line-9 -> line-7
- U3 pad 5: line-1 -> line-3
- U4 pad 1: gnd-1 -> gnd
- U5 pad 2: gnd-1 -> gnd
- U5 pad 4: line-9 -> line-7
- U5 pad 5: line-1 -> line-3
- U5 pad 6: gnd-1 -> gnd
- U6 pad 1: hv-2 -> hv-6
- U6 pad 3: gnd-1 -> gnd
- U6 pad 7: gnd-1 -> gnd
- U7 pad 1: line-6 -> line-8
- U7 pad 2: gnd-1 -> gnd
- U7 pad 3: hv -> hv-4
- U7 pad 4: hv-7 -> hv-8
- U7 pad 5: gnd-1 -> gnd
- U8 pad 3: gnd-6 -> gnd-2
- U8 pad 4: gnd-1 -> gnd
- U8 pad 5: hv-7 -> hv-8
- U8 pad 6: hv-8 -> hv-2
- U9 pad 4: gnd-1 -> gnd
- U9 pad 5: hv-7 -> hv-8
- U9 pad 6: hv-4 -> hv-7
Routing:
- net gnd-1: track 105.5 -> 0.00 mm, vias 31 -> 0
- net gnd: track 10.8 -> 105.5 mm, vias 1 -> 31
- net line-9: track 44.5 -> 0.00 mm, vias 4 -> 0
- net line-3: track 7.72 -> 43.5 mm, vias 2 -> 5
- net line-1: track 43.5 -> 7.72 mm, vias 5 -> 2
- net line-7: track 12.8 -> 44.5 mm, vias 2 -> 4
- net line-11: track 2.29 -> 30.4 mm, vias 0 -> 2
- net line-8: track 31.7 -> 4.47 mm, vias 2 -> 0
- net line-6: track 4.47 -> 31.7 mm, vias 0 -> 2
- net hv-7: track 27.5 -> 1.58 mm, vias 1 -> 0
- net line-2: track 30.4 -> 12.8 mm
- net hv-8: track 14.3 -> 27.5 mm
- net hv: track 13.2 -> 0.00 mm, vias 2 -> 0
- net line-4: track 1.44 -> 13.5 mm, vias 0 -> 2
- net hv-4: track 1.58 -> 13.2 mm, vias 0 -> 2
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- added copper zone on B.Cu, net gnd
- added copper zone on F.Cu, net gnd
- added copper zone on In2.Cu, net gnd
- removed copper zone on B.Cu, net gnd-1
- removed copper zone on F.Cu, net gnd-1
- removed copper zone on In2.Cu, net gnd-1

Commit message: update cell with addressing
Parts:
- removed C8: 10µF ±10% 25V X5R, atopile:C0805-3b2e55
- C1: value 2.2µF ±10% 25V X7R -> 2.2µF ±10% 50V X5R
- C5: value 100nF ±10% 16V X7R -> 10µF ±10% 25V X5R; footprint atopile:C0402-b3ef17 -> atopile:C0805-3b2e55
- R1, R11, R14: value 1kΩ ±1% 62.5mW -> 2.2kΩ ±1% 62.5mW
- R3: value 36.5kΩ ±0% 62.5mW -> 36.5kΩ ±1% 62.5mW
- R6: value 43.2kΩ ±1% 62.5mW -> 43kΩ ±1% 62.5mW
- U10: footprint atopile:QFN-16_L3.0-W3.0-P0.50-BL-EP1.7-3a4c56 -> lib:SOT-23-6_L2.9-W1.6-P0.95-LS2.8-BL
- U5: footprint lib:SOT-23-6_L2.9-W1.6-P0.95-LS2.8-BL -> atopile:QFN-16_L3.0-W3.0-P0.50-BL-EP1.7-3a4c56
- moved C5 11.1 mm to (136.3, 108.2), turned to -90 degrees
- moved U5 6.35 mm to (143.1, 103.6), turned to -90 degrees
- moved U10 6.30 mm to (136.8, 103.3), turned to 180 degrees
- moved C7 4.22 mm to (132.7, 108.2)
- moved C6 0.43 mm to (134.5, 108.2)
- moved C3 0.38 mm to (124.2, 102.9)
- moved C4 0.17 mm to (122.3, 102.9)
- moved U3 0.05 mm to (133.8, 103.3)
Connections:
- net buck-line renamed buck-VOUT
- C1 pad 1: hv-1 -> hv-5
- C1 pad 2: gnd-8 -> gnd-4
- C10 pad 1: hv-6 -> hv
- C10 pad 2: gnd -> gnd-5
- C11 pad 1: hv-6 -> hv
- C11 pad 2: gnd -> gnd-5
- C12 pad 2: gnd -> gnd-5
- C13 pad 1: hv-9 -> hv-8
- C13 pad 2: gnd-4 -> gnd-1
- C14 pad 1: hv-9 -> hv-8
- C14 pad 2: gnd-4 -> gnd-1
- C15 pad 2: gnd -> gnd-5
- C16 pad 2: gnd -> gnd-5
- C2 pad 2: gnd -> gnd-5
- C3 pad 2: gnd -> gnd-5
- C4 pad 2: gnd -> gnd-5
- C5 pad 1: 5V -> hv-7
- C5 pad 2: gnd -> gnd-5
- C6 pad 1: hv-3 -> hv-7
- C6 pad 2: gnd -> gnd-5
- C7 pad 1: hv-3 -> hv-7
- C7 pad 2: gnd -> gnd-5
- L1 pad 2: hv-3 -> hv-7
- L2 pad 1: hv-6 -> hv
- LED3 pad 2: hv-9 -> hv-8
- Q1 pad 2: gnd -> gnd-5
- Q2 pad 2: gnd-4 -> gnd-1
- Q3 pad 2: gnd -> gnd-5
- Q3 pad 3: gnd-5 -> gnd-3
- Q4 pad 2: gnd-2 -> gnd-5
- R10 pad 2: hv-8 -> hv-6
- R11 pad 2: gnd -> gnd-5
- R12 pad 1: line-11 -> line-8
- R13 pad 1: line-11 -> line-8
- R13 pad 2: gnd -> gnd-5
- R15 pad 1: line -> line-1
- R16 pad 1: line -> line-1
- R16 pad 2: gnd-4 -> gnd-1
- R17 pad 1: line-4 -> line-7
- R18 pad 1: line-4 -> line-7
- R18 pad 2: gnd -> gnd-5
- R19 pad 2: gnd-5 -> gnd-3
- R20 pad 1: line-7 -> SDA
- R21 pad 1: line-3 -> SCL
- R22 pad 1: line-6 -> line
- R23 pad 1: line-6 -> line
- R23 pad 2: gnd-2 -> gnd-5
- R24 pad 1: hv-7 -> hv-3
- R24 pad 2: hv-5 -> hv-2
- R25 pad 2: gnd-1 -> gnd
- R26 pad 1: hv-2 -> hv-9
- R3 pad 1: hv-3 -> hv-7
- R4 pad 2: gnd -> gnd-5
- R6 pad 1: ldo-line -> ldo-VOUT
- R7 pad 1: hv-6 -> hv
- R8 pad 2: gnd -> gnd-5
- R9 pad 1: line-1 -> line-4
- U1 pad 1: hv-1 -> hv-5
- U1 pad 2: gnd-8 -> gnd-4
- U1 pad 4: gnd -> gnd-5
- U10 pad 1: 3V3 -> ldo-VOUT
- U10 pad 2: gpio-net-1 -> gnd-5
- U10 pad 3: gpio-net-2 -> 3V3
- U10 pad 4: line-2 -> SDA
- U10 pad 5: line-1 -> SCL
- U10 pad 6: gnd -> gnd-5
- U11 pad 1: hv -> hv-1
- U11 pad 2: line-9 -> line-3
- U11 pad 3: line-10 -> line-5
- U11 pad 4: gnd-3 -> gnd-2
- U11 pad 5: gnd -> gnd-5
- U11 pad 6: line-3 -> SCL
- U11 pad 7: line-7 -> SDA
- U12 pad 1: hv-9 -> hv-8
- U12 pad 3: gnd-4 -> gnd-1
- U12 pad 4: line-5 -> line-6
- U13 pad 1: hv-9 -> hv-8
- U13 pad 2: line-5 -> line-6
- U13 pad 3: gnd-4 -> gnd-1
- U14 pad 1: gnd -> gnd-5
- U2 pad 1: gnd -> gnd-5
- U2 pad 10: line-3 -> SCL
- U2 pad 3: gnd -> gnd-5
- U2 pad 4: hv-3 -> hv-7
- U2 pad 5: hv-6 -> hv
- U2 pad 6: line-8 -> line-9
- U2 pad 7: hv-8 -> hv-6
- U2 pad 9: line-7 -> SDA
- U3 pad 2: gnd -> gnd-5
- U3 pad 4: line-7 -> SDA
- U3 pad 5: line-3 -> SCL
- U3 pad 6: 5V -> 3V3
- U4 pad 1: gnd -> gnd-5
- U5 pad 1: ldo-line -> 3V3
- U5 pad 2: gnd -> gpio-line-2
- U5 pad 3: 3V3 -> line-2
- U5 pad 4: line-7 -> gpio-line
- U5 pad 5: line-3 -> line-4
- U5 pad 6: gnd -> gnd-5
- U6 pad 1: hv-6 -> hv
- U6 pad 3: gnd -> gnd-5
- U6 pad 6: hv-3 -> hv-7
- U6 pad 7: gnd -> gnd-5
- U7 pad 1: line-8 -> line-9
- U7 pad 2: gnd -> gnd-5
- U7 pad 4: hv-8 -> hv-6
- U7 pad 5: gnd -> gnd-5
- U8 pad 3: gnd-2 -> gnd-5
- U8 pad 4: gnd -> gnd-5
- U8 pad 5: hv-8 -> hv-6
- U8 pad 6: hv-2 -> hv-9
- U9 pad 1: hv-9 -> hv-8
- U9 pad 4: gnd -> gnd-5
- U9 pad 5: hv-8 -> hv-6
- U9 pad 6: hv-7 -> hv-3
Routing:
- net gnd: track 105.5 -> 0.00 mm, vias 31 -> 0
- net gnd-5: track 3.42 -> 107.9 mm, vias 0 -> 33
- net SDA: track 0.00 -> 46.7 mm, vias 0 -> 4
- net SCL: track 0.00 -> 44.4 mm, vias 0 -> 5
- net line-3: track 43.5 -> 0.00 mm, vias 5 -> 0
- net line-7: track 44.5 -> 13.5 mm, vias 4 -> 2
- net line-11: track 30.4 -> 0.00 mm, vias 2 -> 0
- net line: track 1.44 -> 31.7 mm, vias 0 -> 2
- net line-6: track 31.7 -> 2.29 mm, vias 2 -> 0
- net line-8: track 4.47 -> 30.4 mm, vias 0 -> 2
- net hv-7: track 1.58 -> 24.3 mm, vias 0 -> 2
- net hv-3: track 24.3 -> 1.58 mm, vias 2 -> 0
- net hv-8: track 27.5 -> 10.0 mm
- net hv: track 0.00 -> 15.6 mm
- net (no net): track 15.3 -> 0.00 mm, vias 7 -> 0
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- added copper zone on B.Cu, net gnd-5
- added copper zone on F.Cu, net gnd-5
- added copper zone on In2.Cu, net gnd-5
- removed copper zone on B.Cu, net gnd
- removed copper zone on F.Cu, net gnd
- removed copper zone on In2.Cu, net gnd
